File: digitalSystemBoard/OOI.sch (KiCad schematic (older format))
At the start: 60 parts, among them U10 IO_Switch, U11 IO_Switch, U12 IO_Switch, U13 IO_Switch, U14 IO_Switch, U5 IO_Switch, U6 IO_Switch, U7 IO_Switch, U8 IO_Switch, U9 IO_Switch

Commit message: Update footprints and CLOCK_BLOCK Sch
Parts:
- U10, U11, U12, U13, U14, U5, U6, U7, U8, U9: symbol digitalSystemBoard:IO_Switch -> digitalSystemBoard-rescue:IO_Switch-digitalSystemBoard
Changed lines of the file:
@@
 NoConn ~ 1376 1440
 $Comp
-L digitalSystemBoard:IO_Switch U5
+L digitalSystemBoard-rescue:IO_Switch-digitalSystemBoard U5
 U 1 1 5F8D12EE
 P 1176 1590
+AR Path="/5F8D12EE" Ref="U5"  Part="1"
+AR Path="/5F8CFBC4/5F8D12EE" Ref="U5"  Part="1"
 F 0 "U5" H 1176 1905 50  0000 C CNN
 F 1 "IO_Switch" H 1176 1814 50  0000 C CNN
@@
 NoConn ~ 3660 1428
 $Comp
-L digitalSystemBoard:IO_Switch U6
+L digitalSystemBoard-rescue:IO_Switch-digitalSystemBoard U6
 U 1 1 5F942F24
 P 3460 1578
+AR Path="/5F942F24" Ref="U6"  Part="1"
+AR Path="/5F8CFBC4/5F942F24" Ref="U6"  Part="1"
 F 0 "U6" H 3460 1893 50  0000 C CNN
 F 1 "IO_Switch" H 3460 1802 50  0000 C CNN
@@
 NoConn ~ 5888 1446
 $Comp
-L digitalSystemBoard:IO_Switch U7
+L digitalSystemBoard-rescue:IO_Switch-digitalSystemBoard U7
 U 1 1 5F944061
 P 5688 1596
+AR Path="/5F944061" Ref="U7"  Part="1"
+AR Path="/5F8CFBC4/5F944061" Ref="U7"  Part="1"
 F 0 "U7" H 5688 1911 50  0000 C CNN
 F 1 "IO_Switch" H 5688 1820 50  0000 C CNN
@@
 NoConn ~ 8116 1462
 $Comp
-L digitalSystemBoard:IO_Switch U8
+L digitalSystemBoard-rescue:IO_Switch-digitalSystemBoard U8
 U 1 1 5F94461F
 P 7916 1612
+AR Path="/5F94461F" Ref="U8"  Part="1"
+AR Path="/5F8CFBC4/5F94461F" Ref="U8"  Part="1"
 F 0 "U8" H 7916 1927 50  0000 C CNN
 F 1 "IO_Switch" H 7916 1836 50  0000 C CNN
@@
 NoConn ~ 1302 3822
 $Comp
-L digitalSystemBoard:IO_Switch U9
+L digitalSystemBoard-rescue:IO_Switch-digitalSystemBoard U9
 U 1 1 5F948861
 P 1102 3972
+AR Path="/5F948861" Ref="U9"  Part="1"
+AR Path="/5F8CFBC4/5F948861" Ref="U9"  Part="1"
 F 0 "U9" H 1102 4287 50  0000 C CNN
 F 1 "IO_Switch" H 1102 4196 50  0000 C CNN
@@
 NoConn ~ 3546 3804
 $Comp
-L digitalSystemBoard:IO_Switch U10
+L digitalSystemBoard-rescue:IO_Switch-digitalSystemBoard U10
 U 1 1 5F94AB7C
 P 3346 3954
+AR Path="/5F94AB7C" Ref="U10"  Part="1"
+AR Path="/5F8CFBC4/5F94AB7C" Ref="U10"  Part="1"
 F 0 "U10" H 3346 4269 50  0000 C CNN
 F 1 "IO_Switch" H 3346 4178 50  0000 C CNN
@@
 NoConn ~ 5888 3772
 $Comp
-L digitalSystemBoard:IO_Switch U11
+L digitalSystemBoard-rescue:IO_Switch-digitalSystemBoard U11
 U 1 1 5F94C7D4
 P 5688 3922
+AR Path="/5F94C7D4" Ref="U11"  Part="1"
+AR Path="/5F8CFBC4/5F94C7D4" Ref="U11"  Part="1"
 F 0 "U11" H 5688 4237 50  0000 C CNN
 F 1 "IO_Switch" H 5688 4146 50  0000 C CNN
@@
 NoConn ~ 8034 3772
 $Comp
-L digitalSystemBoard:IO_Switch U12
+L digitalSystemBoard-rescue:IO_Switch-digitalSystemBoard U12
 U 1 1 5F950A04
 P 7834 3922
+AR Path="/5F950A04" Ref="U12"  Part="1"
+AR Path="/5F8CFBC4/5F950A04" Ref="U12"  Part="1"
 F 0 "U12" H 7834 4237 50  0000 C CNN
 F 1 "IO_Switch" H 7834 4146 50  0000 C CNN
@@
 NoConn ~ 1298 6066
 $Comp
-L digitalSystemBoard:IO_Switch U13
+L digitalSystemBoard-rescue:IO_Switch-digitalSystemBoard U13
 U 1 1 5F9542D3
 P 1098 6216
+AR Path="/5F9542D3" Ref="U13"  Part="1"
+AR Path="/5F8CFBC4/5F9542D3" Ref="U13"  Part="1"
 F 0 "U13" H 1098 6531 50  0000 C CNN
 F 1 "IO_Switch" H 1098 6440 50  0000 C CNN
@@
 NoConn ~ 3536 6046
 $Comp
-L digitalSystemBoard:IO_Switch U14
+L digitalSystemBoard-rescue:IO_Switch-digitalSystemBoard U14
 U 1 1 5F95718A
 P 3336 6196
+AR Path="/5F95718A" Ref="U14"  Part="1"
+AR Path="/5F8CFBC4/5F95718A" Ref="U14"  Part="1"
 F 0 "U14" H 3336 6511 50  0000 C CNN
 F 1 "IO_Switch" H 3336 6420 50  0000 C CNN

Commit message: Merge and delete clock block
Parts:
- removed D? (x9): LED, symbol Device:LED
- removed Q? (x9): 2N7002, Package_TO_SOT_SMD:SOT-23, symbol Transistor_FET:2N7002
- removed R? (x27): R, symbol Device:R
- added D10, D11, D2, D3, D5, D6, D7, D8, D9: LED, symbol Device:LED
- added Q10, Q11, Q3, Q4, Q5, Q6, Q7, Q8, Q9: 2N7002, Package_TO_SOT_SMD:SOT-23, symbol Transistor_FET:2N7002
- added R10, R13, R16, R19, R21, R23, R27, R31, R34: 10k, symbol Device:R
- added R11, R14, R17, R20, R24, R28, R29, R32, R35: 470, symbol Device:R
- added R12, R15, R18, R22, R25, R26, R30, R33, R9: 10, symbol Device:R
- R6: renamed from R?; value R -> 10
- R7: renamed from R?; value R -> 10k
- R8: renamed from R?; value R -> 470
- gave numbers to parts that had none: 2
Other:
- moved on the sheet: U6, U7

Commit message: Upload Timer Block
Connections:
- net labels removed: I1, I10, I2, I3, I4, I5, I6, I7, I8, I9
Changed lines of the file:
@@
 Wire Wire Line
 	3680 6346 3680 6486
-Text HLabel 1520 1880 3    50   Input ~ 0
-I1
 Text HLabel 1524 1452 1    50   Input ~ 0
 O1
-Text HLabel 6118 1866 3    50   Input ~ 0
-I3
 Text HLabel 6122 1438 1    50   Input ~ 0
 O3
-Text HLabel 8260 1902 3    50   Input ~ 0
-I4
 Text HLabel 8264 1474 1    50   Input ~ 0
 O4
-Text HLabel 1446 4262 3    50   Input ~ 0
-I5
 Text HLabel 1450 3834 1    50   Input ~ 0
 O5
-Text HLabel 3690 4244 3    50   Input ~ 0
-I6
 Text HLabel 3694 3816 1    50   Input ~ 0
 O6
-Text HLabel 6032 4212 3    50   Input ~ 0
-I7
 Text HLabel 6036 3784 1    50   Input ~ 0
 O7
-Text HLabel 8178 4212 3    50   Input ~ 0
-I8
 Text HLabel 8182 3784 1    50   Input ~ 0
 O8
-Text HLabel 1442 6506 3    50   Input ~ 0
-I9
 Text HLabel 1446 6078 1    50   Input ~ 0
 O9
-Text HLabel 3680 6486 3    50   Input ~ 0
-I10
 Text HLabel 3684 6058 1    50   Input ~ 0
 O10
@@
 Text HLabel 3484 1394 1    50   Input ~ 0
 O2
-Text HLabel 3480 1822 3    50   Input ~ 0
-I2
 NoConn ~ 3336 1382
 NoConn ~ 3086 1882
@@
 	1    0    0    -1
 $EndComp
+Text HLabel 1520 1880 3    50   Input ~ 0
+V_SOURCE
+Text HLabel 3480 1822 3    50   Input ~ 0
+V_SOURCE
+Text HLabel 6118 1866 3    50   Input ~ 0
+V_SOURCE
+Text HLabel 8260 1902 3    50   Input ~ 0
+V_SOURCE
+Text HLabel 1446 4262 3    50   Input ~ 0
+V_SOURCE
+Text HLabel 3690 4244 3    50   Input ~ 0
+V_SOURCE
+Text HLabel 6032 4212 3    50   Input ~ 0
+V_SOURCE
+Text HLabel 8178 4212 3    50   Input ~ 0
+V_SOURCE
+Text HLabel 1442 6506 3    50   Input ~ 0
+V_SOURCE
+Text HLabel 3680 6486 3    50   Input ~ 0
+V_SOURCE
 $EndSCHEMATC

Commit message: Redesign CLOCK_GENERATOR and add footprints for LM317, 5W resistor
Parts:
- U10, U11, U12, U13, U14, U5, U6, U7, U8, U9: footprint (none) -> digitalSystemBoard:SS-12F44G5
Connections:
- wire segments 90 -> 94
Other:
- note added: "SWITCH_INPUT"
- moved on the sheet: R25, R27
Changed lines of the file:
@@
 $Descr A4 11693 8268
 encoding utf-8
-Sheet 2 3
+Sheet 2 4
 Title ""
 Date ""
@@
 F 0 "U5" H 1176 1905 50  0000 C CNN
 F 1 "IO_Switch" H 1176 1814 50  0000 C CNN
-F 2 "" H 1176 1590 50  0001 C CNN
+F 2 "digitalSystemBoard:SS-12F44G5" H 1176 1590 50  0001 C CNN
 F 3 "" H 1176 1590 50  0001 C CNN
 	1    1176 1590
@@
 F 0 "U7" H 5774 1891 50  0000 C CNN
 F 1 "IO_Switch" H 5774 1800 50  0000 C CNN
-F 2 "" H 5774 1576 50  0001 C CNN
+F 2 "digitalSystemBoard:SS-12F44G5" H 5774 1576 50  0001 C CNN
 F 3 "" H 5774 1576 50  0001 C CNN
 	1    5774 1576
@@
 F 0 "U8" H 7916 1927 50  0000 C CNN
 F 1 "IO_Switch" H 7916 1836 50  0000 C CNN
-F 2 "" H 7916 1612 50  0001 C CNN
+F 2 "digitalSystemBoard:SS-12F44G5" H 7916 1612 50  0001 C CNN
 F 3 "" H 7916 1612 50  0001 C CNN
 	1    7916 1612
@@
 F 0 "U9" H 1102 4287 50  0000 C CNN
 F 1 "IO_Switch" H 1102 4196 50  0000 C CNN
-F 2 "" H 1102 3972 50  0001 C CNN
+F 2 "digitalSystemBoard:SS-12F44G5" H 1102 3972 50  0001 C CNN
 F 3 "" H 1102 3972 50  0001 C CNN
 	1    1102 3972
@@
 F 0 "U10" H 3346 4269 50  0000 C CNN
 F 1 "IO_Switch" H 3346 4178 50  0000 C CNN
-F 2 "" H 3346 3954 50  0001 C CNN
+F 2 "digitalSystemBoard:SS-12F44G5" H 3346 3954 50  0001 C CNN
 F 3 "" H 3346 3954 50  0001 C CNN
 	1    3346 3954
@@
 F 0 "U11" H 5688 4237 50  0000 C CNN
 F 1 "IO_Switch" H 5688 4146 50  0000 C CNN
-F 2 "" H 5688 3922 50  0001 C CNN
+F 2 "digitalSystemBoard:SS-12F44G5" H 5688 3922 50  0001 C CNN
 F 3 "" H 5688 3922 50  0001 C CNN
 	1    5688 3922
@@
 F 0 "U12" H 7834 4237 50  0000 C CNN
 F 1 "IO_Switch" H 7834 4146 50  0000 C CNN
-F 2 "" H 7834 3922 50  0001 C CNN
+F 2 "digitalSystemBoard:SS-12F44G5" H 7834 3922 50  0001 C CNN
 F 3 "" H 7834 3922 50  0001 C CNN
 	1    7834 3922
@@
 F 0 "U13" H 1098 6531 50  0000 C CNN
 F 1 "IO_Switch" H 1098 6440 50  0000 C CNN
-F 2 "" H 1098 6216 50  0001 C CNN
+F 2 "digitalSystemBoard:SS-12F44G5" H 1098 6216 50  0001 C CNN
 F 3 "" H 1098 6216 50  0001 C CNN
 	1    1098 6216
@@
 F 0 "U14" H 3336 6511 50  0000 C CNN
 F 1 "IO_Switch" H 3336 6420 50  0000 C CNN
-F 2 "" H 3336 6196 50  0001 C CNN
+F 2 "digitalSystemBoard:SS-12F44G5" H 3336 6196 50  0001 C CNN
 F 3 "" H 3336 6196 50  0001 C CNN
 	1    3336 6196
@@
 	3536 6196 3684 6196
 Wire Wire Line
-	3794 6196 3794 6186
-Wire Wire Line
 	3684 6196 3684 6058
-Connection ~ 3684 6196
-Wire Wire Line
-	3684 6196 3794 6196
 Wire Wire Line
 	3536 6346 3680 6346
@@
 Wire Wire Line
 	8674 1954 8974 1954
-Wire Wire Line
-	8976 1948 8976 1796
 $Comp
 L power:GND #PWR016
@@
 F 0 "U6" H 3136 1847 50  0000 C CNN
 F 1 "IO_Switch" H 3136 1756 50  0000 C CNN
-F 2 "" H 3136 1532 50  0001 C CNN
+F 2 "digitalSystemBoard:SS-12F44G5" H 3136 1532 50  0001 C CNN
 F 3 "" H 3136 1532 50  0001 C CNN
 	1    3136 1532
@@
 L Device:R R25
 U 1 1 5F9982BE
-P 3944 6186
-F 0 "R25" H 4014 6232 50  0000 L CNN
-F 1 "10" H 4014 6141 50  0000 L CNN
-F 2 "" V 3874 6186 50  0001 C CNN
-F 3 "~" H 3944 6186 50  0001 C CNN
-	1    3944 6186
+P 3896 6182
+F 0 "R25" H 3966 6228 50  0000 L CNN
+F 1 "10" H 3966 6137 50  0000 L CNN
+F 2 "" V 3826 6182 50  0001 C CNN
+F 3 "~" H 3896 6182 50  0001 C CNN
+	1    3896 6182
 	0    1    1    0
 $EndComp
@@
 L Device:R R27
 U 1 1 5F9982C8
-P 4094 6336
-F 0 "R27" H 4164 6382 50  0000 L CNN
-F 1 "10k" H 4164 6291 50  0000 L CNN
-F 2 "" V 4024 6336 50  0001 C CNN
-F 3 "~" H 4094 6336 50  0001 C CNN
-	1    4094 6336
-	1    0    0    -1
-$EndComp
-Wire Wire Line
-	4094 6486 4094 6538
-Wire Wire Line
-	4094 6538 4394 6538
-Wire Wire Line
-	4394 6538 4394 6386
+P 4068 6390
+F 0 "R27" H 4138 6436 50  0000 L CNN
+F 1 "10k" H 4138 6345 50  0000 L CNN
+F 2 "" V 3998 6390 50  0001 C CNN
+F 3 "~" H 4068 6390 50  0001 C CNN
+	1    4068 6390
+	1    0    0    -1
+$EndComp
 $Comp
 L power:GND #PWR011
@@
 	1    0    0    -1
 $EndComp
-Connection ~ 4394 6538
 Text HLabel 4394 5384 0    50   Input ~ 0
 V_SOURCE
@@
 Text HLabel 3680 6486 3    50   Input ~ 0
 V_SOURCE
+Wire Wire Line
+	4394 6538 4394 6384
+Wire Wire Line
+	8974 1954 8974 1802
+Connection ~ 8974 1954
+Wire Wire Line
+	4068 6540 4394 6540
+Wire Wire Line
+	4394 6540 4394 6538
+Connection ~ 4394 6538
+Wire Wire Line
+	4046 6182 4068 6182
+Wire Wire Line
+	4094 6182 4094 6184
+Wire Wire Line
+	4068 6240 4068 6182
+Connection ~ 4068 6182
+Wire Wire Line
+	4068 6182 4094 6182
+Wire Wire Line
+	3684 6196 3746 6196
+Wire Wire Line
+	3746 6196 3746 6182
+Connection ~ 3684 6196
+Text Notes 6116 5736 0    139  ~ 0
+SWITCH_INPUT
 $EndSCHEMATC

Commit message: Update a part of footprint
Parts:
- removed U10, U11, U12, U13, U14, U5, U6, U7, U8, U9: IO_Switch, digitalSystemBoard:SS-12F44G5, symbol digitalSystemBoard-rescue:IO_Switch-digitalSystemBoard
- added U10, U11, U12, U13, U14, U5, U6, U7, U8, U9: IO_Switch, digitalSystemBoard:SS-12F44G5, symbol digitalSystemBoard:IO_Switch
- D10, D11, D2, D3, D4, D5, D6, D7, D8, D9: footprint (none) -> LED_SMD:LED_0805_2012Metric
- R10, R11, R12, R13, R14, R15, R16, R17, R18, R19, R20, R21, R22, R23, R24, R25, R26, R27, R28, R29, R30, R31, R32, R33, R34, R35, R6, R7, R8, R9: footprint (none) -> Resistor_SMD:R_0603_1608Metric
Connections:
- net O1: now also U5.2
- net O10: now also U14.2
- net O2: now also U6.2
- net O3: now also U7.2
- net O4: now also U8.2
- net O5: now also U9.2
- net O6: now also U10.2
- net O7: now also U11.2
- net O8: now also U12.2
- net O9: now also U13.2
- net V_SOURCE: now also U10.3, U11.3, U12.3, U13.3, U14.3, U5.1, U6.3, U7.3, U8.3, U9.3

Commit message: Upload all footprint
Parts:
- Q10, Q11, Q2, Q3, Q4, Q5, Q6, Q7, Q8, Q9: footprint Package_TO_SOT_SMD:SOT-23 -> digitalSystemBoard:SO65P210X100-3N
Changed lines of the file:
@@
 F 0 "Q2" H 2338 1626 50  0000 L CNN
 F 1 "2N7002" H 2338 1535 50  0000 L CNN
-F 2 "Package_TO_SOT_SMD:SOT-23" H 2334 1505 50  0001 L CIN
+F 2 "digitalSystemBoard:SO65P210X100-3N" H 2334 1505 50  0001 L CIN
 F 3 "https://www.fairchildsemi.com/datasheets/2N/2N7002.pdf" H 2134 1580 50  0001 L CNN
 	1    2134 1580
@@
 F 0 "Q5" H 9078 1648 50  0000 L CNN
 F 1 "2N7002" H 9078 1557 50  0000 L CNN
-F 2 "Package_TO_SOT_SMD:SOT-23" H 9074 1527 50  0001 L CIN
+F 2 "digitalSystemBoard:SO65P210X100-3N" H 9074 1527 50  0001 L CIN
 F 3 "https://www.fairchildsemi.com/datasheets/2N/2N7002.pdf" H 8874 1602 50  0001 L CNN
 	1    8874 1602
@@
 F 0 "Q3" H 4298 1568 50  0000 L CNN
 F 1 "2N7002" H 4298 1477 50  0000 L CNN
-F 2 "Package_TO_SOT_SMD:SOT-23" H 4294 1447 50  0001 L CIN
+F 2 "digitalSystemBoard:SO65P210X100-3N" H 4294 1447 50  0001 L CIN
 F 3 "https://www.fairchildsemi.com/datasheets/2N/2N7002.pdf" H 4094 1522 50  0001 L CNN
 	1    4094 1522
@@
 F 0 "Q4" H 6936 1612 50  0000 L CNN
 F 1 "2N7002" H 6936 1521 50  0000 L CNN
-F 2 "Package_TO_SOT_SMD:SOT-23" H 6932 1491 50  0001 L CIN
+F 2 "digitalSystemBoard:SO65P210X100-3N" H 6932 1491 50  0001 L CIN
 F 3 "https://www.fairchildsemi.com/datasheets/2N/2N7002.pdf" H 6732 1566 50  0001 L CNN
 	1    6732 1566
@@
 F 0 "Q7" H 2264 4008 50  0000 L CNN
 F 1 "2N7002" H 2264 3917 50  0000 L CNN
-F 2 "Package_TO_SOT_SMD:SOT-23" H 2260 3887 50  0001 L CIN
+F 2 "digitalSystemBoard:SO65P210X100-3N" H 2260 3887 50  0001 L CIN
 F 3 "https://www.fairchildsemi.com/datasheets/2N/2N7002.pdf" H 2060 3962 50  0001 L CNN
 	1    2060 3962
@@
 F 0 "Q9" H 4508 3990 50  0000 L CNN
 F 1 "2N7002" H 4508 3899 50  0000 L CNN
-F 2 "Package_TO_SOT_SMD:SOT-23" H 4504 3869 50  0001 L CIN
+F 2 "digitalSystemBoard:SO65P210X100-3N" H 4504 3869 50  0001 L CIN
 F 3 "https://www.fairchildsemi.com/datasheets/2N/2N7002.pdf" H 4304 3944 50  0001 L CNN
 	1    4304 3944
@@
 F 0 "Q10" H 6850 3958 50  0000 L CNN
 F 1 "2N7002" H 6850 3867 50  0000 L CNN
-F 2 "Package_TO_SOT_SMD:SOT-23" H 6846 3837 50  0001 L CIN
+F 2 "digitalSystemBoard:SO65P210X100-3N" H 6846 3837 50  0001 L CIN
 F 3 "https://www.fairchildsemi.com/datasheets/2N/2N7002.pdf" H 6646 3912 50  0001 L CNN
 	1    6646 3912
@@
 F 0 "Q11" H 8996 3958 50  0000 L CNN
 F 1 "2N7002" H 8996 3867 50  0000 L CNN
-F 2 "Package_TO_SOT_SMD:SOT-23" H 8992 3837 50  0001 L CIN
+F 2 "digitalSystemBoard:SO65P210X100-3N" H 8992 3837 50  0001 L CIN
 F 3 "https://www.fairchildsemi.com/datasheets/2N/2N7002.pdf" H 8792 3912 50  0001 L CNN
 	1    8792 3912
@@
 F 0 "Q6" H 2260 6252 50  0000 L CNN
 F 1 "2N7002" H 2260 6161 50  0000 L CNN
-F 2 "Package_TO_SOT_SMD:SOT-23" H 2256 6131 50  0001 L CIN
+F 2 "digitalSystemBoard:SO65P210X100-3N" H 2256 6131 50  0001 L CIN
 F 3 "https://www.fairchildsemi.com/datasheets/2N/2N7002.pdf" H 2056 6206 50  0001 L CNN
 	1    2056 6206
@@
 F 0 "Q8" H 4498 6230 50  0000 L CNN
 F 1 "2N7002" H 4498 6139 50  0000 L CNN
-F 2 "Package_TO_SOT_SMD:SOT-23" H 4494 6109 50  0001 L CIN
+F 2 "digitalSystemBoard:SO65P210X100-3N" H 4494 6109 50  0001 L CIN
 F 3 "https://www.fairchildsemi.com/datasheets/2N/2N7002.pdf" H 4294 6184 50  0001 L CNN
 	1    4294 6184

Commit message: Change PCB
Parts:
- U10, U11, U12, U13, U14, U5, U6, U7, U8, U9: symbol digitalSystemBoard:IO_Switch -> digitalSystemBoard-rescue:IO_Switch-digitalSystemBoard
- renumbered D2 to D10, D6 to D11, D4 to D2, D5 to D3, D9 to D4, D11 to D5, D3 to D6, D10 to D9, Q6 to Q10, Q8 to Q11, Q7 to Q6, Q9 to Q7, Q10 to Q8, Q11 to Q9, R26 to R21, R21 to R22, R29 to R23, R30 to R24, R31 to R25, R32 to R26, R33 to R27, R34 to R28, R35 to R29, R22 to R30, R23 to R31, R24 to R32, R25 to R33, R27 to R34, R28 to R35
Connections:
- net V_SOURCE: now also U5.3; no longer U5.1

Commit message: Prepare for PCB
Parts:
- removed Q10, Q11, Q2, Q3, Q4, Q5, Q6, Q7, Q8, Q9: 2N7002, digitalSystemBoard:SO65P210X100-3N, symbol Transistor_FET:2N7002
- added Q10, Q11, Q2, Q3, Q4, Q5, Q6, Q7, Q8, Q9: BC847, digitalSystemBoard:SO65P210X100-3N, symbol Transistor_BJT:BC847
- R10, R13, R16, R19, R22, R25, R28, R31, R34, R7: value 10k -> 1k8
- R12, R15, R18, R21, R24, R27, R30, R33, R6, R9: value 10 -> 10k
Connections:
- net GND: now also Q10.2 (E), Q11.2 (E), Q2.2 (E), Q3.2 (E), Q4.2 (E), Q5.2 (E), Q6.2 (E), Q7.2 (E), Q8.2 (E), Q9.2 (E)
- net at R10.1, R9.1: now also Q3.1 (B)
- net at D3.1 (K): now also Q3.3 (C)
- net at R12.1, R13.1: now also Q4.1 (B)
- net at D4.1 (K): now also Q4.3 (C)
- net at R6.1, R7.1: now also Q2.1 (B)
- net at D2.1 (K): now also Q2.3 (C)
- net at R15.1, R16.1: now also Q5.1 (B)
- net at D5.1 (K): now also Q5.3 (C)
- net at R18.1, R19.1: now also Q6.1 (B)
- net at D6.1 (K): now also Q6.3 (C)
- net at R21.1, R22.1: now also Q7.1 (B)
- net at D7.1 (K): now also Q7.3 (C)
- net at R24.1, R25.1: now also Q8.1 (B)
- net at D8.1 (K): now also Q8.3 (C)
- net at R27.1, R28.1: now also Q9.1 (B)
- net at D9.1 (K): now also Q9.3 (C)
- net at R30.1, R31.1: now also Q10.1 (B)
- net at D10.1 (K): now also Q10.3 (C)
- net at R33.1, R34.1: now also Q11.1 (B)
- net at D11.1 (K): now also Q11.3 (C)
