File: digitalSystemBoard/OOI.sch (KiCad schematic (older format))
At the start: 60 parts, among them Q10 BC847, Q11 BC847, Q2 BC847, Q3 BC847, Q4 BC847, Q5 BC847, Q6 BC847, Q7 BC847, Q8 BC847, Q9 BC847, U10 IO_Switch, U11 IO_Switch, U12 IO_Switch, U13 IO_Switch, U14 IO_Switch, U5 IO_Switch, U6 IO_Switch, U7 IO_Switch, U8 IO_Switch, U9 IO_Switch

Commit message: Hot fix libs. Update schematic
Parts:
- U10, U11, U12, U13, U14, U5, U6, U7, U8, U9: symbol digitalSystemBoard-rescue:IO_Switch-digitalSystemBoard -> digitalSystemBoard:IO_Switch
Changed lines of the file:
@@
 SWITCH_INPUT
 $Comp
-L digitalSystemBoard-rescue:IO_Switch-digitalSystemBoard U6
+L digitalSystemBoard:IO_Switch U6
 U 1 1 5FA7DE48
 P 3136 1532
@@
 $EndComp
 $Comp
-L digitalSystemBoard-rescue:IO_Switch-digitalSystemBoard U7
+L digitalSystemBoard:IO_Switch U7
 U 1 1 5FA83231
 P 5774 1576
@@
 $EndComp
 $Comp
-L digitalSystemBoard-rescue:IO_Switch-digitalSystemBoard U8
+L digitalSystemBoard:IO_Switch U8
 U 1 1 5FA84041
 P 7916 1612
@@
 $EndComp
 $Comp
-L digitalSystemBoard-rescue:IO_Switch-digitalSystemBoard U9
+L digitalSystemBoard:IO_Switch U9
 U 1 1 5FA84F0E
 P 1102 3972
@@
 $EndComp
 $Comp
-L digitalSystemBoard-rescue:IO_Switch-digitalSystemBoard U10
+L digitalSystemBoard:IO_Switch U10
 U 1 1 5FA8ABC8
 P 3346 3954
@@
 $EndComp
 $Comp
-L digitalSystemBoard-rescue:IO_Switch-digitalSystemBoard U11
+L digitalSystemBoard:IO_Switch U11
 U 1 1 5FA8BBA6
 P 5688 3922
@@
 $EndComp
 $Comp
-L digitalSystemBoard-rescue:IO_Switch-digitalSystemBoard U12
+L digitalSystemBoard:IO_Switch U12
 U 1 1 5FA8D4ED
 P 7834 3922
@@
 $EndComp
 $Comp
-L digitalSystemBoard-rescue:IO_Switch-digitalSystemBoard U13
+L digitalSystemBoard:IO_Switch U13
 U 1 1 5FA8E32F
 P 1098 6216
@@
 $EndComp
 $Comp
-L digitalSystemBoard-rescue:IO_Switch-digitalSystemBoard U14
+L digitalSystemBoard:IO_Switch U14
 U 1 1 5FA8F0FB
 P 3336 6196
@@
 $EndComp
 $Comp
-L digitalSystemBoard-rescue:IO_Switch-digitalSystemBoard U5
+L digitalSystemBoard:IO_Switch U5
 U 1 1 5FA7D407
 P 1176 1590
