File: digitalSystemBoard/CLOCK_GENERATOR.sch (KiCad schematic (older format))
At the start: 31 parts, among them J12 USB_OTG, SW4 ButtonFirst, SW5 ButtonFirst, SW6 ButtonFirst, SW7 ButtonFirst, U17 Potentiometer-digitalSystemBo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, U18 ICSP, U19 ATmega32U2-AU, Y1 16MHz

Commit message: Update a part of footprint
Parts:
- removed J12: USB_OTG, symbol digitalSystemBoard-rescue:USB_OTG-project
- removed U19: ATmega32U2-AU, Package_QFP:TQFP-32_7x7mm_P0.8mm, symbol MCU_Microchip_ATmega:ATmega32U2-AU
- added C12: 0.1uF, Capacitor_SMD:C_0603_1608Metric, symbol Device:C
- added FB5, FB6: 80Ohm, footprints:FerriteBead, symbol Device:Ferrite_Bead_Small
- added J12: USB_OTG, digitalSystemBoard:SAMTEC_USB-B-S-X-X-TH-TR, symbol digitalSystemBoard:USB-B-S-X-X-TH-TR
- added U3: ATmega32U4-AU, Package_QFP:TQFP-44_10x10mm_P0.8mm, symbol MCU_Microchip_ATmega:ATmega32U4-AU
- C10, C11, C5, C6, C7, C8, C9: footprint (none) -> Capacitor_SMD:C_0603_1608Metric
- D22: footprint SC70-6 -> footprints:SC70-6
- FB1, FB2, FB3, FB4: footprint (none) -> footprints:FerriteBead
- R66, R67, R68, R69, R70, R71, R72, R73, R74: footprint (none) -> Resistor_SMD:R_0603_1608Metric
- SW4, SW5, SW6, SW7: footprint TE_4-1437565-9 -> digitalSystemBoard:Button
- U17: footprint digitalSystemBoard:RV09S -> digitalSystemBoard:TRIM_3296W-1-501
- Y1: footprint (none) -> Crystal:Crystal_SMD_5032-4Pin_5.0x3.2mm
Connections:
- wire segments 74 -> 81
- no-connect marks 15 -> 19
Other:
- moved on the sheet: C10, C11, C5, C6, C7, C8, C9, D22, FB1, FB2, FB3, FB4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

Commit message: Upload schematic full agan
Parts:
- U17: footprint digitalSystemBoard:TRIM_3296W-1-501 -> digitalSystemBoard:RK09D117000B
Changed lines of the file:
@@
 F 0 "U17" V 2459 7116 50  0000 L CNN
 F 1 "Potentiometer-digitalSystemBoard" V 2790 6334 50  0000 L CNN
-F 2 "digitalSystemBoard:TRIM_3296W-1-501" H 2438 6988 50  0001 C CNN
+F 2 "digitalSystemBoard:RK09D117000B" H 2438 6988 50  0001 C CNN
 F 3 "" H 2438 6988 50  0001 C CNN
 	1    2438 6988

Commit message: Change PCB
Parts:
- J12: symbol digitalSystemBoard:USB-B-S-X-X-TH-TR -> digitalSystemBoard-rescue:USB-B-S-X-X-TH-TR-digitalSystemBoard
Changed lines of the file:
@@
 	1670 1806 1670 1912
 $Comp
-L digitalSystemBoard:USB-B-S-X-X-TH-TR J12
+L digitalSystemBoard-rescue:USB-B-S-X-X-TH-TR-digitalSystemBoard J12
 U 1 1 5F99974B
 P 1270 1406

Commit message: Add usb source block
Parts:
- added C13: 22nF, Capacitor_SMD:C_0603_1608Metric, symbol Device:C
- added C14, C16: 1uF, Capacitor_SMD:C_0603_1608Metric, symbol Device:C
- added C15: 0.1uF, Capacitor_SMD:C_0603_1608Metric, symbol Device:C
- added D23: LED, LED_SMD:LED_0805_2012Metric, symbol Device:LED
- added Q22: Q_PMOS_GSD, digitalSystemBoard:P_SOURCE, symbol Device:Q_PMOS_GSD
- added R75, R76: 10k, Resistor_SMD:R_0603_1608Metric, symbol Device:R
- added R77: 220, Resistor_SMD:R_0603_1608Metric, symbol Device:R
- added U19: LP2985-3.3, digitalSystemBoard:LP2985, symbol project:LP2985-3.3
- added U4: LMV358IDGKR, digitalSystemBoard:LM358, symbol digitalSystemBoard:LMV358IDGKR
Connections:
- net +5V: now also C14.1, C15.2, Q22.2 (S), U19.1 (VIN), U19.3 (ON/~OFF~), U4.8 (VCC+)
- net D2: now also U3.22 (PD5); no longer U3.32 (PC7)
- net GND: now also C13.2, C14.2, C15.1, C16.2, D23.1 (K), R76.2, U19.2 (GND), U4.4 (GND)
- net VBUS: now also Q22.3 (D)
- new net: Q22.1 (G), U4.1
- new net: C13.1, R75.2, R76.1, U4.3
- new net: R77.1, U4.6, U4.7
- new net: D23.2 (A), R77.2
- new net +3V3: C16.1, U19.5 (VOUT), U4.2
- new net PC7: U3.32 (PC7), U4.5
- new net VIN: R75.1
