File: digitalSystemBoard/CLOCK_GENERATOR.sch (KiCad schematic (older format))
At the start: 34 parts, among them J12 USB_OTG, SW4 ButtonFirst, SW5 ButtonFirst, SW6 ButtonFirst, SW7 ButtonFirst, U17 Potentiometer-digitalSystemBo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, U18 ICSP, U3 ATmega32U4-AU, Y1 16MHz

Commit message: Update board layout
Parts:
- SW5, SW6, SW7: footprint digitalSystemBoard:Button -> digitalSystemBoard:Button_CLOCK
Changed lines of the file:
@@
 F 0 "SW7" H 5348 7359 50  0000 C CNN
 F 1 "ButtonFirst" H 5348 7268 50  0000 C CNN
-F 2 "digitalSystemBoard:Button" H 5348 7044 50  0001 L BNN
+F 2 "digitalSystemBoard:Button_CLOCK" H 5348 7044 50  0001 L BNN
 F 3 "4-1437565-9" H 5348 7044 50  0001 L BNN
 F 4 "50 mA" H 5348 7044 50  0001 L BNN "Field4"
@@
 F 0 "SW5" H 2442 6197 50  0000 C CNN
 F 1 "ButtonFirst" H 2442 6106 50  0000 C CNN
-F 2 "digitalSystemBoard:Button" H 2442 5882 50  0001 L BNN
+F 2 "digitalSystemBoard:Button_CLOCK" H 2442 5882 50  0001 L BNN
 F 3 "4-1437565-9" H 2442 5882 50  0001 L BNN
 F 4 "50 mA" H 2442 5882 50  0001 L BNN "Field4"
@@
 F 0 "SW6" H 5352 6187 50  0000 C CNN
 F 1 "ButtonFirst" H 5352 6096 50  0000 C CNN
-F 2 "digitalSystemBoard:Button" H 5352 5872 50  0001 L BNN
+F 2 "digitalSystemBoard:Button_CLOCK" H 5352 5872 50  0001 L BNN
 F 3 "4-1437565-9" H 5352 5872 50  0001 L BNN
 F 4 "50 mA" H 5352 5872 50  0001 L BNN "Field4"
