File: digitalSystemBoard/CLOCK_GENERATOR.sch (KiCad schematic (older format))
At the start: 45 parts, among them J12 USB_OTG, Q22 Q_PMOS_GSD, SW4 ButtonFirst, SW5 ButtonFirst, SW6 ButtonFirst, SW7 ButtonFirst, U17 Potentiometer-digitalSystemBo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, U18 ICSP, U19 LP2985-3.3, U3 ATmega32U4-AU, U4 LMV358IDGKR, Y1 16MHz

Commit message: Update I/O and MCU schematic
Parts:
- added IN_1, IN_2: 74LS165, symbol 74xx:74LS165
- added OUT_1, OUT_2: 74HC164, symbol 74xx:74HC164
Connections:
- net +5V: now also IN_1.16 (VCC), IN_2.16 (VCC), OUT_1.14 (VCC), OUT_1.2 (DSB), OUT_2.14 (VCC), OUT_2.2 (DSB)
- net D1: now also OUT_2.6 (Q3)
- net D2: now also OUT_2.13 (Q7)
- net GND: now also IN_1.10 (DS), IN_1.15 (~CE), IN_1.8 (GND), IN_2.15 (~CE), IN_2.8 (GND), OUT_1.7 (GND), OUT_2.7 (GND)
- net OUT_ctrl: now reaches U3.1 (PE6)
- net OUT_ctrl: now also OUT_1.9 (~MR), OUT_2.9 (~MR)
- net IN_data: now reaches U3.12 (PB7)
- net IN_data: now also IN_2.9 (Q7)
- net IN_ctrl: now reaches U3.18 (PD0)
- net IN_ctrl: now also IN_1.1 (~PL), IN_2.1 (~PL)
- net OUT_clk: now reaches U3.25 (PD4)
- net OUT_clk: now also OUT_1.8 (CP), OUT_2.8 (CP)
- net OUT_data: now reaches U3.26 (PD6)
- net OUT_data: now also OUT_1.1 (DSA)
- net IN_clk: now reaches U3.8 (PB0)
- net IN_clk: now also IN_1.2 (CP), IN_2.2 (CP)
- new net A1: OUT_2.3 (Q0)
- new net A2: OUT_2.10 (Q4)
- new net B1: OUT_2.4 (Q1)
- new net B2: OUT_2.11 (Q5)
- new net C1: OUT_2.5 (Q2)
- new net C2: OUT_2.12 (Q6)
- new net OA1: IN_2.11 (D0)
- new net OA2: IN_2.3 (D4)
- new net OB1: IN_2.12 (D1)
- new net OB2: IN_2.4 (D5)
- new net OC1: IN_2.13 (D2)
- new net OC2: IN_2.5 (D6)
- new net OD1: IN_2.14 (D3)
- new net OD2: IN_2.6 (D7)
- new net OELD6: OUT_1.12 (Q6)
- new net OLED0: OUT_1.3 (Q0)
- new net OLED1: OUT_1.4 (Q1)
- new net OLED2: OUT_1.5 (Q2)
- new net OLED3: OUT_1.6 (Q3)
- new net OLED4: OUT_1.10 (Q4)
- new net OLED5: OUT_1.11 (Q5)
- new net OLED7: OUT_1.13 (Q7), OUT_2.1 (DSA)
- new net S_TO: IN_1.9 (Q7), IN_2.10 (DS)
- new net TLED0: IN_1.11 (D0)
- new net TLED1: IN_1.12 (D1)
- new net TLED2: IN_1.13 (D2)
- new net TLED3: IN_1.14 (D3)
- new net TLED4: IN_1.3 (D4)
- new net TLED5: IN_1.4 (D5)
- new net TLED6: IN_1.5 (D6)
- new net TLED7: IN_1.6 (D7)
- no-connect marks 19 -> 15
Other:
- moved on the sheet: C10, C11, C12, C13, C14, C15, C16, C5, C6, C7, C8, C9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

Commit message: Update I/O schematic, Complete layout, Start routing
Parts:
- added U20: 74HC04, symbol 74xx:74HC04
- IN_1, IN_2: footprint (none) -> Package_SO:SOIC-16_3.9x9.9mm_P1.27mm
- OUT_1, OUT_2: footprint (none) -> Package_SO:SOIC-14_3.9x8.7mm_P1.27mm
Connections:
- net CHANGE_CLK_SRC: now also U20.8; no longer R73.2, SW7.1
- net DOWN_CLK: now also U20.6; no longer R72.2, SW6.1
- net UP_CLK: now also U20.4; no longer R71.2, SW5.1
- new net: R72.2, SW6.1, U20.5
- new net: R71.2, SW5.1, U20.3
- new net: R73.2, SW7.1, U20.9
Other:
- moved on the sheet: R71, R72, R73, SW5, SW6, SW7, U17

Commit message: Hot fix schematics. Update MCU layout
Parts:
- U20: footprint (none) -> Package_SO:SOIC-14_3.9x8.7mm_P1.27mm
Connections:
- net +5V: now also U17.3; no longer U17.1
- net D1: no longer DS1.8 (D1), U3.31 (PC6)
- net D2: no longer DS1.9 (D2), U3.22 (PD5)
- net GND: now also U17.1
- net IN_clk: now also OUT_1.8 (CP), OUT_2.8 (CP), U3.31 (PC6); no longer U3.8 (PB0)
- net OUT_ctrl: now also U3.25 (PD4); no longer U3.1 (PE6)
- net D0 renamed I0
- net I0: now also U3.8 (PB0); no longer U3.30 (PB6)
- net D3 renamed I3
- net D4 renamed I4
- net D5 renamed I5
- net D6 renamed I6
- net D7 renamed I7
- removed net OUT_clk: OUT_1.8 (CP), OUT_2.8 (CP), U3.25 (PD4)
- new net I1: DS1.8 (D1), U3.30 (PB6)
- new net I2: DS1.9 (D2), U3.22 (PD5)
Other:
- moved on the sheet: U17
Changed lines of the file:
@@
 L digitalSystemBoard-rescue:Potentiometer-digitalSystemBoard U17
 U 1 1 5F9A7CE1
-P 1382 7140
-F 0 "U17" V 1403 7268 50  0000 L CNN
-F 1 "Potentiometer-digitalSystemBoard" V 1734 6486 50  0000 L CNN
-F 2 "digitalSystemBoard:RK09D117000B" H 1382 7140 50  0001 C CNN
-F 3 "" H 1382 7140 50  0001 C CNN
-	1    1382 7140
-	0    1    1    0
-$EndComp
-NoConn ~ 1382 7390
+P 830 7082
+F 0 "U17" V 851 7210 50  0000 L CNN
+F 1 "Potentiometer-digitalSystemBoard" V 258 6102 50  0000 L CNN
+F 2 "digitalSystemBoard:RK09D117000B" H 830 7082 50  0001 C CNN
+F 3 "" H 830 7082 50  0001 C CNN
+	1    830  7082
+	0    -1   -1   0
+$EndComp
 $Comp
 L power:+5V #PWR0124
 U 1 1 5F9C1892
-P 1382 6784
-F 0 "#PWR0124" H 1382 6634 50  0001 C CNN
-F 1 "+5V" H 1397 6957 50  0000 C CNN
-F 2 "" H 1382 6784 50  0001 C CNN
-F 3 "" H 1382 6784 50  0001 C CNN
-	1    1382 6784
-	1    0    0    -1
-$EndComp
-Text Label 1032 7090 2    50   ~ 0
+P 830 6776
+F 0 "#PWR0124" H 830 6626 50  0001 C CNN
+F 1 "+5V" H 845 6949 50  0000 C CNN
+F 2 "" H 830 6776 50  0001 C CNN
+F 3 "" H 830 6776 50  0001 C CNN
+	1    830  6776
+	1    0    0    -1
+$EndComp
+Text Label 1180 7132 0    50   ~ 0
 CLOCK_WHEEL
 Text Label 3628 6664 2    50   ~ 0
@@
 	9410 1294 9628 1294
 Text Label 9628 1694 2    50   ~ 0
-D0
+I0
 Text Label 9628 1794 2    50   ~ 0
-D1
+I1
 Text Label 9628 1894 2    50   ~ 0
-D2
+I2
 $Comp
 L Display_Character:WC1602A DS?
@@
 $EndComp
 Text Label 9628 1994 2    50   ~ 0
-D3
+I3
 Text Label 9628 2094 2    50   ~ 0
-D4
+I4
 Text Label 9628 2194 2    50   ~ 0
-D5
+I5
 Text Label 9628 2294 2    50   ~ 0
-D6
+I6
 Text Label 9628 2394 2    50   ~ 0
-D7
+I7
 Text Notes 3096 6006 0    100  ~ 0
 MCU_BLOCK\n
@@
 Connection ~ 3812 2284
 Text Label 4406 2884 3    50   ~ 0
-D7
-Text Label 4506 2884 3    50   ~ 0
-D6
+I7
 Text Label 4606 2884 3    50   ~ 0
-D5
+I5
 Text Label 4706 2884 3    50   ~ 0
-D4
+I4
 Text Label 4806 2884 3    50   ~ 0
-D3
+I3
 Text Label 5506 2884 3    50   ~ 0
-D2
-Text Label 6306 2884 3    50   ~ 0
-D1
+I2
 Text Label 6606 2884 3    50   ~ 0
-D0
+I1
+Text Label 7206 2884 3    50   ~ 0
+I0
 Text Label 5306 2884 3    50   ~ 0
 RS
@@
 Text Label 4868 5612 3    50   ~ 0
 IN_data
-Text Label 7206 2884 3    50   ~ 0
+Text Label 6194 3312 3    50   ~ 0
 IN_clk
 Text Label 1238 4616 1    50   ~ 0
@@
 	5168 5112 5168 5090
 NoConn ~ 4768 5612
-Text Label 5606 2884 3    50   ~ 0
+Text Label 6390 3312 3    50   ~ 0
 OUT_clk
 Text Label 5406 2884 3    50   ~ 0
 OUT_data
-Text Label 5006 2884 3    50   ~ 0
+Text Label 5606 2884 3    50   ~ 0
 OUT_ctrl
 Wire Wire Line
@@
 	2676 6816 2676 6774
 Wire Wire Line
-	1382 6784 1382 6840
+	830  6776 830  6832
 $Comp
 L Device:Ferrite_Bead_Small FB?
@@
 F 0 "U20" H 3972 6821 50  0000 C CNN
 F 1 "74HC04" H 3972 6912 50  0000 C CNN
-F 2 "" H 3972 7138 50  0001 C CNN
+F 2 "Package_SO:SOIC-14_3.9x8.7mm_P1.27mm" H 3972 7138 50  0001 C CNN
 F 3 "https://assets.nexperia.com/documents/data-sheet/74HC_HCT04.pdf" H 3972 7138 50  0001 C CNN
 	2    3972 7138
@@
 F 0 "U20" H 5728 6801 50  0000 C CNN
 F 1 "74HC04" H 5728 6892 50  0000 C CNN
-F 2 "" H 5728 7118 50  0001 C CNN
+F 2 "Package_SO:SOIC-14_3.9x8.7mm_P1.27mm" H 5728 7118 50  0001 C CNN
 F 3 "https://assets.nexperia.com/documents/data-sheet/74HC_HCT04.pdf" H 5728 7118 50  0001 C CNN
 	3    5728 7118
@@
 F 0 "U20" H 2182 6821 50  0000 C CNN
 F 1 "74HC04" H 2182 6912 50  0000 C CNN
-F 2 "" H 2182 7138 50  0001 C CNN
+F 2 "Package_SO:SOIC-14_3.9x8.7mm_P1.27mm" H 2182 7138 50  0001 C CNN
 F 3 "https://assets.nexperia.com/documents/data-sheet/74HC_HCT04.pdf" H 2182 7138 50  0001 C CNN
 	4    2182 7138
 	-1   0    0    1
 $EndComp
+Text Label 4506 2884 3    50   ~ 0
+I6
+NoConn ~ 5006 2884
+Wire Wire Line
+	6306 2884 6306 3312
+Wire Wire Line
+	6306 3312 6390 3312
+Wire Wire Line
+	6306 3312 6194 3312
+Connection ~ 6306 3312
+$Comp
+L power:GND #PWR0155
+U 1 1 5F976784
+P 830 7382
+F 0 "#PWR0155" H 830 7132 50  0001 C CNN
+F 1 "GND" H 835 7209 50  0000 C CNN
+F 2 "" H 830 7382 50  0001 C CNN
+F 3 "" H 830 7382 50  0001 C CNN
+	1    830  7382
+	1    0    0    -1
+$EndComp
 $EndSCHEMATC

Commit message: Update new layout, add power vias
Parts:
- U4: footprint digitalSystemBoard:LM358 -> Package_SO:VSSOP-8_3.0x3.0mm_P0.65mm
Changed lines of the file:
@@
 F 0 "U4" H 1854 3921 50  0000 C CNN
 F 1 "LMV358IDGKR" H 1854 3830 50  0000 C CNN
-F 2 "digitalSystemBoard:LM358" H 1854 3354 50  0001 L BNN
+F 2 "Package_SO:VSSOP-8_3.0x3.0mm_P0.65mm" H 1854 3354 50  0001 L BNN
 F 3 "1.1mm" H 1854 3354 50  0001 L BNN
 F 4 "Texas Instruments" H 1854 3354 50  0001 L BNN "Field4"

Commit message: Hot fix libs. Update schematic
Parts:
- D22: symbol digitalSystemBoard-rescue:SMF05C.TCT-project -> digitalSystemBoard:SMF05C.TCT
- J12: symbol digitalSystemBoard-rescue:USB-B-S-X-X-TH-TR-digitalSystemBoard -> digitalSystemBoard:USB-B-S-X-X-TH-TR
- SW4, SW5, SW6, SW7: symbol digitalSystemBoard-rescue:ButtonFirst-project -> digitalSystemBoard:ButtonFirst
- U17: symbol digitalSystemBoard-rescue:Potentiometer-digitalSystemBoard -> digitalSystemBoard:Potentiometer
- U18: symbol digitalSystemBoard-rescue:ICSP -> digitalSystemBoard:ICSP
- U19: symbol digitalSystemBoard-rescue:LP2985-3.3-project -> digitalSystemBoard:LP2985-3.3
- U4: symbol digitalSystemBoard-rescue:LMV358IDGKR-digitalSystemBoard -> digitalSystemBoard:LMV358IDGKR
- Y1: symbol digitalSystemBoard-rescue:Resonator-project -> digitalSystemBoard:Resonator
Changed lines of the file:
@@
 D+
 $Comp
-L digitalSystemBoard-rescue:ICSP U18
+L digitalSystemBoard:ICSP U18
 U 1 1 5F97639D
 P 10042 3574
+AR Path="/5F97639D" Ref="U18"  Part="1"
+AR Path="/5F94C37C/5F97639D" Ref="U18"  Part="1"
 F 0 "U18" H 10570 3562 50  0000 L CNN
 F 1 "ICSP" H 10570 3471 50  0000 L CNN
@@
 SCK
 $Comp
-L digitalSystemBoard-rescue:Potentiometer-digitalSystemBoard U17
+L digitalSystemBoard:Potentiometer U17
 U 1 1 5F9A7CE1
 P 830 7082
+AR Path="/5F9A7CE1" Ref="U17"  Part="1"
+AR Path="/5F94C37C/5F9A7CE1" Ref="U17"  Part="1"
 F 0 "U17" V 851 7210 50  0000 L CNN
 F 1 "Potentiometer-digitalSystemBoard" V 258 6102 50  0000 L CNN
@@
 UP_CLK
 $Comp
-L digitalSystemBoard-rescue:ButtonFirst-project SW?
+L digitalSystemBoard:ButtonFirst SW?
 U 1 1 5F9A548F
 P 3062 7238
@@
 	2812 7138 2676 7138
 $Comp
-L digitalSystemBoard-rescue:ButtonFirst-project SW?
+L digitalSystemBoard:ButtonFirst SW?
 U 1 1 5F964111
 P 4754 7238
@@
 NoConn ~ 1642 1356
 $Comp
-L digitalSystemBoard-rescue:SMF05C.TCT-project D?
+L digitalSystemBoard:SMF05C.TCT D?
 U 1 1 5F96412B
 P 1942 1456
@@
 Connection ~ 7400 1598
 $Comp
-L digitalSystemBoard-rescue:ButtonFirst-project SW?
+L digitalSystemBoard:ButtonFirst SW?
 U 1 1 5F964203
 P 7772 1698
@@
 Connection ~ 7048 1312
 $Comp
-L digitalSystemBoard-rescue:Resonator-project Y?
+L digitalSystemBoard:Resonator Y?
 U 1 1 5F964216
 P 6890 1312
@@
 $EndComp
 $Comp
-L digitalSystemBoard-rescue:LP2985-3.3-project U19
+L digitalSystemBoard:LP2985-3.3 U19
 U 1 1 5F9193C2
 P 4138 1088
+AR Path="/5F9193C2" Ref="U19"  Part="1"
+AR Path="/5F94C37C/5F9193C2" Ref="U19"  Part="1"
 F 0 "U19" H 4138 1430 50  0000 C CNN
 F 1 "LP2985-3.3" H 4138 1339 50  0000 C CNN
@@
 $EndComp
 $Comp
-L digitalSystemBoard-rescue:LMV358IDGKR-digitalSystemBoard U4
+L digitalSystemBoard:LMV358IDGKR U4
 U 1 1 5F9D48CE
 P 1854 3354
@@
 DOWN_CLK
 $Comp
-L digitalSystemBoard-rescue:ButtonFirst-project SW?
+L digitalSystemBoard:ButtonFirst SW?
 U 1 1 5F9640EF
 P 6504 7218
@@
 $EndComp
 $Comp
-L digitalSystemBoard-rescue:USB-B-S-X-X-TH-TR-digitalSystemBoard J12
+L digitalSystemBoard:USB-B-S-X-X-TH-TR J12
 U 1 1 5F99974B
 P 852 1128
+AR Path="/5F99974B" Ref="J12"  Part="1"
+AR Path="/5F94C37C/5F99974B" Ref="J12"  Part="1"
 F 0 "J12" H 745 561 50  0000 C CNN
 F 1 "USB_OTG" H 745 652 50  0000 C CNN
