File: digitalSystemBoard/OUT_PIN.sch (KiCad schematic (older format))
At the start: 50 parts

Commit message: Complete Output Block
Connections:
- net labels added: OLED1, OLED10, OLED2, OLED3, OLED4, OLED5, OLED6, OLED7, OLED8, OLED9

Commit message: Merge and delete clock block
Parts:
- removed D? (x9): LED, symbol Device:LED
- removed Q? (x9): 2N7002, Package_TO_SOT_SMD:SOT-23, symbol Transistor_FET:2N7002
- removed R? (x27): R, symbol Device:R
- added D12, D14, D15, D16, D17, D18, D19, D20, D21: LED, symbol Device:LED
- added Q12, Q14, Q15, Q16, Q17, Q18, Q19, Q20, Q21: 2N7002, Package_TO_SOT_SMD:SOT-23, symbol Transistor_FET:2N7002
- added R36, R42, R43, R48, R49, R54, R55, R60, R61: 10, symbol Device:R
- added R38, R44, R45, R50, R51, R56, R57, R62, R63: 10k, symbol Device:R
- added R40, R46, R47, R52, R53, R58, R59, R64, R65: 330, symbol Device:R
- R37: renamed from R?; value R -> 10
- R39: renamed from R?; value R -> 10k
- R41: renamed from R?; value R -> 330
- gave numbers to parts that had none: 2
Connections:
- net GND: now also Q12.2 (S), Q14.2 (S), Q15.2 (S), Q16.2 (S), Q17.2 (S), Q18.2 (S), Q19.2 (S), Q20.2 (S), Q21.2 (S), R38.2, R44.2, R45.2, R50.2, R51.2, R56.2, R57.2, R62.2, R63.2
- net OLED10: now also R61.2
- net OLED2: now also R43.2
- net OLED3: now also R49.2
- net OLED4: now also R55.2
- net OLED5: now also R60.2
- net OLED6: now also R36.2
- net OLED7: now also R42.2
- net OLED8: now also R48.2
- net OLED9: now also R54.2
- net V_SOURCE: now also R40.1, R46.1, R47.1, R52.1, R53.1, R58.1, R59.1, R64.1, R65.1
- new net: Q15.1 (G), R43.1, R45.1
- new net: D15.1 (K), Q15.3 (D)
- new net: D15.2 (A), R47.2
- new net: Q17.1 (G), R49.1, R51.1
- new net: D17.1 (K), Q17.3 (D)
- new net: D17.2 (A), R53.2
- new net: Q19.1 (G), R55.1, R57.1
- new net: D19.1 (K), Q19.3 (D)
- new net: D19.2 (A), R59.2
- new net: Q20.1 (G), R60.1, R62.1
- new net: D20.1 (K), Q20.3 (D)
- new net: D20.2 (A), R64.2
- new net: Q12.1 (G), R36.1, R38.1
- new net: D12.1 (K), Q12.3 (D)
- new net: D12.2 (A), R40.2
- new net: Q14.1 (G), R42.1, R44.1
- new net: D14.1 (K), Q14.3 (D)
- new net: D14.2 (A), R46.2
- new net: Q16.1 (G), R48.1, R50.1
- new net: D16.1 (K), Q16.3 (D)
- new net: D16.2 (A), R52.2
- new net: Q18.1 (G), R54.1, R56.1
- new net: D18.1 (K), Q18.3 (D)
- new net: D18.2 (A), R58.2
- new net: Q21.1 (G), R61.1, R63.1
- new net: D21.1 (K), Q21.3 (D)
- new net: D21.2 (A), R65.2

Commit message: Redesign CLOCK_GENERATOR and add footprints for LM317, 5W resistor
Other:
- note added: "LED_DISPLAY\n"
Changed lines of the file:
@@
 $Descr A4 11693 8268
 encoding utf-8
-Sheet 3 3
+Sheet 3 4
 Title ""
 Date ""
@@
 Text HLabel 9110 3142 0    50   Input ~ 0
 V_SOURCE
+Text Notes 4842 5480 0    139  ~ 0
+LED_DISPLAY\n
 $EndSCHEMATC

Commit message: Update a part of footprint
Parts:
- D12, D13, D14, D15, D16, D17, D18, D19, D20, D21: footprint (none) -> digitalSystemBoard:LED_3528
- R36, R37, R38, R39, R40, R41, R42, R43, R44, R45, R46, R47, R48, R49, R50, R51, R52, R53, R54, R55, R56, R57, R58, R59, R60, R61, R62, R63, R64, R65: footprint (none) -> Resistor_SMD:R_0603_1608Metric
Changed lines of the file:
@@
 F 0 "R37" H 1866 1668 50  0000 L CNN
 F 1 "10" H 1866 1577 50  0000 L CNN
-F 2 "" V 1726 1622 50  0001 C CNN
+F 2 "Resistor_SMD:R_0603_1608Metric" V 1726 1622 50  0001 C CNN
 F 3 "~" H 1796 1622 50  0001 C CNN
 	1    1796 1622
@@
 F 0 "R39" H 2016 1818 50  0000 L CNN
 F 1 "10k" H 2016 1727 50  0000 L CNN
-F 2 "" V 1876 1772 50  0001 C CNN
+F 2 "Resistor_SMD:R_0603_1608Metric" V 1876 1772 50  0001 C CNN
 F 3 "~" H 1946 1772 50  0001 C CNN
 	1    1946 1772
@@
 F 0 "R41" H 2316 1018 50  0000 L CNN
 F 1 "330" H 2316 927 50  0000 L CNN
-F 2 "" V 2176 972 50  0001 C CNN
+F 2 "Resistor_SMD:R_0603_1608Metric" V 2176 972 50  0001 C CNN
 F 3 "~" H 2246 972 50  0001 C CNN
 	1    2246 972
@@
 F 0 "D13" V 2285 1155 50  0000 R CNN
 F 1 "LED" V 2194 1155 50  0000 R CNN
-F 2 "" H 2246 1272 50  0001 C CNN
+F 2 "digitalSystemBoard:LED_3528" H 2246 1272 50  0001 C CNN
 F 3 "~" H 2246 1272 50  0001 C CNN
 	1    2246 1272
@@
 Wire Wire Line
 	6638 3940 6638 3930
-Wire Wire Line
-	6528 3940 6638 3940
 Wire Wire Line
 	8510 3952 8510 3942
@@
 F 0 "R45" H 3508 1762 50  0000 L CNN
 F 1 "10k" H 3508 1671 50  0000 L CNN
-F 2 "" V 3368 1716 50  0001 C CNN
+F 2 "Resistor_SMD:R_0603_1608Metric" V 3368 1716 50  0001 C CNN
 F 3 "~" H 3438 1716 50  0001 C CNN
 	1    3438 1716
@@
 F 0 "R43" H 3358 1612 50  0000 L CNN
 F 1 "10" H 3358 1521 50  0000 L CNN
-F 2 "" V 3218 1566 50  0001 C CNN
+F 2 "Resistor_SMD:R_0603_1608Metric" V 3218 1566 50  0001 C CNN
 F 3 "~" H 3288 1566 50  0001 C CNN
 	1    3288 1566
@@
 F 0 "R47" H 3808 962 50  0000 L CNN
 F 1 "330" H 3808 871 50  0000 L CNN
-F 2 "" V 3668 916 50  0001 C CNN
+F 2 "Resistor_SMD:R_0603_1608Metric" V 3668 916 50  0001 C CNN
 F 3 "~" H 3738 916 50  0001 C CNN
 	1    3738 916
@@
 F 0 "D15" V 3777 1099 50  0000 R CNN
 F 1 "LED" V 3686 1099 50  0000 R CNN
-F 2 "" H 3738 1216 50  0001 C CNN
+F 2 "digitalSystemBoard:LED_3528" H 3738 1216 50  0001 C CNN
 F 3 "~" H 3738 1216 50  0001 C CNN
 	1    3738 1216
@@
 F 0 "R51" H 5252 1738 50  0000 L CNN
 F 1 "10k" H 5252 1647 50  0000 L CNN
-F 2 "" V 5112 1692 50  0001 C CNN
+F 2 "Resistor_SMD:R_0603_1608Metric" V 5112 1692 50  0001 C CNN
 F 3 "~" H 5182 1692 50  0001 C CNN
 	1    5182 1692
@@
 F 0 "R49" H 5102 1588 50  0000 L CNN
 F 1 "10" H 5102 1497 50  0000 L CNN
-F 2 "" V 4962 1542 50  0001 C CNN
+F 2 "Resistor_SMD:R_0603_1608Metric" V 4962 1542 50  0001 C CNN
 F 3 "~" H 5032 1542 50  0001 C CNN
 	1    5032 1542
@@
 F 0 "R53" H 5552 938 50  0000 L CNN
 F 1 "330" H 5552 847 50  0000 L CNN
-F 2 "" V 5412 892 50  0001 C CNN
+F 2 "Resistor_SMD:R_0603_1608Metric" V 5412 892 50  0001 C CNN
 F 3 "~" H 5482 892 50  0001 C CNN
 	1    5482 892
@@
 F 0 "D17" V 5521 1075 50  0000 R CNN
 F 1 "LED" V 5430 1075 50  0000 R CNN
-F 2 "" H 5482 1192 50  0001 C CNN
+F 2 "digitalSystemBoard:LED_3528" H 5482 1192 50  0001 C CNN
 F 3 "~" H 5482 1192 50  0001 C CNN
 	1    5482 1192
@@
 F 0 "R57" H 7034 1724 50  0000 L CNN
 F 1 "10k" H 7034 1633 50  0000 L CNN
-F 2 "" V 6894 1678 50  0001 C CNN
+F 2 "Resistor_SMD:R_0603_1608Metric" V 6894 1678 50  0001 C CNN
 F 3 "~" H 6964 1678 50  0001 C CNN
 	1    6964 1678
@@
 F 0 "R55" H 6884 1574 50  0000 L CNN
 F 1 "10" H 6884 1483 50  0000 L CNN
-F 2 "" V 6744 1528 50  0001 C CNN
+F 2 "Resistor_SMD:R_0603_1608Metric" V 6744 1528 50  0001 C CNN
 F 3 "~" H 6814 1528 50  0001 C CNN
 	1    6814 1528
@@
 F 0 "R59" H 7334 924 50  0000 L CNN
 F 1 "330" H 7334 833 50  0000 L CNN
-F 2 "" V 7194 878 50  0001 C CNN
+F 2 "Resistor_SMD:R_0603_1608Metric" V 7194 878 50  0001 C CNN
 F 3 "~" H 7264 878 50  0001 C CNN
 	1    7264 878
@@
 F 0 "D19" V 7303 1061 50  0000 R CNN
 F 1 "LED" V 7212 1061 50  0000 R CNN
-F 2 "" H 7264 1178 50  0001 C CNN
+F 2 "digitalSystemBoard:LED_3528" H 7264 1178 50  0001 C CNN
 F 3 "~" H 7264 1178 50  0001 C CNN
 	1    7264 1178
@@
 F 0 "R62" H 8840 1672 50  0000 L CNN
 F 1 "10k" H 8840 1581 50  0000 L CNN
-F 2 "" V 8700 1626 50  0001 C CNN
+F 2 "Resistor_SMD:R_0603_1608Metric" V 8700 1626 50  0001 C CNN
 F 3 "~" H 8770 1626 50  0001 C CNN
 	1    8770 1626
@@
 F 0 "R60" H 8690 1522 50  0000 L CNN
 F 1 "10" H 8690 1431 50  0000 L CNN
-F 2 "" V 8550 1476 50  0001 C CNN
+F 2 "Resistor_SMD:R_0603_1608Metric" V 8550 1476 50  0001 C CNN
 F 3 "~" H 8620 1476 50  0001 C CNN
 	1    8620 1476
@@
 F 0 "R64" H 9140 872 50  0000 L CNN
 F 1 "330" H 9140 781 50  0000 L CNN
-F 2 "" V 9000 826 50  0001 C CNN
+F 2 "Resistor_SMD:R_0603_1608Metric" V 9000 826 50  0001 C CNN
 F 3 "~" H 9070 826 50  0001 C CNN
 	1    9070 826
@@
 F 0 "D20" V 9109 1009 50  0000 R CNN
 F 1 "LED" V 9018 1009 50  0000 R CNN
-F 2 "" H 9070 1126 50  0001 C CNN
+F 2 "digitalSystemBoard:LED_3528" H 9070 1126 50  0001 C CNN
 F 3 "~" H 9070 1126 50  0001 C CNN
 	1    9070 1126
@@
 F 0 "R36" H 1770 4118 50  0000 L CNN
 F 1 "10" H 1770 4027 50  0000 L CNN
-F 2 "" V 1630 4072 50  0001 C CNN
+F 2 "Resistor_SMD:R_0603_1608Metric" V 1630 4072 50  0001 C CNN
 F 3 "~" H 1700 4072 50  0001 C CNN
 	1    1700 4072
@@
 F 0 "R38" H 1920 4268 50  0000 L CNN
 F 1 "10k" H 1920 4177 50  0000 L CNN
-F 2 "" V 1780 4222 50  0001 C CNN
+F 2 "Resistor_SMD:R_0603_1608Metric" V 1780 4222 50  0001 C CNN
 F 3 "~" H 1850 4222 50  0001 C CNN
 	1    1850 4222
@@
 F 0 "R40" H 2220 3468 50  0000 L CNN
 F 1 "330" H 2220 3377 50  0000 L CNN
-F 2 "" V 2080 3422 50  0001 C CNN
+F 2 "Resistor_SMD:R_0603_1608Metric" V 2080 3422 50  0001 C CNN
 F 3 "~" H 2150 3422 50  0001 C CNN
 	1    2150 3422
@@
 F 0 "D12" V 2189 3605 50  0000 R CNN
 F 1 "LED" V 2098 3605 50  0000 R CNN
-F 2 "" H 2150 3722 50  0001 C CNN
+F 2 "digitalSystemBoard:LED_3528" H 2150 3722 50  0001 C CNN
 F 3 "~" H 2150 3722 50  0001 C CNN
 	1    2150 3722
@@
 F 0 "R42" H 3320 4040 50  0000 L CNN
 F 1 "10" H 3320 3949 50  0000 L CNN
-F 2 "" V 3180 3994 50  0001 C CNN
+F 2 "Resistor_SMD:R_0603_1608Metric" V 3180 3994 50  0001 C CNN
 F 3 "~" H 3250 3994 50  0001 C CNN
 	1    3250 3994
@@
 F 0 "R44" H 3470 4190 50  0000 L CNN
 F 1 "10k" H 3470 4099 50  0000 L CNN
-F 2 "" V 3330 4144 50  0001 C CNN
+F 2 "Resistor_SMD:R_0603_1608Metric" V 3330 4144 50  0001 C CNN
 F 3 "~" H 3400 4144 50  0001 C CNN
 	1    3400 4144
@@
 F 0 "R46" H 3770 3390 50  0000 L CNN
 F 1 "330" H 3770 3299 50  0000 L CNN
-F 2 "" V 3630 3344 50  0001 C CNN
+F 2 "Resistor_SMD:R_0603_1608Metric" V 3630 3344 50  0001 C CNN
 F 3 "~" H 3700 3344 50  0001 C CNN
 	1    3700 3344
@@
 F 0 "D14" V 3739 3527 50  0000 R CNN
 F 1 "LED" V 3648 3527 50  0000 R CNN
-F 2 "" H 3700 3644 50  0001 C CNN
+F 2 "digitalSystemBoard:LED_3528" H 3700 3644 50  0001 C CNN
 F 3 "~" H 3700 3644 50  0001 C CNN
 	1    3700 3644
@@
 F 0 "R48" H 5050 3988 50  0000 L CNN
 F 1 "10" H 5050 3897 50  0000 L CNN
-F 2 "" V 4910 3942 50  0001 C CNN
+F 2 "Resistor_SMD:R_0603_1608Metric" V 4910 3942 50  0001 C CNN
 F 3 "~" H 4980 3942 50  0001 C CNN
 	1    4980 3942
@@
 F 0 "R50" H 5200 4138 50  0000 L CNN
 F 1 "10k" H 5200 4047 50  0000 L CNN
-F 2 "" V 5060 4092 50  0001 C CNN
+F 2 "Resistor_SMD:R_0603_1608Metric" V 5060 4092 50  0001 C CNN
 F 3 "~" H 5130 4092 50  0001 C CNN
 	1    5130 4092
@@
 F 0 "R52" H 5500 3338 50  0000 L CNN
 F 1 "330" H 5500 3247 50  0000 L CNN
-F 2 "" V 5360 3292 50  0001 C CNN
+F 2 "Resistor_SMD:R_0603_1608Metric" V 5360 3292 50  0001 C CNN
 F 3 "~" H 5430 3292 50  0001 C CNN
 	1    5430 3292
@@
 F 0 "D16" V 5469 3475 50  0000 R CNN
 F 1 "LED" V 5378 3475 50  0000 R CNN
-F 2 "" H 5430 3592 50  0001 C CNN
+F 2 "digitalSystemBoard:LED_3528" H 5430 3592 50  0001 C CNN
 F 3 "~" H 5430 3592 50  0001 C CNN
 	1    5430 3592
@@
 F 0 "R54" H 6858 3976 50  0000 L CNN
 F 1 "10" H 6858 3885 50  0000 L CNN
-F 2 "" V 6718 3930 50  0001 C CNN
+F 2 "Resistor_SMD:R_0603_1608Metric" V 6718 3930 50  0001 C CNN
 F 3 "~" H 6788 3930 50  0001 C CNN
 	1    6788 3930
@@
 F 0 "R56" H 7008 4126 50  0000 L CNN
 F 1 "10k" H 7008 4035 50  0000 L CNN
-F 2 "" V 6868 4080 50  0001 C CNN
+F 2 "Resistor_SMD:R_0603_1608Metric" V 6868 4080 50  0001 C CNN
 F 3 "~" H 6938 4080 50  0001 C CNN
 	1    6938 4080
@@
 F 0 "R58" H 7308 3326 50  0000 L CNN
 F 1 "330" H 7308 3235 50  0000 L CNN
-F 2 "" V 7168 3280 50  0001 C CNN
+F 2 "Resistor_SMD:R_0603_1608Metric" V 7168 3280 50  0001 C CNN
 F 3 "~" H 7238 3280 50  0001 C CNN
 	1    7238 3280
@@
 F 0 "D18" V 7277 3463 50  0000 R CNN
 F 1 "LED" V 7186 3463 50  0000 R CNN
-F 2 "" H 7238 3580 50  0001 C CNN
+F 2 "digitalSystemBoard:LED_3528" H 7238 3580 50  0001 C CNN
 F 3 "~" H 7238 3580 50  0001 C CNN
 	1    7238 3580
@@
 F 0 "R61" H 8730 3988 50  0000 L CNN
 F 1 "10" H 8730 3897 50  0000 L CNN
-F 2 "" V 8590 3942 50  0001 C CNN
+F 2 "Resistor_SMD:R_0603_1608Metric" V 8590 3942 50  0001 C CNN
 F 3 "~" H 8660 3942 50  0001 C CNN
 	1    8660 3942
@@
 F 0 "R63" H 8880 4138 50  0000 L CNN
 F 1 "10k" H 8880 4047 50  0000 L CNN
-F 2 "" V 8740 4092 50  0001 C CNN
+F 2 "Resistor_SMD:R_0603_1608Metric" V 8740 4092 50  0001 C CNN
 F 3 "~" H 8810 4092 50  0001 C CNN
 	1    8810 4092
@@
 F 0 "R65" H 9180 3338 50  0000 L CNN
 F 1 "330" H 9180 3247 50  0000 L CNN
-F 2 "" V 9040 3292 50  0001 C CNN
+F 2 "Resistor_SMD:R_0603_1608Metric" V 9040 3292 50  0001 C CNN
 F 3 "~" H 9110 3292 50  0001 C CNN
 	1    9110 3292
@@
 F 0 "D21" V 9149 3475 50  0000 R CNN
 F 1 "LED" V 9058 3475 50  0000 R CNN
-F 2 "" H 9110 3592 50  0001 C CNN
+F 2 "digitalSystemBoard:LED_3528" H 9110 3592 50  0001 C CNN
 F 3 "~" H 9110 3592 50  0001 C CNN
 	1    9110 3592
@@
 Text Notes 4842 5480 0    139  ~ 0
 LED_DISPLAY\n
+Wire Wire Line
+	6528 3940 6638 3940
 $EndSCHEMATC

Commit message: Upload all footprint
Parts:
- Q12, Q13, Q14, Q15, Q16, Q17, Q18, Q19, Q20, Q21: footprint Package_TO_SOT_SMD:SOT-23 -> digitalSystemBoard:SO65P210X100-3N
Changed lines of the file:
@@
 F 0 "Q13" H 2350 1668 50  0000 L CNN
 F 1 "2N7002" H 2350 1577 50  0000 L CNN
-F 2 "Package_TO_SOT_SMD:SOT-23" H 2346 1547 50  0001 L CIN
+F 2 "digitalSystemBoard:SO65P210X100-3N" H 2346 1547 50  0001 L CIN
 F 3 "https://www.fairchildsemi.com/datasheets/2N/2N7002.pdf" H 2146 1622 50  0001 L CNN
 	1    2146 1622
@@
 F 0 "Q15" H 3842 1612 50  0000 L CNN
 F 1 "2N7002" H 3842 1521 50  0000 L CNN
-F 2 "Package_TO_SOT_SMD:SOT-23" H 3838 1491 50  0001 L CIN
+F 2 "digitalSystemBoard:SO65P210X100-3N" H 3838 1491 50  0001 L CIN
 F 3 "https://www.fairchildsemi.com/datasheets/2N/2N7002.pdf" H 3638 1566 50  0001 L CNN
 	1    3638 1566
@@
 F 0 "Q17" H 5586 1588 50  0000 L CNN
 F 1 "2N7002" H 5586 1497 50  0000 L CNN
-F 2 "Package_TO_SOT_SMD:SOT-23" H 5582 1467 50  0001 L CIN
+F 2 "digitalSystemBoard:SO65P210X100-3N" H 5582 1467 50  0001 L CIN
 F 3 "https://www.fairchildsemi.com/datasheets/2N/2N7002.pdf" H 5382 1542 50  0001 L CNN
 	1    5382 1542
@@
 F 0 "Q19" H 7368 1574 50  0000 L CNN
 F 1 "2N7002" H 7368 1483 50  0000 L CNN
-F 2 "Package_TO_SOT_SMD:SOT-23" H 7364 1453 50  0001 L CIN
+F 2 "digitalSystemBoard:SO65P210X100-3N" H 7364 1453 50  0001 L CIN
 F 3 "https://www.fairchildsemi.com/datasheets/2N/2N7002.pdf" H 7164 1528 50  0001 L CNN
 	1    7164 1528
@@
 F 0 "Q20" H 9174 1522 50  0000 L CNN
 F 1 "2N7002" H 9174 1431 50  0000 L CNN
-F 2 "Package_TO_SOT_SMD:SOT-23" H 9170 1401 50  0001 L CIN
+F 2 "digitalSystemBoard:SO65P210X100-3N" H 9170 1401 50  0001 L CIN
 F 3 "https://www.fairchildsemi.com/datasheets/2N/2N7002.pdf" H 8970 1476 50  0001 L CNN
 	1    8970 1476
@@
 F 0 "Q12" H 2254 4118 50  0000 L CNN
 F 1 "2N7002" H 2254 4027 50  0000 L CNN
-F 2 "Package_TO_SOT_SMD:SOT-23" H 2250 3997 50  0001 L CIN
+F 2 "digitalSystemBoard:SO65P210X100-3N" H 2250 3997 50  0001 L CIN
 F 3 "https://www.fairchildsemi.com/datasheets/2N/2N7002.pdf" H 2050 4072 50  0001 L CNN
 	1    2050 4072
@@
 F 0 "Q14" H 3804 4040 50  0000 L CNN
 F 1 "2N7002" H 3804 3949 50  0000 L CNN
-F 2 "Package_TO_SOT_SMD:SOT-23" H 3800 3919 50  0001 L CIN
+F 2 "digitalSystemBoard:SO65P210X100-3N" H 3800 3919 50  0001 L CIN
 F 3 "https://www.fairchildsemi.com/datasheets/2N/2N7002.pdf" H 3600 3994 50  0001 L CNN
 	1    3600 3994
@@
 F 0 "Q16" H 5534 3988 50  0000 L CNN
 F 1 "2N7002" H 5534 3897 50  0000 L CNN
-F 2 "Package_TO_SOT_SMD:SOT-23" H 5530 3867 50  0001 L CIN
+F 2 "digitalSystemBoard:SO65P210X100-3N" H 5530 3867 50  0001 L CIN
 F 3 "https://www.fairchildsemi.com/datasheets/2N/2N7002.pdf" H 5330 3942 50  0001 L CNN
 	1    5330 3942
@@
 F 0 "Q18" H 7342 3976 50  0000 L CNN
 F 1 "2N7002" H 7342 3885 50  0000 L CNN
-F 2 "Package_TO_SOT_SMD:SOT-23" H 7338 3855 50  0001 L CIN
+F 2 "digitalSystemBoard:SO65P210X100-3N" H 7338 3855 50  0001 L CIN
 F 3 "https://www.fairchildsemi.com/datasheets/2N/2N7002.pdf" H 7138 3930 50  0001 L CNN
 	1    7138 3930
@@
 F 0 "Q21" H 9214 3988 50  0000 L CNN
 F 1 "2N7002" H 9214 3897 50  0000 L CNN
-F 2 "Package_TO_SOT_SMD:SOT-23" H 9210 3867 50  0001 L CIN
+F 2 "digitalSystemBoard:SO65P210X100-3N" H 9210 3867 50  0001 L CIN
 F 3 "https://www.fairchildsemi.com/datasheets/2N/2N7002.pdf" H 9010 3942 50  0001 L CNN
 	1    9010 3942

Commit message: Change PCB
Parts:
- renumbered D13 to D12, D15 to D13, D17 to D14, D19 to D15, D20 to D16, D12 to D17, D14 to D18, D16 to D19, D18 to D20, Q13 to Q12, Q15 to Q13, Q17 to Q14, Q19 to Q15, Q20 to Q16, Q12 to Q17, Q14 to Q18, Q16 to Q19, Q18 to Q20, R37 to R36, R39 to R37, R41 to R38, R43 to R39, R45 to R40, R47 to R41, R49 to R42, R51 to R43, R53 to R44, R55 to R45, R57 to R46, R59 to R47, R60 to R48, R62 to R49, R64 to R50, R36 to R51, R38 to R52, R40 to R53, R42 to R54, R44 to R55, R46 to R56, R48 to R57, R50 to R58, R52 to R59, R54 to R60, R56 to R61, R58 to R62, R61 to R63, R63 to R64

Commit message: Prepare for PCB
Parts:
- removed Q12, Q13, Q14, Q15, Q16, Q17, Q18, Q19, Q20, Q21: 2N7002, digitalSystemBoard:SO65P210X100-3N, symbol Transistor_FET:2N7002
- added Q12, Q13, Q14, Q15, Q16, Q17, Q18, Q19, Q20, Q21: BC847, digitalSystemBoard:SO65P210X100-3N, symbol Transistor_BJT:BC847
- R36, R39, R42, R45, R48, R51, R54, R57, R60, R63: value 10 -> 10k
- R37, R40, R43, R46, R49, R52, R55, R58, R61, R64: value 10k -> 1k8
Connections:
- net GND: now also Q12.2 (E), Q13.2 (E), Q14.2 (E), Q15.2 (E), Q16.2 (E), Q17.2 (E), Q18.2 (E), Q19.2 (E), Q20.2 (E), Q21.2 (E)
- net at R39.1, R40.1: now also Q13.1 (B)
- net at D13.1 (K): now also Q13.3 (C)
- net at R36.1, R37.1: now also Q12.1 (B)
- net at D12.1 (K): now also Q12.3 (C)
- net at R42.1, R43.1: now also Q14.1 (B)
- net at D14.1 (K): now also Q14.3 (C)
- net at R45.1, R46.1: now also Q15.1 (B)
- net at D15.1 (K): now also Q15.3 (C)
- net at R48.1, R49.1: now also Q16.1 (B)
- net at D16.1 (K): now also Q16.3 (C)
- net at R51.1, R52.1: now also Q17.1 (B)
- net at D17.1 (K): now also Q17.3 (C)
- net at R54.1, R55.1: now also Q18.1 (B)
- net at D18.1 (K): now also Q18.3 (C)
- net at R57.1, R58.1: now also Q19.1 (B)
- net at D19.1 (K): now also Q19.3 (C)
- net at R60.1, R61.1: now also Q20.1 (B)
- net at D20.1 (K): now also Q20.3 (C)
- net at R63.1, R64.1: now also Q21.1 (B)
- net at D21.1 (K): now also Q21.3 (C)

Commit message: Update I/O and MCU schematic
Parts:
- removed D20, D21: LED, digitalSystemBoard:LED_3528, symbol Device:LED
- removed Q20, Q21: BC847, digitalSystemBoard:SO65P210X100-3N, symbol Transistor_BJT:BC847
- removed R60, R63: 10k, Resistor_SMD:R_0603_1608Metric, symbol Device:R
- removed R61, R64: 1k8, Resistor_SMD:R_0603_1608Metric, symbol Device:R
- removed R62, R65: 330, Resistor_SMD:R_0603_1608Metric, symbol Device:R
