File: digitalSystemBoard/digitalSystemBoard.sch (KiCad schematic (older format))
At the start: 30 parts, among them J1 Barrel_Jack, J10 Conn_02x04_Odd_Even, J11 Screw_Terminal_01x12, J2 Conn_02x10_Odd_Even, J3 Conn_02x07_Odd_Even, J4 Conn_02x07_Odd_Even, J5 R_7447, J6 R_7447, J7 L_7447, J8 L_7447, J9 Conn_02x04_Odd_Even, Q1 NPN, SW1 SW_SPDT, U1 LM317, U15 KCSA02-105, U16 KCSA02-105, U2 Potentiometer, U3 button, U4 button

Commit message: Upload Timer Block
Parts:
- removed U3, U4: button, symbol digitalSystemBoard:button
- added C? (x2): 22pF, symbol Device:C
- added C? (x5): 0.1uF, symbol Device:C
- added D?: SMF05C.TCT, SC70-6, symbol project:SMF05C.TCT
- added DS?: WC1602A, Display:WC1602A, symbol Display_Character:WC1602A
- added FB? (x4): 80Ohm, symbol Device:Ferrite_Bead_Small
- added J?: USB_OTG, symbol project:USB_OTG
- added R? (x3): 10K, symbol Device:R
- added R?: 1M, symbol Device:R
- added R?: 10k, symbol Device:R
- added R? (x3): 22, symbol Device:R
- added SW2, SW3, SW? (x3): ButtonFirst, TE_4-1437565-9, symbol project:ButtonFirst
- added U?: ATmega32U2-AU, Package_QFP:TQFP-32_7x7mm_P0.8mm, symbol MCU_Microchip_ATmega:ATmega32U2-AU
- added Y?: 16MHz, symbol project:Resonator
- F1: value 4A -> 2A
- Q1: value NPN -> MJD122T4G
Connections:
- net labels added: +5V, D+, D-, VBUS
- net labels removed: V_SOURCE
- wire segments 73 -> 138
- no-connect marks 7 -> 17
Other:
- moved on the sheet: R4

Commit message: Redesign CLOCK_GENERATOR and add footprints for LM317, 5W resistor
Parts:
- removed C? (x2): 22pF, symbol Device:C
- removed C? (x5): 0.1uF, symbol Device:C
- removed D?: SMF05C.TCT, SC70-6, symbol project:SMF05C.TCT
- removed DS?: WC1602A, Display:WC1602A, symbol Display_Character:WC1602A
- removed FB? (x4): 80Ohm, symbol Device:Ferrite_Bead_Small
- removed J?: USB_OTG, symbol project:USB_OTG
- removed R? (x3): 10K, symbol Device:R
- removed R?: 1M, symbol Device:R
- removed R?: 10k, symbol Device:R
- removed R? (x3): 22, symbol Device:R
- removed SW? (x3): ButtonFirst, TE_4-1437565-9, symbol project:ButtonFirst
- removed U?: ATmega32U2-AU, Package_QFP:TQFP-32_7x7mm_P0.8mm, symbol MCU_Microchip_ATmega:ATmega32U2-AU
- removed Y?: 16MHz, symbol project:Resonator
- added J13: Conn_02x03_Odd_Even, symbol Connector_Generic:Conn_02x03_Odd_Even
- F1: footprint (none) -> digitalSystemBoard:Fuse
- J1: footprint (none) -> Connector_BarrelJack:BarrelJack_Horizontal
- Q1: footprint (none) -> digitalSystemBoard:MJD122T4G
- R2: footprint (none) -> digitalSystemBoard:5W_0.22R
- SW1: footprint (none) -> digitalSystemBoard:SS-12D11
- SW2, SW3: symbol project:ButtonFirst -> digitalSystemBoard-rescue:ButtonFirst-project
- U1: footprint (none) -> digitalSystemBoard:LM317; symbol digitalSystemBoard:LM317 -> digitalSystemBoard-rescue:LM317-digitalSystemBoard
- U15, U16: footprint Display_7Segment:KCSC02-105 -> Display_7Segment:7SegmentLED_LTS6760_LTS6780
- U2: footprint (none) -> digitalSystemBoard:TRIM_3296W-1-501; symbol digitalSystemBoard:Potentiometer -> digitalSystemBoard-rescue:Potentiometer-digitalSystemBoard
Connections:
- net labels added: CLK_OUT
- net labels removed: D+, D-, VBUS
- wire segments 138 -> 73
- no-connect marks 17 -> 7

Commit message: Update a part of footprint
Parts:
- removed J11: Screw_Terminal_01x12, symbol Connector:Screw_Terminal_01x12
- removed J5, J6: R_7447, symbol Connector:Screw_Terminal_01x08
- removed J7, J8: L_7447, symbol Connector:Screw_Terminal_01x08
- added J5: INPUT_HEADER, Connector_PinHeader_2.54mm:PinHeader_2x12_P2.54mm_Vertical_SMD, symbol Connector_Generic:Conn_02x12_Odd_Even
- added J6, J7: SN7447, digitalSystemBoard:SN7447, symbol Connector_Generic:Conn_02x08_Odd_Even
- C1, C3: footprint (none) -> Capacitor_SMD:C_0603_1608Metric
- C2: value 10uF -> 100uF_C; footprint (none) -> Capacitor_SMD:CP_Elec_5x5.8
- C4: value 100uF -> 10uF; footprint (none) -> Capacitor_SMD:C_0603_1608Metric
- D1: footprint (none) -> LED_SMD:LED_0805_2012Metric
- J10: value Conn_02x04_Odd_Even -> BCD_1; footprint (none) -> Connector_PinHeader_2.54mm:PinHeader_2x04_P2.54mm_Vertical_SMD
- J13: footprint (none) -> Connector_PinHeader_2.54mm:PinHeader_2x03_P2.54mm_Vertical_SMD
- J2: value Conn_02x10_Odd_Even -> OUTPUT_HEADER; footprint (none) -> Connector_PinHeader_2.54mm:PinHeader_2x10_P2.54mm_Vertical_SMD
- J3: value Conn_02x07_Odd_Even -> 7_LED_IN_2; footprint (none) -> Connector_PinHeader_2.54mm:PinHeader_2x07_P2.54mm_Vertical_SMD
- J4: value Conn_02x07_Odd_Even -> 7_LED_IN_1; footprint (none) -> Connector_PinHeader_2.54mm:PinHeader_2x07_P2.54mm_Vertical_SMD
- J9: value Conn_02x04_Odd_Even -> BCD_2; footprint (none) -> Connector_PinHeader_2.54mm:PinHeader_2x04_P2.54mm_Vertical_SMD
- R1, R3, R4, R5: footprint (none) -> Resistor_SMD:R_0603_1608Metric
- SW2, SW3: footprint TE_4-1437565-9 -> digitalSystemBoard:Button
Connections:
- net labels added: A1, A2, A_J, A_K, A_X, A_Y, B1, B2, B_J, B_K, B_X, B_Y, C1, C2, C_J, C_K, C_X, C_Y, D1, D2, D_J, D_K, D_X, D_Y, E_J, E_K, E_X, E_Y, F_J, F_K, F_X, F_Y, G_J, G_K, G_X, G_Y
- net labels removed: A, B, C, D, E, F, G, a, b, c, d, e, f, g

Commit message: Upload PCB footprint
Parts:
- J1: footprint Connector_BarrelJack:BarrelJack_Horizontal -> footprints:BARREL_JACK
Changed lines of the file:
@@
 F 0 "J1" H 907 1491 50  0000 C CNN
 F 1 "Barrel_Jack" H 907 1400 50  0000 C CNN
-F 2 "Connector_BarrelJack:BarrelJack_Horizontal" H 900 1126 50  0001 C CNN
+F 2 "footprints:BARREL_JACK" H 900 1126 50  0001 C CNN
 F 3 "~" H 900 1126 50  0001 C CNN
 	1    850  1166

Commit message: Upload after error
Connections:
- net GND: now also SW2.2, SW3.2; no longer SW2.1, SW3.1
Changed lines of the file:
@@
 F 6 "Compliant" H 1872 4446 50  0001 L BNN "Field6"
 	1    1872 4446
-	1    0    0    -1
+	0    1    1    0
 $EndComp
 Text Label 2350 4346 0    50   ~ 0
@@
 	1    0    0    -1
 $EndComp
-NoConn ~ 2122 4546
-NoConn ~ 1622 4546
+NoConn ~ 1772 4696
+NoConn ~ 1972 4196
 $Comp
 L power:GND #PWR0101
@@
 F 6 "Compliant" H 3178 4414 50  0001 L BNN "Field6"
 	1    3178 4414
-	1    0    0    -1
+	0    1    1    0
 $EndComp
 Connection ~ 3554 4314
@@
 	1    0    0    -1
 $EndComp
-NoConn ~ 3428 4514
-NoConn ~ 2928 4514
+NoConn ~ 3278 4164
+NoConn ~ 3078 4664
 $Comp
 L power:+5V #PWR0102
@@
 Text Label 2026 3088 2    50   ~ 0
 O9
+Wire Wire Line
+	1772 4196 1622 4196
+Wire Wire Line
+	1622 4196 1622 4346
+Wire Wire Line
+	2122 4346 2122 4696
+Wire Wire Line
+	2122 4696 1972 4696
+Wire Wire Line
+	3078 4164 2928 4164
+Wire Wire Line
+	2928 4164 2928 4314
+Wire Wire Line
+	3428 4314 3428 4664
+Wire Wire Line
+	3428 4664 3278 4664
 $EndSCHEMATC

Commit message: Add usb source block
Connections:
- net VIN: now reaches C1.1, Q1.2 (C), SW1.3 (C), U1.3 (VIN)
Changed lines of the file:
@@
 F1 "CLOCK_GENERATOR.sch" 50
 F2 "CLOCK_OUT" I R 8970 1740 50
+F3 "VIN" I L 5470 1258 50
 $EndSheet
 Text Label 8970 1740 0    50   ~ 0
@@
 Wire Wire Line
 	3428 4664 3278 4664
+Text Label 1690 1082 0    50   ~ 0
+VIN
+Text Label 5470 1258 2    50   ~ 0
+VIN
 $EndSCHEMATC

Commit message: Update I/O and MCU schematic
Parts:
- removed J10: BCD_1, Connector_PinHeader_2.54mm:PinHeader_2x04_P2.54mm_Vertical_SMD, symbol Connector_Generic:Conn_02x04_Odd_Even
- removed J2: OUTPUT_HEADER, Connector_PinHeader_2.54mm:PinHeader_2x10_P2.54mm_Vertical_SMD, symbol Connector_Generic:Conn_02x10_Odd_Even
- removed J9: BCD_2, Connector_PinHeader_2.54mm:PinHeader_2x04_P2.54mm_Vertical_SMD, symbol Connector_Generic:Conn_02x04_Odd_Even
- added J9: Conn_02x08_Counter_Clockwise, symbol Connector_Generic:Conn_02x08_Counter_Clockwise
- added U20: 74LS04, symbol 74xx:74LS04
- U1: footprint digitalSystemBoard:LM317 -> digitalSystemBoard:TO228P991X255-3N
Connections:
- net IB2: now also U20.2; no longer R5.2, SW3.3
- new net: R5.2, SW3.3, U20.1
- new net OA1: J9.12 (Pin_12)
- new net OA2: J9.16 (Pin_16)
- new net OB1: J9.11 (Pin_11)
- new net OB2: J9.15 (Pin_15)
- new net OC1: J9.10 (Pin_10)
- new net OC2: J9.14 (Pin_14)
- new net OD1: J9.9 (Pin_9)
- new net OD2: J9.13 (Pin_13)
- new net TLED1: J9.1 (Pin_1)
- new net TLED2: J9.2 (Pin_2)
- new net TLED3: J9.3 (Pin_3)
- new net TLED4: J9.4 (Pin_4)
- new net TLED5: J9.5 (Pin_5)
- new net TLED6: J9.6 (Pin_6)
- new net TLED7: J9.7 (Pin_7)
- new net TLED8: J9.8 (Pin_8)

Commit message: Update I/O schematic, Complete layout, Start routing
Parts:
- removed J9: Conn_02x08_Counter_Clockwise, symbol Connector_Generic:Conn_02x08_Counter_Clockwise
- removed U20: 74LS04, symbol 74xx:74LS04
- added H0, H1, H2, H3: MountingHole, MountingHole:MountingHole_3.2mm_M3, symbol Mechanical:MountingHole
- added J9: Conn_02x08_Odd_Even, Connector_PinHeader_2.54mm:PinHeader_2x08_P2.54mm_Vertical_SMD, symbol Connector_Generic:Conn_02x08_Odd_Even
- added U20: 74HC04, Package_SO:SOIC-14_3.9x8.7mm_P1.27mm, symbol 74xx:74HC04
Connections:
- net +5V: now also U20.14 (VCC)
- net GND: now also U20.7 (GND)
- net IB2: now also U20.2
- net OA1: now also J9.16 (Pin_16)
- net OA2: now also J9.15 (Pin_15)
- net OB1: now also J9.14 (Pin_14)
- net OB2: now also J9.13 (Pin_13)
- net OC1: now also J9.12 (Pin_12)
- net OC2: now also J9.11 (Pin_11)
- net OD1: now also J9.10 (Pin_10)
- net OD2: now also J9.9 (Pin_9)
- net TLED1: now also J9.1 (Pin_1)
- net TLED2: now also J9.3 (Pin_3)
- net TLED3: now also J9.5 (Pin_5)
- net TLED4: now also J9.7 (Pin_7)
- net TLED5: now also J9.2 (Pin_2)
- net TLED6: now also J9.4 (Pin_4)
- net TLED7: now also J9.6 (Pin_6)
- net TLED8: now also J9.8 (Pin_8)
- net at R5.2, SW3.3: now also U20.1
Changed lines of the file:
@@
 Text Label 6046 6182 2    50   ~ 0
 A_J
-Text Label 6058 7054 0    50   ~ 0
+Text Label 5558 7154 2    50   ~ 0
 OD2
-Text Label 6058 6954 0    50   ~ 0
+Text Label 5558 7254 2    50   ~ 0
 OC2
-Text Label 6058 6854 0    50   ~ 0
+Text Label 5558 7354 2    50   ~ 0
 OB2
-Text Label 6058 6754 0    50   ~ 0
+Text Label 5558 7454 2    50   ~ 0
 OA2
 Text Label 7102 6202 2    50   ~ 0
@@
 Text Label 7380 4194 2    50   ~ 0
 F_Y
+Text Label 6058 7154 0    50   ~ 0
+OD1
+Text Label 6058 7254 0    50   ~ 0
+OC1
+Text Label 6058 7354 0    50   ~ 0
+OB1
 Text Label 6058 7454 0    50   ~ 0
-OD1
-Text Label 6058 7354 0    50   ~ 0
-OC1
-Text Label 6058 7254 0    50   ~ 0
-OB1
-Text Label 6058 7154 0    50   ~ 0
 OA1
 Text Label 7880 4294 0    50   ~ 0
@@
 Text Label 5470 1074 2    50   ~ 0
 VIN
-$Comp
-L 74xx:74LS04 U20
-U 1 1 5F925F26
-P 3956 4314
-F 0 "U20" H 3956 4631 50  0000 C CNN
-F 1 "74LS04" H 3956 4540 50  0000 C CNN
-F 2 "" H 3956 4314 50  0001 C CNN
-F 3 "http://www.ti.com/lit/gpn/sn74LS04" H 3956 4314 50  0001 C CNN
-	1    3956 4314
-	1    0    0    -1
-$EndComp
 Connection ~ 3502 1082
 $Comp
@@
 Text Label 5470 2688 2    50   ~ 0
 D2
-$Comp
-L Connector_Generic:Conn_02x08_Counter_Clockwise J9
-U 1 1 5FB9AF61
-P 5758 7054
-F 0 "J9" H 5808 7571 50  0000 C CNN
-F 1 "Conn_02x08_Counter_Clockwise" H 5808 7480 50  0000 C CNN
-F 2 "" H 5758 7054 50  0001 C CNN
-F 3 "~" H 5758 7054 50  0001 C CNN
-	1    5758 7054
-	1    0    0    -1
-$EndComp
-Text Label 5558 7454 2    50   ~ 0
+Text Label 6058 7054 0    50   ~ 0
 TLED8
-Text Label 5558 7354 2    50   ~ 0
+Text Label 6058 6954 0    50   ~ 0
 TLED7
-Text Label 5558 7254 2    50   ~ 0
+Text Label 6058 6854 0    50   ~ 0
 TLED6
-Text Label 5558 7154 2    50   ~ 0
+Text Label 6058 6754 0    50   ~ 0
 TLED5
 Text Label 5558 7054 2    50   ~ 0
@@
 Wire Wire Line
 	3554 3930 3554 3870
+$Comp
+L Mechanical:MountingHole H2
+U 1 1 5F976335
+P 10036 2838
+F 0 "H2" H 10136 2884 50  0000 L CNN
+F 1 "MountingHole" H 10136 2793 50  0000 L CNN
+F 2 "MountingHole:MountingHole_3.2mm_M3" H 10036 2838 50  0001 C CNN
+F 3 "~" H 10036 2838 50  0001 C CNN
+	1    10036 2838
+	1    0    0    -1
+$EndComp
+$Comp
+L Mechanical:MountingHole H1
+U 1 1 5F976AFE
+P 10036 3030
+F 0 "H1" H 10136 3076 50  0000 L CNN
+F 1 "MountingHole" H 10136 2985 50  0000 L CNN
+F 2 "MountingHole:MountingHole_3.2mm_M3" H 10036 3030 50  0001 C CNN
+F 3 "~" H 10036 3030 50  0001 C CNN
+	1    10036 3030
+	1    0    0    -1
+$EndComp
+$Comp
+L Mechanical:MountingHole H0
+U 1 1 5F97928D
+P 10036 2660
+F 0 "H0" H 10136 2706 50  0000 L CNN
+F 1 "MountingHole" H 10136 2615 50  0000 L CNN
+F 2 "MountingHole:MountingHole_3.2mm_M3" H 10036 2660 50  0001 C CNN
+F 3 "~" H 10036 2660 50  0001 C CNN
+	1    10036 2660
+	1    0    0    -1
+$EndComp
+$Comp
+L Mechanical:MountingHole H3
+U 1 1 5F97B437
+P 10040 3216
+F 0 "H3" H 10140 3262 50  0000 L CNN
+F 1 "MountingHole" H 10140 3171 50  0000 L CNN
+F 2 "MountingHole:MountingHole_3.2mm_M3" H 10040 3216 50  0001 C CNN
+F 3 "~" H 10040 3216 50  0001 C CNN
+	1    10040 3216
+	1    0    0    -1
+$EndComp
+$Comp
+L Connector_Generic:Conn_02x08_Odd_Even J9
+U 1 1 5FA24AF5
+P 5758 7054
+F 0 "J9" H 5808 7571 50  0000 C CNN
+F 1 "Conn_02x08_Odd_Even" H 5808 7480 50  0000 C CNN
+F 2 "Connector_PinHeader_2.54mm:PinHeader_2x08_P2.54mm_Vertical_SMD" H 5758 7054 50  0001 C CNN
+F 3 "~" H 5758 7054 50  0001 C CNN
+	1    5758 7054
+	1    0    0    -1
+$EndComp
+$Comp
+L 74xx:74HC04 U20
+U 1 1 5F9D4EE8
+P 3956 4314
+F 0 "U20" H 3956 4631 50  0000 C CNN
+F 1 "74HC04" H 3956 4540 50  0000 C CNN
+F 2 "Package_SO:SOIC-14_3.9x8.7mm_P1.27mm" H 3956 4314 50  0001 C CNN
+F 3 "https://assets.nexperia.com/documents/data-sheet/74HC_HCT04.pdf" H 3956 4314 50  0001 C CNN
+	1    3956 4314
+	1    0    0    -1
+$EndComp
+$Comp
+L 74xx:74HC04 U20
+U 7 1 5F9E537A
+P 3948 3300
+F 0 "U20" V 4315 3300 50  0000 C CNN
+F 1 "74HC04" V 4224 3300 50  0000 C CNN
+F 2 "Package_SO:SOIC-14_3.9x8.7mm_P1.27mm" H 3948 3300 50  0001 C CNN
+F 3 "https://assets.nexperia.com/documents/data-sheet/74HC_HCT04.pdf" H 3948 3300 50  0001 C CNN
+	7    3948 3300
+	0    -1   -1   0
+$EndComp
+$Comp
+L power:GND #PWR0153
+U 1 1 5F9EDC9A
+P 4502 3300
+F 0 "#PWR0153" H 4502 3050 50  0001 C CNN
+F 1 "GND" H 4507 3127 50  0000 C CNN
+F 2 "" H 4502 3300 50  0001 C CNN
+F 3 "" H 4502 3300 50  0001 C CNN
+	1    4502 3300
+	1    0    0    -1
+$EndComp
+$Comp
+L power:+5V #PWR0154
+U 1 1 5F9EE990
+P 3382 3300
+F 0 "#PWR0154" H 3382 3150 50  0001 C CNN
+F 1 "+5V" H 3397 3473 50  0000 C CNN
+F 2 "" H 3382 3300 50  0001 C CNN
+F 3 "" H 3382 3300 50  0001 C CNN
+	1    3382 3300
+	1    0    0    -1
+$EndComp
+Wire Wire Line
+	3382 3300 3448 3300
+Wire Wire Line
+	4448 3300 4502 3300
 $EndSCHEMATC
