File: digitalSystemBoard/digitalSystemBoard.sch (KiCad schematic (older format))
At the start: 32 parts, among them J1 Barrel_Jack, J13 Conn_02x03_Odd_Even, J3 7_LED_IN_2, J4 7_LED_IN_1, J5 INPUT_HEADER, J6 SN7447, J7 SN7447, J9 Conn_02x08_Odd_Even, Q1 MJD122T4G, SW1 SW_SPDT, SW2 ButtonFirst, SW3 ButtonFirst, U1 LM317, U15 KCSA02-105, U16 KCSA02-105, U2 Potentiometer, U20 74HC04

Commit message: Update new layout, add power vias
Parts:
- added J10: Conn_02x08_Odd_Even, Connector_PinHeader_2.54mm:PinHeader_2x08_P2.54mm_Vertical_SMD, symbol Connector_Generic:Conn_02x08_Odd_Even
- added J11: Conn_02x03_Odd_Even, Connector_PinHeader_2.54mm:PinHeader_2x03_P2.54mm_Vertical_SMD, symbol Connector_Generic:Conn_02x03_Odd_Even
- added V0, V1, V2, V3, V4: POWER_VIAS, digitalSystemBoard:POWER_VIA, symbol digitalSystemBoard-rescue:POWER_VIAS
Connections:
- net labels added: VIA_0, VIA_1
- wire segments 86 -> 96
Other:
- moved on the sheet: R4, R5, U20A, U20G

Commit message: Hot fix libs. Update schematic
Parts:
- removed V0, V1, V2, V3, V4: POWER_VIAS, digitalSystemBoard:POWER_VIA, symbol digitalSystemBoard-rescue:POWER_VIAS
- SW2, SW3: symbol digitalSystemBoard-rescue:ButtonFirst-project -> digitalSystemBoard:ButtonFirst
- U1: symbol digitalSystemBoard-rescue:LM317-digitalSystemBoard -> digitalSystemBoard:LM317
- U2: symbol digitalSystemBoard-rescue:Potentiometer-digitalSystemBoard -> digitalSystemBoard:Potentiometer
Connections:
- net labels removed: VIA_0, VIA_1
Changed lines of the file:
@@
 $EndComp
 $Comp
-L digitalSystemBoard-rescue:ButtonFirst-project SW2
+L digitalSystemBoard:ButtonFirst SW2
 U 1 1 5F8C8A55
 P 1742 5100
@@
 $EndComp
 $Comp
-L digitalSystemBoard-rescue:ButtonFirst-project SW3
+L digitalSystemBoard:ButtonFirst SW3
 U 1 1 5F8DA262
 P 3048 5068
@@
 	2016 2108 2556 2108
 $Comp
-L digitalSystemBoard-rescue:Potentiometer-digitalSystemBoard U2
+L digitalSystemBoard:Potentiometer U2
 U 1 1 5F873747
 P 2556 1632
@@
 	1810 1266 1810 2108
 $Comp
-L digitalSystemBoard-rescue:LM317-digitalSystemBoard U1
+L digitalSystemBoard:LM317 U1
 U 1 1 5F871BB7
 P 2556 1082
@@
 Wire Wire Line
 	3922 2932 3972 2932
-$Comp
-L digitalSystemBoard-rescue:POWER_VIAS V0
-U 1 1 5F9A9094
-P 988 2716
-F 0 "V0" V 1092 2538 50  0000 R CNN
-F 1 "POWER_VIAS" V 1001 2538 50  0000 R CNN
-F 2 "digitalSystemBoard:POWER_VIA" H 988 2716 50  0001 C CNN
-F 3 "" H 988 2716 50  0001 C CNN
-	1    988  2716
-	0    -1   -1   0
-$EndComp
-Text Label 988  2366 0    50   ~ 0
-VIA_0
-Text Label 3924 806  0    50   ~ 0
-VIA_0
-$Comp
-L digitalSystemBoard-rescue:POWER_VIAS V1
-U 1 1 5F9C57FC
-P 1758 2792
-F 0 "V1" V 1862 2614 50  0000 R CNN
-F 1 "POWER_VIAS" V 1771 2614 50  0000 R CNN
-F 2 "digitalSystemBoard:POWER_VIA" H 1758 2792 50  0001 C CNN
-F 3 "" H 1758 2792 50  0001 C CNN
-	1    1758 2792
-	0    -1   -1   0
-$EndComp
-$Comp
-L digitalSystemBoard-rescue:POWER_VIAS V2
-U 1 1 5F9C895C
-P 2542 2764
-F 0 "V2" V 2646 2586 50  0000 R CNN
-F 1 "POWER_VIAS" V 2555 2586 50  0000 R CNN
-F 2 "digitalSystemBoard:POWER_VIA" H 2542 2764 50  0001 C CNN
-F 3 "" H 2542 2764 50  0001 C CNN
-	1    2542 2764
-	0    -1   -1   0
-$EndComp
-Text Label 1758 2442 0    50   ~ 0
-VIA_0
-Text Label 2542 2414 0    50   ~ 0
-VIA_0
-$Comp
-L digitalSystemBoard-rescue:POWER_VIAS V3
-U 1 1 5FA14C14
-P 802 1888
-F 0 "V3" V 906 1710 50  0000 R CNN
-F 1 "POWER_VIAS" V 790 2122 50  0000 R CNN
-F 2 "digitalSystemBoard:POWER_VIA" H 802 1888 50  0001 C CNN
-F 3 "" H 802 1888 50  0001 C CNN
-	1    802  1888
-	0    -1   -1   0
-$EndComp
-Text Label 3032 1680 0    50   ~ 0
-VIA_1
-Text Label 802  1538 0    50   ~ 0
-VIA_1
-$Comp
-L digitalSystemBoard-rescue:POWER_VIAS V4
-U 1 1 5FA1E10B
-P 1232 1874
-F 0 "V4" V 1336 1696 50  0000 R CNN
-F 1 "POWER_VIAS" V 1208 2102 50  0000 R CNN
-F 2 "digitalSystemBoard:POWER_VIA" H 1232 1874 50  0001 C CNN
-F 3 "" H 1232 1874 50  0001 C CNN
-	1    1232 1874
-	0    -1   -1   0
-$EndComp
-Text Label 1232 1524 0    50   ~ 0
-VIA_1
 $EndSCHEMATC

Commit message: Update new schematic.
Parts:
- removed H0, H1, H2, H3: MountingHole, MountingHole:MountingHole_3.2mm_M3, symbol Mechanical:MountingHole
- removed J10, J9: Conn_02x08_Odd_Even, Connector_PinHeader_2.54mm:PinHeader_2x08_P2.54mm_Vertical_SMD, symbol Connector_Generic:Conn_02x08_Odd_Even
- removed J11, J13: Conn_02x03_Odd_Even, Connector_PinHeader_2.54mm:PinHeader_2x03_P2.54mm_Vertical_SMD, symbol Connector_Generic:Conn_02x03_Odd_Even
- removed J3: 7_LED_IN_2, Connector_PinHeader_2.54mm:PinHeader_2x07_P2.54mm_Vertical_SMD, symbol Connector_Generic:Conn_02x07_Odd_Even
- removed J4: 7_LED_IN_1, Connector_PinHeader_2.54mm:PinHeader_2x07_P2.54mm_Vertical_SMD, symbol Connector_Generic:Conn_02x07_Odd_Even
- removed J5: INPUT_HEADER, Connector_PinHeader_2.54mm:PinHeader_2x12_P2.54mm_Vertical_SMD, symbol Connector_Generic:Conn_02x12_Odd_Even
- removed J6, J7: SN7447, digitalSystemBoard:SN7447, symbol Connector_Generic:Conn_02x08_Odd_Even
- removed Q1: MJD122T4G, digitalSystemBoard:MJD122T4G, symbol Device:Q_NPN_BCE
- removed R4, R5: 10K, Resistor_SMD:R_0603_1608Metric, symbol Device:R
- removed SW2, SW3: ButtonFirst, digitalSystemBoard:Button, symbol digitalSystemBoard:ButtonFirst
- removed U15, U16: KCSA02-105, Display_7Segment:7SegmentLED_LTS6760_LTS6780, symbol Display_Character:KCSA02-105
- removed U2: Potentiometer, digitalSystemBoard:TRIM_3296W-1-501, symbol digitalSystemBoard:Potentiometer
- removed U20: 74HC04, Package_SO:SOIC-14_3.9x8.7mm_P1.27mm, symbol 74xx:74HC04
- added J2, J3: Conn_02x02_Odd_Even, symbol Connector_Generic:Conn_02x02_Odd_Even
- added Q1: MJD122T4G, symbol digitalSystemBoard:MJD122T4G
- added TRIM1: Potentiometer, symbol digitalSystemBoard:Potentiometer
- C1, C3, C4: footprint Capacitor_SMD:C_0603_1608Metric -> (none)
- C2: value 100uF_C -> 100uF; footprint Capacitor_SMD:CP_Elec_5x5.8 -> (none)
- D1: footprint LED_SMD:LED_0805_2012Metric -> (none)
- F1: footprint digitalSystemBoard:Fuse -> (none)
- J1: footprint footprints:BARREL_JACK -> (none)
- R1, R3: footprint Resistor_SMD:R_0603_1608Metric -> (none)
- R2: value 0.22Ohm_5W -> 0.22_5W; footprint digitalSystemBoard:5W_0.22R -> (none)
- SW1: footprint digitalSystemBoard:SS-12D11 -> (none)
- U1: footprint digitalSystemBoard:TO228P991X255-3N -> (none)
Connections:
- net labels added: ADJ_CLOCK, BCD_A_0, BCD_A_1, BCD_B_0, BCD_B_1, BCD_C_0, BCD_C_1, BCD_D_0, BCD_D_1, CHANGE_CLK_SRC, DOWN_CLOCK, LED1, LED2, LED3, LED4, LED5, LED6, LED7, LED8, UP_CLOCK, VCC5V
- net labels removed: A1, A2, A_J, A_K, A_X, A_Y, B1, B2, BI_RBO, B_J, B_K, B_X, B_Y, C1, C2, CLK_OUT, C_J, C_K, C_X, C_Y, D1, D2, D_J, D_K, D_X, D_Y, E_J, E_K, E_X, E_Y, F_J, F_K, F_X, F_Y, G_J, G_K, G_X, G_Y, IB1, IB2, LT, O1, O10, O2, O3, O4, O5, O6, O7, O8, O9, OA1, OA2, OB1, OB2, OC1, OC2, OD1, OD2, OLED1, OLED2, OLED3, OLED4, OLED5, OLED6, OLED7, OLED8, RBI, TLED1, TLED2, TLED3, TLED4, TLED5, TLED6, TLED7, TLED8, VCC, VIN
- wire segments 96 -> 35
- no-connect marks 7 -> 2
Other:
- note removed: "CLOCK_BLOCK\n"
- note removed: "INPUT_BLOCK"
- note removed: "OUTPUT_BLOCK\n"
- note removed: "SOURCE_BLOCK\n"

Commit message: Change grid size to 10mils and wire components in power supply and display sheet
Parts:
- removed J2, J3: Conn_02x02_Odd_Even, symbol Connector_Generic:Conn_02x02_Odd_Even
Connections:
- no-connect marks 2 -> 1
Other:
- moved on the sheet: C1, C2, C3, C4, D1, F1, J1, Q1, R1, R2, R3, SW1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

Commit message: Update Schematic for review
Parts:
- C2: footprint (none) -> Capacitor_SMD:CP_Elec_5x5.3
- C3, C4: footprint (none) -> Capacitor_SMD:C_0603_1608Metric
- D1: footprint (none) -> LED_SMD:LED_PLCC-2
- F1: footprint (none) -> digitalSystemBoard:Fuse
- J1: footprint (none) -> Connector_BarrelJack:BarrelJack_Horizontal
- Q1: footprint (none) -> digitalSystemBoard:TO229P990X238-4N
- R1, R3: footprint (none) -> Resistor_SMD:R_0603_1608Metric
- R2: footprint (none) -> digitalSystemBoard:5W_0.22R
- SW1: footprint (none) -> digitalSystemBoard:SS-12D11
- TRIM1: footprint (none) -> digitalSystemBoard:TRIM_3296W-1-501
- U1: footprint (none) -> digitalSystemBoard:TO228P991X255-3N
Connections:
- net +5V is gone; now on net VCC5V: F1.2

Commit message: Add full footprint. Draw layout board
Parts:
- C1: footprint (none) -> Capacitor_SMD:CP_Elec_5x5.8
- C2: footprint Capacitor_SMD:CP_Elec_5x5.3 -> Capacitor_SMD:CP_Elec_5x5.8
- D1: footprint LED_SMD:LED_PLCC-2 -> LED_SMD:LED_0603_1608Metric
- Q1: footprint digitalSystemBoard:TO229P990X238-4N -> digitalSystemBoard:MJD122T4G
- U1: footprint digitalSystemBoard:TO228P991X255-3N -> digitalSystemBoard:LM317AMDT
Changed lines of the file:
@@
 F 0 "D1" V 1019 2192 50  0000 R CNN
 F 1 "LED" V 928 2192 50  0000 R CNN
-F 2 "LED_SMD:LED_PLCC-2" H 980 2310 50  0001 C CNN
+F 2 "LED_SMD:LED_0603_1608Metric" H 980 2310 50  0001 C CNN
 F 3 "~" H 980 2310 50  0001 C CNN
 	1    980  2310
@@
 F 0 "Q1" H 6270 1716 50  0000 L CNN
 F 1 "MJD122T4G" H 6270 1625 50  0000 L CNN
-F 2 "digitalSystemBoard:TO229P990X238-4N" H 6080 1670 50  0001 C CNN
+F 2 "digitalSystemBoard:MJD122T4G" H 6080 1670 50  0001 C CNN
 F 3 "" H 6080 1670 50  0001 C CNN
 	1    6080 1670
@@
 F 0 "C2" H 5015 2096 50  0000 L CNN
 F 1 "100uF" H 5015 2005 50  0000 L CNN
-F 2 "Capacitor_SMD:CP_Elec_5x5.3" H 4900 2050 50  0001 C CNN
+F 2 "Capacitor_SMD:CP_Elec_5x5.8" H 4900 2050 50  0001 C CNN
 F 3 "~" H 4900 2050 50  0001 C CNN
 	1    4900 2050
@@
 F 0 "C1" H 3325 2016 50  0000 L CNN
 F 1 "0.1uF" H 3325 1925 50  0000 L CNN
-F 2 "" H 3210 1970 50  0001 C CNN
+F 2 "Capacitor_SMD:CP_Elec_5x5.8" H 3210 1970 50  0001 C CNN
 F 3 "~" H 3210 1970 50  0001 C CNN
 	1    3210 1970
@@
 F 0 "U1" H 3910 1985 50  0000 C CNN
 F 1 "LM317" H 3910 1894 50  0000 C CNN
-F 2 "digitalSystemBoard:TO228P991X255-3N" H 3810 1570 50  0001 C CNN
+F 2 "digitalSystemBoard:LM317AMDT" H 3810 1570 50  0001 C CNN
 F 3 "" H 3810 1570 50  0001 C CNN
 	1    3910 1670
@@
 Text Label 6180 2680 0    50   ~ 0
 VCC5V
-$Sheet
-S 4710 3740 1590 3910
-U 5FBA3F95
-F0 "Header" 50
-F1 "Header.sch" 50
-F2 "GPIO_BCD_A_0" I L 4710 4200 50
-F3 "GPIO_BCD_B_0" I L 4710 4400 50
-F4 "GPIO_BCD_C_0" I L 4710 4600 50
-F5 "GPIO_BCD_D_0" I L 4710 4800 50
-F6 "GPIO_LED_8" I L 4710 5900 50
-F7 "GPIO_LED_7" I L 4710 6100 50
-F8 "GPIO_LED_6" I L 4710 6300 50
-F9 "GPIO_LED_5" I L 4710 6500 50
-F10 "GPIO_LED_3" I L 4710 6900 50
-F11 "GPIO_LED_4" I L 4710 6700 50
-F12 "GPIO_LED_2" I L 4710 7100 50
-F13 "GPIO_LED_1" I L 4710 7300 50
-F14 "GPIO_BCD_A_1" I L 4710 5000 50
-F15 "GPIO_BCD_B_1" I L 4710 5200 50
-F16 "GPIO_BCD_C_1" I L 4710 5400 50
-F17 "GPIO_BCD_D_1" I L 4710 5600 50
-F18 "SEG_A_0" I R 6300 3800 50
-F19 "SEG_B_0" I R 6300 4000 50
-F20 "SEG_C_0" I R 6300 4200 50
-F21 "SEG_D_0" I R 6300 4400 50
-F22 "SEG_E_0" I R 6300 4600 50
-F23 "SEG_F_0" I R 6300 4800 50
-F24 "SEG_G_0" I R 6300 5000 50
-F25 "SEG_A_1" I R 6300 5200 50
-F26 "SEG_B_1" I R 6300 5400 50
-F27 "SEG_C_1" I R 6300 5600 50
-F28 "SEG_D_1" I R 6300 5800 50
-F29 "SEG_E_1" I R 6300 6000 50
-F30 "SEG_F_1" I R 6300 6200 50
-F31 "SEG_G_1" I R 6300 6400 50
-F32 "SW1" I R 6300 6900 50
-F33 "SW2" I R 6300 7000 50
-F34 "SW3" I R 6300 7100 50
-F35 "SW4" I R 6300 7200 50
-F36 "SW5" I R 6300 7300 50
-F37 "SW6" I R 6300 7400 50
-F38 "SW7" I R 6300 7500 50
-F39 "SW8" I R 6300 7600 50
-F40 "KEY0" I R 6300 6600 50
-F41 "KEY1" I R 6300 6700 50
-F42 "CLK_OUT" I L 4710 4000 50
-F43 "VCC5V" I L 4710 3800 50
-$EndSheet
 Text Label 4710 3800 2    50   ~ 0
 VCC5V
@@
 Text Label 10110 4680 0    50   ~ 0
 KEY1
+$Sheet
+S 4710 3740 1590 3910
+U 5FBA3F95
+F0 "Header and Mounting" 50
+F1 "Header_and_Mounting.sch" 50
+F2 "GPIO_BCD_A_0" I L 4710 4200 50
+F3 "GPIO_BCD_B_0" I L 4710 4400 50
+F4 "GPIO_BCD_C_0" I L 4710 4600 50
+F5 "GPIO_BCD_D_0" I L 4710 4800 50
+F6 "GPIO_LED_8" I L 4710 5900 50
+F7 "GPIO_LED_7" I L 4710 6100 50
+F8 "GPIO_LED_6" I L 4710 6300 50
+F9 "GPIO_LED_5" I L 4710 6500 50
+F10 "GPIO_LED_3" I L 4710 6900 50
+F11 "GPIO_LED_4" I L 4710 6700 50
+F12 "GPIO_LED_2" I L 4710 7100 50
+F13 "GPIO_LED_1" I L 4710 7300 50
+F14 "GPIO_BCD_A_1" I L 4710 5000 50
+F15 "GPIO_BCD_B_1" I L 4710 5200 50
+F16 "GPIO_BCD_C_1" I L 4710 5400 50
+F17 "GPIO_BCD_D_1" I L 4710 5600 50
+F18 "SEG_A_0" I R 6300 3800 50
+F19 "SEG_B_0" I R 6300 4000 50
+F20 "SEG_C_0" I R 6300 4200 50
+F21 "SEG_D_0" I R 6300 4400 50
+F22 "SEG_E_0" I R 6300 4600 50
+F23 "SEG_F_0" I R 6300 4800 50
+F24 "SEG_G_0" I R 6300 5000 50
+F25 "SEG_A_1" I R 6300 5200 50
+F26 "SEG_B_1" I R 6300 5400 50
+F27 "SEG_C_1" I R 6300 5600 50
+F28 "SEG_D_1" I R 6300 5800 50
+F29 "SEG_E_1" I R 6300 6000 50
+F30 "SEG_F_1" I R 6300 6200 50
+F31 "SEG_G_1" I R 6300 6400 50
+F32 "SW1" I R 6300 6900 50
+F33 "SW2" I R 6300 7000 50
+F34 "SW3" I R 6300 7100 50
+F35 "SW4" I R 6300 7200 50
+F36 "SW5" I R 6300 7300 50
+F37 "SW6" I R 6300 7400 50
+F38 "SW7" I R 6300 7500 50
+F39 "SW8" I R 6300 7600 50
+F40 "KEY0" I R 6300 6600 50
+F41 "KEY1" I R 6300 6700 50
+F42 "CLK_OUT" I L 4710 4000 50
+F43 "VCC5V" I L 4710 3800 50
+$EndSheet
 $EndSCHEMATC

Commit message: Layout power block
Parts:
- R3: value 220 -> 330
Changed lines of the file:
@@
 P 980 1970
 F 0 "R3" H 1050 2016 50  0000 L CNN
-F 1 "220" H 1050 1925 50  0000 L CNN
+F 1 "330" H 1050 1925 50  0000 L CNN
 F 2 "Resistor_SMD:R_0603_1608Metric" V 910 1970 50  0001 C CNN
 F 3 "~" H 980 1970 50  0001 C CNN

Commit message: Layout 70 percent board
Changed lines of the file:
@@
 LED6
 Text Label 8000 1790 2    50   ~ 0
+LED4
+Text Label 8000 1590 2    50   ~ 0
 LED5
-Text Label 8000 1590 2    50   ~ 0
-LED4
 Text Label 8000 1390 2    50   ~ 0
 LED3
