File: digitalSystemBoard/digitalSystemBoard.sch (KiCad schematic (older format))
At the start: 14 parts, among them J1 Barrel_Jack, Q1 MJD122T4G, SW1 SW_SPDT, U1 LM317

Commit message: Hot fix: change symbol and footprint of the barrell jack
Parts:
- J1: symbol Connector:Barrel_Jack -> Connector:Barrel_Jack_Switch
Connections:
- wire segments 38 -> 39
Changed lines of the file:
@@
 EESchema Schematic File Version 4
-LIBS:digitalSystemBoard-cache
-EELAYER 29 0
+EELAYER 30 0
 EELAYER END
 $Descr A4 11693 8268
@@
 $EndComp
 $Comp
-L Connector:Barrel_Jack J1
+L Connector:Barrel_Jack_Switch J1
 U 1 1 5FB7408F
 P 1700 1670
@@
 	3210 1470 3210 1670
 NoConn ~ 2440 1670
+Wire Wire Line
+	2000 1670 2000 1770
+Connection ~ 2000 1770
 $EndSCHEMATC

Commit message: Hot fix: Change footprint. Fix power schematic.
Parts:
- C2: footprint Capacitor_SMD:CP_Elec_5x5.8 -> Capacitor_SMD:CP_Elec_6.3x7.7
Connections:
- net at TRIM1.3, U1.1 (ADJ): now also R1.2, TRIM1.2
Other:
- moved on the sheet: R1
Changed lines of the file:
@@
 F 0 "C2" H 5015 2096 50  0000 L CNN
 F 1 "100uF" H 5015 2005 50  0000 L CNN
-F 2 "Capacitor_SMD:CP_Elec_5x5.8" H 4900 2050 50  0001 C CNN
+F 2 "Capacitor_SMD:CP_Elec_6.3x7.7" H 4900 2050 50  0001 C CNN
 F 3 "~" H 4900 2050 50  0001 C CNN
 	1    4900 2050
@@
 F 3 "~" H 6180 2110 50  0001 C CNN
 	1    6180 2110
-	1    0    0    -1
-$EndComp
-$Comp
-L Device:R R1
-U 1 1 5FB7DFDC
-P 4490 2050
-F 0 "R1" H 4560 2096 50  0000 L CNN
-F 1 "220" H 4560 2005 50  0000 L CNN
-F 2 "Resistor_SMD:R_0603_1608Metric" V 4420 2050 50  0001 C CNN
-F 3 "~" H 4490 2050 50  0001 C CNN
-	1    4490 2050
 	1    0    0    -1
 $EndComp
@@
 	2000 1570 2040 1570
 Wire Wire Line
-	3910 1970 3910 2050
+	3910 1970 3910 2000
 Wire Wire Line
 	3210 2120 3210 2690
@@
 Connection ~ 3210 2690
 Wire Wire Line
-	4490 2200 4490 2350
-Wire Wire Line
-	4490 2350 4260 2350
-Wire Wire Line
-	4310 1670 4490 1670
-Wire Wire Line
 	6180 1870 6180 1960
 Wire Wire Line
@@
 Wire Wire Line
 	6180 2620 6180 2680
-Wire Wire Line
-	4490 1900 4490 1670
-Connection ~ 4490 1670
-Wire Wire Line
-	4490 1670 4900 1670
 Wire Wire Line
 	4900 1900 4900 1670
@@
 	2000 1670 2000 1770
 Connection ~ 2000 1770
+$Comp
+L Device:R R1
+U 1 1 5FB7DFDC
+P 4470 1850
+F 0 "R1" H 4540 1896 50  0000 L CNN
+F 1 "220" H 4540 1805 50  0000 L CNN
+F 2 "Resistor_SMD:R_0603_1608Metric" V 4400 1850 50  0001 C CNN
+F 3 "~" H 4470 1850 50  0001 C CNN
+	1    4470 1850
+	1    0    0    -1
+$EndComp
+Wire Wire Line
+	4310 1670 4470 1670
+Wire Wire Line
+	4470 2000 3910 2000
+Connection ~ 3910 2000
+Wire Wire Line
+	3910 2000 3910 2050
+Wire Wire Line
+	4470 1700 4470 1670
+Connection ~ 4470 1670
+Wire Wire Line
+	4470 1670 4900 1670
+Wire Wire Line
+	4470 2000 4470 2350
+Wire Wire Line
+	4470 2350 4260 2350
+Connection ~ 4470 2000
 $EndSCHEMATC

Commit message: Debug error part 2
Parts:
- R3: value 330 -> 470
Changed lines of the file:
@@
-$EndComp
-$Comp
-L Device:R R3
-U 1 1 5FB7DD09
-P 980 1970
-F 0 "R3" H 1050 2016 50  0000 L CNN
-F 1 "330" H 1050 1925 50  0000 L CNN
-F 2 "Resistor_SMD:R_0603_1608Metric" V 910 1970 50  0001 C CNN
-F 3 "~" H 980 1970 50  0001 C CNN
-	1    980  1970
-	1    0    0    -1
 $EndComp
 $Comp
@@
 	4470 2350 4260 2350
 Connection ~ 4470 2000
+$Comp
+L Device:R R3
+U 1 1 5FB7DD09
+P 980 1970
+F 0 "R3" H 1050 2016 50  0000 L CNN
+F 1 "470" H 1050 1925 50  0000 L CNN
+F 2 "Resistor_SMD:R_0603_1608Metric" V 910 1970 50  0001 C CNN
+F 3 "~" H 980 1970 50  0001 C CNN
+	1    980  1970
+	1    0    0    -1
+$EndComp
 $EndSCHEMATC

Commit message: Add discharge resistor for power block
Parts:
- added R77: 1k, Resistor_SMD:R_0603_1608Metric, symbol Device:R
Connections:
- net GND: now also R77.1
- net at C4.1, F1.1, R2.2: now also R77.2
Changed lines of the file:
@@
 Text Label 10110 4680 0    50   ~ 0
 KEY1
+Wire Wire Line
+	2440 1470 3210 1470
+Connection ~ 3210 1470
+Wire Wire Line
+	3210 1470 3210 1670
+NoConn ~ 2440 1670
+Wire Wire Line
+	2000 1670 2000 1770
+Connection ~ 2000 1770
+$Comp
+L Device:R R1
+U 1 1 5FB7DFDC
+P 4470 1850
+F 0 "R1" H 4540 1896 50  0000 L CNN
+F 1 "220" H 4540 1805 50  0000 L CNN
+F 2 "Resistor_SMD:R_0603_1608Metric" V 4400 1850 50  0001 C CNN
+F 3 "~" H 4470 1850 50  0001 C CNN
+	1    4470 1850
+	1    0    0    -1
+$EndComp
+Wire Wire Line
+	4310 1670 4470 1670
+Wire Wire Line
+	4470 2000 3910 2000
+Connection ~ 3910 2000
+Wire Wire Line
+	3910 2000 3910 2050
+Wire Wire Line
+	4470 1700 4470 1670
+Connection ~ 4470 1670
+Wire Wire Line
+	4470 1670 4900 1670
+Wire Wire Line
+	4470 2000 4470 2350
+Wire Wire Line
+	4470 2350 4260 2350
+Connection ~ 4470 2000
+$Comp
+L Device:R R3
+U 1 1 5FB7DD09
+P 980 1970
+F 0 "R3" H 1050 2016 50  0000 L CNN
+F 1 "470" H 1050 1925 50  0000 L CNN
+F 2 "Resistor_SMD:R_0603_1608Metric" V 910 1970 50  0001 C CNN
+F 3 "~" H 980 1970 50  0001 C CNN
+	1    980  1970
+	1    0    0    -1
+$EndComp
+$Comp
+L Device:R R77
+U 1 1 601177E6
+P 6570 2470
+F 0 "R77" H 6500 2424 50  0000 R CNN
+F 1 "1k" H 6500 2515 50  0000 R CNN
+F 2 "Resistor_SMD:R_0603_1608Metric" V 6500 2470 50  0001 C CNN
+F 3 "~" H 6570 2470 50  0001 C CNN
+	1    6570 2470
+	-1   0    0    1
+$EndComp
 $Sheet
 S 4710 3740 1590 3910
@@
 F43 "VCC5V" I L 4710 3800 50
 $EndSheet
-Wire Wire Line
-	2440 1470 3210 1470
-Connection ~ 3210 1470
-Wire Wire Line
-	3210 1470 3210 1670
-NoConn ~ 2440 1670
-Wire Wire Line
-	2000 1670 2000 1770
-Connection ~ 2000 1770
 $Comp
-L Device:R R1
-U 1 1 5FB7DFDC
-P 4470 1850
-F 0 "R1" H 4540 1896 50  0000 L CNN
-F 1 "220" H 4540 1805 50  0000 L CNN
-F 2 "Resistor_SMD:R_0603_1608Metric" V 4400 1850 50  0001 C CNN
-F 3 "~" H 4470 1850 50  0001 C CNN
-	1    4470 1850
+L power:GND #PWR0166
+U 1 1 6011F9E2
+P 6570 2620
+F 0 "#PWR0166" H 6570 2370 50  0001 C CNN
+F 1 "GND" H 6575 2447 50  0000 C CNN
+F 2 "" H 6570 2620 50  0001 C CNN
+F 3 "" H 6570 2620 50  0001 C CNN
+	1    6570 2620
 	1    0    0    -1
 $EndComp
 Wire Wire Line
-	4310 1670 4470 1670
+	6180 2290 6570 2290
 Wire Wire Line
-	4470 2000 3910 2000
-Connection ~ 3910 2000
-Wire Wire Line
-	3910 2000 3910 2050
-Wire Wire Line
-	4470 1700 4470 1670
-Connection ~ 4470 1670
-Wire Wire Line
-	4470 1670 4900 1670
-Wire Wire Line
-	4470 2000 4470 2350
-Wire Wire Line
-	4470 2350 4260 2350
-Connection ~ 4470 2000
-$Comp
-L Device:R R3
-U 1 1 5FB7DD09
-P 980 1970
-F 0 "R3" H 1050 2016 50  0000 L CNN
-F 1 "470" H 1050 1925 50  0000 L CNN
-F 2 "Resistor_SMD:R_0603_1608Metric" V 910 1970 50  0001 C CNN
-F 3 "~" H 980 1970 50  0001 C CNN
-	1    980  1970
-	1    0    0    -1
-$EndComp
+	6570 2290 6570 2320
 $EndSCHEMATC

Commit message: Fix bug in BCD, add an rheostat on Vo and add an resistor on LED+
Changed lines of the file:
@@
 Text Label 10100 2990 0    50   ~ 0
 BCD_A_1
-Text Label 10100 2865 0    50   ~ 0
+Text Label 10100 2740 0    50   ~ 0
 BCD_C_0
-Text Label 10100 2740 0    50   ~ 0
-BCD_D_0
 Text Label 10100 2615 0    50   ~ 0
 BCD_B_0
@@
 Text Label 10110 4880 0    50   ~ 0
 UP_CLOCK
-$Sheet
-S 1240 3740 2010 3900
-U 5FBA4597
-F0 "MCU" 50
-F1 "MCU.sch" 50
-F2 "VCC5V" I L 1240 3840 50
-F3 "GPIO_LED_1" I L 1240 4040 50
-F4 "GPIO_LED_2" I L 1240 4190 50
-F5 "GPIO_LED_3" I L 1240 4340 50
-F6 "GPIO_LED_4" I L 1240 4490 50
-F7 "GPIO_LED_7" I L 1240 4940 50
-F8 "GPIO_LED_8" I L 1240 5090 50
-F9 "GPIO_BCD_A_0" I L 1240 5390 50
-F10 "GPIO_BCD_B_0" I L 1240 5540 50
-F11 "GPIO_BCD_C_0" I L 1240 5690 50
-F12 "GPIO_BCD_D_0" I L 1240 5840 50
-F13 "GPIO_BCD_B_1" I L 1240 6190 50
-F14 "GPIO_BCD_C_1" I L 1240 6340 50
-F15 "GPIO_BCD_D_1" I L 1240 6490 50
-F16 "GPIO_LED_6" I L 1240 4790 50
-F17 "GPIO_LED_5" I L 1240 4640 50
-F18 "GPIO_BCD_A_1" I L 1240 6040 50
-F19 "LED1" I R 3250 4040 50
-F20 "LED2" I R 3250 4190 50
-F21 "LED3" I R 3250 4340 50
-F22 "LED4" I R 3250 4490 50
-F23 "LED5" I R 3250 4640 50
-F24 "LED6" I R 3250 4790 50
-F25 "LED7" I R 3250 4940 50
-F26 "LED8" I R 3250 5090 50
-F27 "BCD_A_0" I R 3250 5390 50
-F28 "BCD_B_0" I R 3250 5540 50
-F29 "BCD_C_0" I R 3250 5690 50
-F30 "BCD_D_0" I R 3250 5840 50
-F31 "BCD_A_1" I R 3250 6040 50
-F32 "BCD_B_1" I R 3250 6190 50
-F33 "BCD_C_1" I R 3250 6340 50
-F34 "BCD_D_1" I R 3250 6490 50
-F35 "CLK_OUT" I R 3250 3840 50
-F36 "ADJ_CLOCK" I L 1240 7240 50
-F37 "UP_CLK" I L 1240 6790 50
-F38 "DOWN_CLK" I L 1240 6940 50
-F39 "CHANGE_CLK_SRC" I L 1240 7090 50
-F40 "7SEGLED_TEST_ON" I R 3250 6800 50
-F41 "7SEGLED_TEST_OFF" I R 3250 7000 50
-$EndSheet
 Text Label 980  1780 0    50   ~ 0
 VCC5V
@@
 Wire Wire Line
 	6570 2290 6570 2320
+Text Label 10100 2865 0    50   ~ 0
+BCD_C_0
+$Sheet
+S 1240 3740 2010 3900
+U 5FBA4597
+F0 "MCU" 50
+F1 "MCU.sch" 50
+F2 "VCC5V" I L 1240 3840 50
+F3 "GPIO_LED_1" I L 1240 4040 50
+F4 "GPIO_LED_2" I L 1240 4190 50
+F5 "GPIO_LED_3" I L 1240 4340 50
+F6 "GPIO_LED_4" I L 1240 4490 50
+F7 "GPIO_LED_7" I L 1240 4940 50
+F8 "GPIO_LED_8" I L 1240 5090 50
+F9 "GPIO_BCD_A_0" I L 1240 5390 50
+F10 "GPIO_BCD_B_0" I L 1240 5540 50
+F11 "GPIO_BCD_C_0" I L 1240 5690 50
+F12 "GPIO_BCD_D_0" I L 1240 5840 50
+F13 "GPIO_BCD_B_1" I L 1240 6190 50
+F14 "GPIO_BCD_C_1" I L 1240 6340 50
+F15 "GPIO_BCD_D_1" I L 1240 6490 50
+F16 "GPIO_LED_6" I L 1240 4790 50
+F17 "GPIO_LED_5" I L 1240 4640 50
+F18 "GPIO_BCD_A_1" I L 1240 6040 50
+F19 "LED1" I R 3250 4040 50
+F20 "LED2" I R 3250 4190 50
+F21 "LED3" I R 3250 4340 50
+F22 "LED4" I R 3250 4490 50
+F23 "LED5" I R 3250 4640 50
+F24 "LED6" I R 3250 4790 50
+F25 "LED7" I R 3250 4940 50
+F26 "LED8" I R 3250 5090 50
+F27 "BCD_A_0" I R 3250 5390 50
+F28 "BCD_B_0" I R 3250 5540 50
+F29 "BCD_C_0" I R 3250 5690 50
+F30 "BCD_D_0" I R 3250 5840 50
+F31 "BCD_A_1" I R 3250 6040 50
+F32 "BCD_B_1" I R 3250 6190 50
+F33 "BCD_C_1" I R 3250 6340 50
+F34 "BCD_D_1" I R 3250 6490 50
+F35 "CLK_OUT" I R 3250 3840 50
+F36 "ADJ_CLOCK" I L 1240 7240 50
+F37 "UP_CLK" I L 1240 6790 50
+F38 "DOWN_CLK" I L 1240 6940 50
+F39 "CHANGE_CLK_SRC" I L 1240 7090 50
+F40 "7SEGLED_TEST_ON" I R 3250 6800 50
+F41 "7SEGLED_TEST_OFF" I R 3250 7000 50
+$EndSheet
 $EndSCHEMATC

Commit message: Add IC 74HC595 and R for input pin
Changed lines of the file:
@@
 	6570 2290 6570 2320
 Text Label 10100 2865 0    50   ~ 0
-BCD_C_0
+BCD_D_0
 $Sheet
 S 1240 3740 2010 3900

Commit message: Add Power_module to schematic and pcb
Parts:
- removed C1: 0.1uF, Capacitor_SMD:CP_Elec_5x5.8, symbol Device:CP1
- removed C2: 100uF, Capacitor_SMD:CP_Elec_6.3x7.7, symbol Device:CP1
- removed C3, C4: 10uF, Capacitor_SMD:C_0603_1608Metric, symbol Device:C
- removed D1: LED, LED_SMD:LED_0603_1608Metric, symbol Device:LED
- removed Q1: MJD122T4G, digitalSystemBoard:MJD122T4G, symbol digitalSystemBoard:MJD122T4G
- removed R1: 220, Resistor_SMD:R_0603_1608Metric, symbol Device:R
- removed R2: 0.22_5W, digitalSystemBoard:5W_0.22R, symbol Device:R
- removed R3: 470, Resistor_SMD:R_0603_1608Metric, symbol Device:R
- removed R77: 1k, Resistor_SMD:R_0603_1608Metric, symbol Device:R
- removed TRIM1: Potentiometer, digitalSystemBoard:TRIM_3296W-1-501, symbol digitalSystemBoard:Potentiometer
- removed U1: LM317, digitalSystemBoard:LM317AMDT, symbol digitalSystemBoard:LM317
- added PW1: Power_Module, digitalSystemBoard:Power_Module, symbol digitalSystemBoard:Power_Module
- F1: value 2A -> 3A
Connections:
- net GND: now also PW1.2 (GND)
- net VCC5V: now also F1.1; no longer F1.2
- net at SW1.1 (A): now also PW1.1 (Vin+)
- new net: F1.2, PW1.3 (Vout+)
- no-connect marks 1 -> 2
Other:
- moved on the sheet: F1, J1, SW1

Commit message: Fix name of all device
Parts:
- renumbered F1 to F0, J1 to J0, PW1 to PM0, SW1 to SW0
Changed lines of the file:
@@
 $EndSheet
 $Comp
-L Switch:SW_SPDT SW1
+L Switch:SW_SPDT SW0
 U 1 1 5FB75652
 P 2730 1910
-F 0 "SW1" H 2730 2195 50  0000 C CNN
+F 0 "SW0" H 2730 2195 50  0000 C CNN
 F 1 "SW_SPDT" H 2730 2104 50  0000 C CNN
 F 2 "digitalSystemBoard:SS-12D11" H 2730 1910 50  0001 C CNN
@@
 	2930 1810 3180 1810
 $Comp
-L Device:Fuse F1
+L Device:Fuse F0
 U 1 1 5FB8596A
 P 4450 1960
-F 0 "F1" H 4510 2006 50  0000 L CNN
+F 0 "F0" H 4510 2006 50  0000 L CNN
 F 1 "3A" H 4510 1915 50  0000 L CNN
 F 2 "digitalSystemBoard:Fuse" V 4380 1960 50  0001 C CNN
@@
 	4180 1810 4450 1810
 $Comp
-L Connector:Barrel_Jack_Switch J1
+L Connector:Barrel_Jack_Switch J0
 U 1 1 5FB7408F
 P 2190 2010
-F 0 "J1" H 2247 2335 50  0000 C CNN
+F 0 "J0" H 2247 2335 50  0000 C CNN
 F 1 "Barrel_Jack" H 2247 2244 50  0000 C CNN
 F 2 "Connector_BarrelJack:BarrelJack_Horizontal" H 2240 1970 50  0001 C CNN
@@
 	3190 2360 3680 2360
 $Comp
-L digitalSystemBoard:Power_Module PW1
+L digitalSystemBoard:Power_Module PM0
 U 1 1 6094F958
 P 3680 1810
-F 0 "PW1" H 3680 2375 50  0000 C CNN
+F 0 "PM0" H 3680 2375 50  0000 C CNN
 F 1 "Power_Module" H 3680 2284 50  0000 C CNN
 F 2 "digitalSystemBoard:Power_Module" H 3680 1810 50  0001 C CNN
