File: digitalSystemBoard/SWITCH_AND_BUTTON.sch (KiCad schematic (older format))
At the start: 65 parts, among them Q10 BC847, Q11 BC847, Q12 BC847, Q13 BC847, Q14 BC847, Q15 BC847, Q16 BC847, Q17 BC847, U10 IO_Switch, U11 IO_Switch, U12 IO_Switch, U13 IO_Switch, U14 74LS04, U15 Potentiometer, U6 IO_Switch, U7 IO_Switch, U8 IO_Switch, U9 IO_Switch

Commit message: Change grid size to 10mils and wire components in power supply and display sheet
Parts:
- removed unit 2 of U14
- removed unit 3 of U14
- removed unit 4 of U14
Connections:
- net KEY2: now also C7.1, KEY2.3, KEY2.4, R54.1
- net KEY4: now also C9.1, KEY4.3, KEY4.4, R56.1
Changed lines of the file:
@@
 Text HLabel 3250 4500 2    50   Input ~ 0
 KEY0
-Text HLabel 3860 6550 2    50   Input ~ 0
+Text HLabel 3230 6550 2    50   Input ~ 0
 KEY2
 Text HLabel 3860 5425 2    50   Input ~ 0
 KEY1
-$Comp
-L 74xx:74LS04 U14
-U 2 1 5FC70EB0
-P 3560 6550
-F 0 "U14" H 3560 6867 50  0000 C CNN
-F 1 "74LS04" H 3560 6776 50  0000 C CNN
-F 2 "" H 3560 6550 50  0001 C CNN
-F 3 "http://www.ti.com/lit/gpn/sn74LS04" H 3560 6550 50  0001 C CNN
-	2    3560 6550
-	1    0    0    -1
-$EndComp
 Text HLabel 5340 5125 0    50   Input ~ 0
 VCC5V
@@
 Wire Wire Line
 	2760 6550 2760 6650
-Wire Wire Line
-	3010 6550 3260 6550
 Connection ~ 3010 6550
-Text HLabel 6180 6550 2    50   Input ~ 0
+Text HLabel 5520 6550 2    50   Input ~ 0
 KEY4
-Text HLabel 6190 5425 2    50   Input ~ 0
-KEY3
-$Comp
-L 74xx:74LS04 U14
-U 4 1 5FC7346F
-P 5880 6550
-F 0 "U14" H 5880 6867 50  0000 C CNN
-F 1 "74LS04" H 5880 6776 50  0000 C CNN
-F 2 "" H 5880 6550 50  0001 C CNN
-F 3 "http://www.ti.com/lit/gpn/sn74LS04" H 5880 6550 50  0001 C CNN
-	4    5880 6550
-	1    0    0    -1
-$EndComp
-$Comp
-L 74xx:74LS04 U14
-U 3 1 5FC72106
-P 5890 5425
-F 0 "U14" H 5890 5742 50  0000 C CNN
-F 1 "74LS04" H 5890 5651 50  0000 C CNN
-F 2 "" H 5890 5425 50  0001 C CNN
-F 3 "http://www.ti.com/lit/gpn/sn74LS04" H 5890 5425 50  0001 C CNN
-	3    5890 5425
-	1    0    0    -1
-$EndComp
 $Comp
 L digitalSystemBoard:ButtonFirst KEY3
@@
 Wire Wire Line
 	5090 5425 5090 5525
-Wire Wire Line
-	5340 5425 5590 5425
 Connection ~ 5340 5425
 $Comp
@@
 Wire Wire Line
 	5080 6550 5080 6650
-Wire Wire Line
-	5330 6550 5580 6550
 Connection ~ 5330 6550
 Text HLabel 8320 5040 0    50   Input ~ 0
@@
 $EndComp
 Connection ~ 4580 6950
+Wire Wire Line
+	3230 6550 3010 6550
+Wire Wire Line
+	5520 6550 5330 6550
+Text HLabel 5481 5422 2    50   Input ~ 0
+KEY3
 $EndSCHEMATC

Commit message: Change grid size of all schematic
Connections:
- net KEY3: now also C8.2, KEY3.3, KEY3.4, R55.1
Other:
- moved on the sheet: C5, C6, C7, C8, C9, D2, KEY0, KEY1, KEY2, KEY3, KEY4, Q10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

Commit message: Update Schematic for review
Parts:
- C5, C6, C7, C8, C9: footprint (none) -> Capacitor_SMD:C_0603_1608Metric
- D2, D3, D4, D5, D6, D7, D8, D9: footprint (none) -> LED_SMD:LED_PLCC-2
- KEY0, KEY1: footprint TE_4-1437565-9 -> digitalSystemBoard:Button
- KEY2, KEY3, KEY4: footprint TE_4-1437565-9 -> digitalSystemBoard:Button_CLOCK
- R28, R29, R30, R31, R32, R33, R34, R35, R36, R37, R38, R39, R40, R41, R42, R43, R44, R45, R46, R47, R48, R49, R50, R51, R52, R53, R54, R55, R56: footprint (none) -> Resistor_SMD:R_0603_1608Metric
- U10, U11, U12, U13, U6, U7, U8, U9: footprint (none) -> digitalSystemBoard:SS-12F44G5
- U15: footprint (none) -> digitalSystemBoard:RV09S

Commit message: Review schematic and change pin in slide switch
Connections:
- net GND: now also U10.3, U11.3, U12.3, U13.3, U6.3, U7.3, U8.3, U9.3
- no-connect marks 24 -> 16
Changed lines of the file:
@@
 NoConn ~ 1090 1300
 NoConn ~ 1090 2000
-NoConn ~ 1340 1500
 Text HLabel 1340 1800 2    50   Input ~ 0
 VCC5V
@@
 NoConn ~ 3240 1280
 NoConn ~ 3240 1980
-NoConn ~ 3490 1480
 Text HLabel 3490 1780 2    50   Input ~ 0
 VCC5V
@@
 NoConn ~ 5540 1280
 NoConn ~ 5540 1980
-NoConn ~ 5790 1480
 Text HLabel 5790 1780 2    50   Input ~ 0
 VCC5V
@@
 $EndComp
 Wire Wire Line
-	8020 1640 8120 1640
-Wire Wire Line
 	8440 1640 8450 1640
 $Comp
@@
 NoConn ~ 7770 1290
 NoConn ~ 7770 1990
-NoConn ~ 8020 1490
 Text HLabel 8020 1790 2    50   Input ~ 0
 VCC5V
@@
 NoConn ~ 1100 3000
 NoConn ~ 1100 3700
-NoConn ~ 1350 3200
 Text HLabel 1350 3500 2    50   Input ~ 0
 VCC5V
@@
 $EndComp
 Wire Wire Line
-	3500 3330 3610 3330
-Wire Wire Line
 	3920 3330 3930 3330
 $Comp
@@
 NoConn ~ 3250 2980
 NoConn ~ 3250 3680
-NoConn ~ 3500 3180
 Text HLabel 3500 3480 2    50   Input ~ 0
 VCC5V
@@
 $EndComp
 Wire Wire Line
-	5740 3340 5810 3340
-Wire Wire Line
 	6160 3340 6170 3340
 $Comp
@@
 NoConn ~ 5490 2990
 NoConn ~ 5490 3690
-NoConn ~ 5740 3190
 Text HLabel 5740 3490 2    50   Input ~ 0
 VCC5V
@@
 NoConn ~ 7760 2990
 NoConn ~ 7760 3690
-NoConn ~ 8010 3190
 Text HLabel 8010 3490 2    50   Input ~ 0
 VCC5V
@@
 Wire Wire Line
 	5880 1630 5910 1630
-Text HLabel 8120 1170 0    50   Input ~ 0
+Text HLabel 8120 940  0    50   Input ~ 0
 SW4
-Wire Wire Line
-	8120 1170 8120 1640
-Connection ~ 8120 1640
-Wire Wire Line
-	8120 1640 8140 1640
-Text HLabel 1460 2860 0    50   Input ~ 0
+Text HLabel 1460 2590 0    50   Input ~ 0
 SW5
-Wire Wire Line
-	1460 2860 1460 3350
 Connection ~ 1460 3350
 Wire Wire Line
 	1460 3350 1470 3350
-Text HLabel 3590 2840 0    50   Input ~ 0
+Text HLabel 3600 2660 0    50   Input ~ 0
 SW6
-Wire Wire Line
-	3590 2840 3610 2840
-Wire Wire Line
-	3610 2840 3610 3330
-Connection ~ 3610 3330
-Wire Wire Line
-	3610 3330 3620 3330
-Text HLabel 5810 2860 0    50   Input ~ 0
+Text HLabel 5810 2680 0    50   Input ~ 0
 SW7
-Wire Wire Line
-	5810 2860 5810 3340
-Connection ~ 5810 3340
-Wire Wire Line
-	5810 3340 5860 3340
-Text HLabel 8100 2910 0    50   Input ~ 0
+Text HLabel 8100 2660 0    50   Input ~ 0
 SW8
-Wire Wire Line
-	8100 2910 8100 3340
 Connection ~ 8100 3340
 Wire Wire Line
@@
 	3300 4910 3300 4880
 Connection ~ 2300 4910
+$Comp
+L power:GND #PWR0158
+U 1 1 5FC9CC7F
+P 1280 1400
+F 0 "#PWR0158" H 1280 1150 50  0001 C CNN
+F 1 "GND" H 1285 1227 50  0000 C CNN
+F 2 "" H 1280 1400 50  0001 C CNN
+F 3 "" H 1280 1400 50  0001 C CNN
+	1    1280 1400
+	-1   0    0    1
+$EndComp
+Wire Wire Line
+	1280 1400 1340 1400
+Wire Wire Line
+	1340 1400 1340 1500
+$Comp
+L power:GND #PWR0159
+U 1 1 5FCD64D4
+P 3400 1320
+F 0 "#PWR0159" H 3400 1070 50  0001 C CNN
+F 1 "GND" H 3405 1147 50  0000 C CNN
+F 2 "" H 3400 1320 50  0001 C CNN
+F 3 "" H 3400 1320 50  0001 C CNN
+	1    3400 1320
+	-1   0    0    1
+$EndComp
+$Comp
+L power:GND #PWR0160
+U 1 1 5FCD80A6
+P 5730 1360
+F 0 "#PWR0160" H 5730 1110 50  0001 C CNN
+F 1 "GND" H 5735 1187 50  0000 C CNN
+F 2 "" H 5730 1360 50  0001 C CNN
+F 3 "" H 5730 1360 50  0001 C CNN
+	1    5730 1360
+	-1   0    0    1
+$EndComp
+$Comp
+L power:GND #PWR0161
+U 1 1 5FCD9869
+P 7980 1360
+F 0 "#PWR0161" H 7980 1110 50  0001 C CNN
+F 1 "GND" H 7985 1187 50  0000 C CNN
+F 2 "" H 7980 1360 50  0001 C CNN
+F 3 "" H 7980 1360 50  0001 C CNN
+	1    7980 1360
+	-1   0    0    1
+$EndComp
+Wire Wire Line
+	8120 1640 8140 1640
+Wire Wire Line
+	8020 1640 8120 1640
+Connection ~ 8120 1640
+Wire Wire Line
+	8120 940  8120 1640
+Wire Wire Line
+	3400 1320 3490 1320
+Wire Wire Line
+	3490 1320 3490 1480
+Wire Wire Line
+	5790 1480 5790 1360
+Wire Wire Line
+	5790 1360 5730 1360
+Wire Wire Line
+	8020 1490 8020 1360
+Wire Wire Line
+	8020 1360 7980 1360
+Wire Wire Line
+	3500 3330 3600 3330
+Wire Wire Line
+	3600 2660 3600 3330
+Connection ~ 3600 3330
+Wire Wire Line
+	3600 3330 3620 3330
+Wire Wire Line
+	5810 3340 5860 3340
+Wire Wire Line
+	5740 3340 5810 3340
+Connection ~ 5810 3340
+Wire Wire Line
+	5810 2680 5810 3340
+Wire Wire Line
+	8100 2660 8100 3340
+Wire Wire Line
+	1460 2590 1460 3350
+$Comp
+L power:GND #PWR0162
+U 1 1 5FD9E08E
+P 1270 3040
+F 0 "#PWR0162" H 1270 2790 50  0001 C CNN
+F 1 "GND" H 1275 2867 50  0000 C CNN
+F 2 "" H 1270 3040 50  0001 C CNN
+F 3 "" H 1270 3040 50  0001 C CNN
+	1    1270 3040
+	-1   0    0    1
+$EndComp
+Wire Wire Line
+	1350 3200 1350 3040
+Wire Wire Line
+	1350 3040 1270 3040
+$Comp
+L power:GND #PWR0163
+U 1 1 5FDC371E
+P 3420 2990
+F 0 "#PWR0163" H 3420 2740 50  0001 C CNN
+F 1 "GND" H 3425 2817 50  0000 C CNN
+F 2 "" H 3420 2990 50  0001 C CNN
+F 3 "" H 3420 2990 50  0001 C CNN
+	1    3420 2990
+	-1   0    0    1
+$EndComp
+$Comp
+L power:GND #PWR0164
+U 1 1 5FDC3D93
+P 5680 3020
+F 0 "#PWR0164" H 5680 2770 50  0001 C CNN
+F 1 "GND" H 5685 2847 50  0000 C CNN
+F 2 "" H 5680 3020 50  0001 C CNN
+F 3 "" H 5680 3020 50  0001 C CNN
+	1    5680 3020
+	-1   0    0    1
+$EndComp
+$Comp
+L power:GND #PWR0165
+U 1 1 5FDC5334
+P 7920 2970
+F 0 "#PWR0165" H 7920 2720 50  0001 C CNN
+F 1 "GND" H 7925 2797 50  0000 C CNN
+F 2 "" H 7920 2970 50  0001 C CNN
+F 3 "" H 7920 2970 50  0001 C CNN
+	1    7920 2970
+	-1   0    0    1
+$EndComp
+Wire Wire Line
+	3500 3180 3500 2990
+Wire Wire Line
+	3500 2990 3420 2990
+Wire Wire Line
+	5740 3190 5740 3020
+Wire Wire Line
+	5740 3020 5680 3020
+Wire Wire Line
+	8010 3190 8010 2970
+Wire Wire Line
+	8010 2970 7920 2970
 $EndSCHEMATC
