File: digitalSystemBoard/SWITCH_AND_BUTTON.sch (KiCad schematic (older format))
At the start: 65 parts, among them Q10 BC847, Q11 BC847, Q12 BC847, Q13 BC847, Q14 BC847, Q15 BC847, Q16 BC847, Q17 BC847, U10 IO_Switch, U11 IO_Switch, U12 IO_Switch, U13 IO_Switch, U14 74LS04, U15 Potentiometer, U6 IO_Switch, U7 IO_Switch, U8 IO_Switch, U9 IO_Switch

Commit message: Add full footprint. Draw layout board
Parts:
- D2, D3, D4, D5, D6, D7, D8, D9: footprint LED_SMD:LED_PLCC-2 -> LED_SMD:LED_0603_1608Metric
- U14: footprint (none) -> Package_SO:SOIC-14_3.9x8.7mm_P1.27mm
Connections:
- no-connect marks 16 -> 0
Changed lines of the file:
@@
 F 0 "D2" V 2289 1092 50  0000 R CNN
 F 1 "LED" V 2198 1092 50  0000 R CNN
-F 2 "LED_SMD:LED_PLCC-2" H 2250 1210 50  0001 C CNN
+F 2 "LED_SMD:LED_0603_1608Metric" H 2250 1210 50  0001 C CNN
 F 3 "~" H 2250 1210 50  0001 C CNN
 	1    2250 1210
@@
 F 0 "U14" H 3540 5867 50  0000 C CNN
 F 1 "74LS04" H 3540 5776 50  0000 C CNN
-F 2 "" H 3540 5550 50  0001 C CNN
+F 2 "Package_SO:SOIC-14_3.9x8.7mm_P1.27mm" H 3540 5550 50  0001 C CNN
 F 3 "http://www.ti.com/lit/gpn/sn74LS04" H 3540 5550 50  0001 C CNN
 	1    3540 5550
@@
 F 0 "U14" H 7060 5116 50  0000 L CNN
 F 1 "74LS04" H 7060 5025 50  0000 L CNN
-F 2 "" H 6830 5070 50  0001 C CNN
+F 2 "Package_SO:SOIC-14_3.9x8.7mm_P1.27mm" H 6830 5070 50  0001 C CNN
 F 3 "http://www.ti.com/lit/gpn/sn74LS04" H 6830 5070 50  0001 C CNN
 	7    6830 5070
@@
 Text HLabel 2250 700  0    50   Input ~ 0
 VCC5V
-NoConn ~ 1090 1300
-NoConn ~ 1090 2000
 Text HLabel 1340 1800 2    50   Input ~ 0
 VCC5V
@@
 F 0 "D3" V 4439 1072 50  0000 R CNN
 F 1 "LED" V 4348 1072 50  0000 R CNN
-F 2 "LED_SMD:LED_PLCC-2" H 4400 1190 50  0001 C CNN
+F 2 "LED_SMD:LED_0603_1608Metric" H 4400 1190 50  0001 C CNN
 F 3 "~" H 4400 1190 50  0001 C CNN
 	1    4400 1190
@@
 Text HLabel 4400 680  0    50   Input ~ 0
 VCC5V
-NoConn ~ 3240 1280
-NoConn ~ 3240 1980
 Text HLabel 3490 1780 2    50   Input ~ 0
 VCC5V
@@
 F 0 "D4" V 6739 1072 50  0000 R CNN
 F 1 "LED" V 6648 1072 50  0000 R CNN
-F 2 "LED_SMD:LED_PLCC-2" H 6700 1190 50  0001 C CNN
+F 2 "LED_SMD:LED_0603_1608Metric" H 6700 1190 50  0001 C CNN
 F 3 "~" H 6700 1190 50  0001 C CNN
 	1    6700 1190
@@
 Text HLabel 6700 680  0    50   Input ~ 0
 VCC5V
-NoConn ~ 5540 1280
-NoConn ~ 5540 1980
 Text HLabel 5790 1780 2    50   Input ~ 0
 VCC5V
@@
 F 0 "D5" V 8969 1082 50  0000 R CNN
 F 1 "LED" V 8878 1082 50  0000 R CNN
-F 2 "LED_SMD:LED_PLCC-2" H 8930 1200 50  0001 C CNN
+F 2 "LED_SMD:LED_0603_1608Metric" H 8930 1200 50  0001 C CNN
 F 3 "~" H 8930 1200 50  0001 C CNN
 	1    8930 1200
@@
 Text HLabel 8930 690  0    50   Input ~ 0
 VCC5V
-NoConn ~ 7770 1290
-NoConn ~ 7770 1990
 Text HLabel 8020 1790 2    50   Input ~ 0
 VCC5V
@@
 F 0 "D6" V 2299 2792 50  0000 R CNN
 F 1 "LED" V 2208 2792 50  0000 R CNN
-F 2 "LED_SMD:LED_PLCC-2" H 2260 2910 50  0001 C CNN
+F 2 "LED_SMD:LED_0603_1608Metric" H 2260 2910 50  0001 C CNN
 F 3 "~" H 2260 2910 50  0001 C CNN
 	1    2260 2910
@@
 Text HLabel 2260 2400 0    50   Input ~ 0
 VCC5V
-NoConn ~ 1100 3000
-NoConn ~ 1100 3700
 Text HLabel 1350 3500 2    50   Input ~ 0
 VCC5V
@@
 F 0 "D7" V 4449 2772 50  0000 R CNN
 F 1 "LED" V 4358 2772 50  0000 R CNN
-F 2 "LED_SMD:LED_PLCC-2" H 4410 2890 50  0001 C CNN
+F 2 "LED_SMD:LED_0603_1608Metric" H 4410 2890 50  0001 C CNN
 F 3 "~" H 4410 2890 50  0001 C CNN
 	1    4410 2890
@@
 Text HLabel 4410 2380 0    50   Input ~ 0
 VCC5V
-NoConn ~ 3250 2980
-NoConn ~ 3250 3680
 Text HLabel 3500 3480 2    50   Input ~ 0
 VCC5V
@@
 F 0 "D8" V 6689 2782 50  0000 R CNN
 F 1 "LED" V 6598 2782 50  0000 R CNN
-F 2 "LED_SMD:LED_PLCC-2" H 6650 2900 50  0001 C CNN
+F 2 "LED_SMD:LED_0603_1608Metric" H 6650 2900 50  0001 C CNN
 F 3 "~" H 6650 2900 50  0001 C CNN
 	1    6650 2900
@@
 Text HLabel 6650 2390 0    50   Input ~ 0
 VCC5V
-NoConn ~ 5490 2990
-NoConn ~ 5490 3690
 Text HLabel 5740 3490 2    50   Input ~ 0
 VCC5V
@@
 F 0 "D9" V 8959 2782 50  0000 R CNN
 F 1 "LED" V 8868 2782 50  0000 R CNN
-F 2 "LED_SMD:LED_PLCC-2" H 8920 2900 50  0001 C CNN
+F 2 "LED_SMD:LED_0603_1608Metric" H 8920 2900 50  0001 C CNN
 F 3 "~" H 8920 2900 50  0001 C CNN
 	1    8920 2900
@@
 Text HLabel 8920 2390 0    50   Input ~ 0
 VCC5V
-NoConn ~ 7760 2990
-NoConn ~ 7760 3690
 Text HLabel 8010 3490 2    50   Input ~ 0
 VCC5V
