File: digitalSystemBoard/SWITCH_AND_BUTTON.sch (KiCad schematic (older format))
At the start: 65 parts, among them Q10 BC847, Q11 BC847, Q12 BC847, Q13 BC847, Q14 BC847, Q15 BC847, Q16 BC847, Q17 BC847, U10 IO_Switch, U11 IO_Switch, U12 IO_Switch, U13 IO_Switch, U14 74LS04, U15 Potentiometer, U6 IO_Switch, U7 IO_Switch, U8 IO_Switch, U9 IO_Switch

Commit message: Hot fix: Change footprint. Fix power schematic.
Parts:
- Q10, Q11, Q12, Q13, Q14, Q15, Q16, Q17: footprint Package_TO_SOT_SMD:SOT-23 -> digitalSystemBoard:SO65P210X100-3N
Changed lines of the file:
@@
 F 0 "Q10" H 2341 1696 50  0000 L CNN
 F 1 "BC847" H 2341 1605 50  0000 L CNN
-F 2 "Package_TO_SOT_SMD:SOT-23" H 2350 1575 50  0001 L CIN
+F 2 "digitalSystemBoard:SO65P210X100-3N" H 2350 1575 50  0001 L CIN
 F 3 "http://www.infineon.com/dgdl/Infineon-BC847SERIES_BC848SERIES_BC849SERIES_BC850SERIES-DS-v01_01-en.pdf?fileId=db3a304314dca389011541d4630a1657" H 2150 1650 50  0001 L CNN
 	1    2150 1650
@@
 F 0 "Q11" H 4491 1676 50  0000 L CNN
 F 1 "BC847" H 4491 1585 50  0000 L CNN
-F 2 "Package_TO_SOT_SMD:SOT-23" H 4500 1555 50  0001 L CIN
+F 2 "digitalSystemBoard:SO65P210X100-3N" H 4500 1555 50  0001 L CIN
 F 3 "http://www.infineon.com/dgdl/Infineon-BC847SERIES_BC848SERIES_BC849SERIES_BC850SERIES-DS-v01_01-en.pdf?fileId=db3a304314dca389011541d4630a1657" H 4300 1630 50  0001 L CNN
 	1    4300 1630
@@
 F 0 "Q12" H 6791 1676 50  0000 L CNN
 F 1 "BC847" H 6791 1585 50  0000 L CNN
-F 2 "Package_TO_SOT_SMD:SOT-23" H 6800 1555 50  0001 L CIN
+F 2 "digitalSystemBoard:SO65P210X100-3N" H 6800 1555 50  0001 L CIN
 F 3 "http://www.infineon.com/dgdl/Infineon-BC847SERIES_BC848SERIES_BC849SERIES_BC850SERIES-DS-v01_01-en.pdf?fileId=db3a304314dca389011541d4630a1657" H 6600 1630 50  0001 L CNN
 	1    6600 1630
@@
 F 0 "Q13" H 9021 1686 50  0000 L CNN
 F 1 "BC847" H 9021 1595 50  0000 L CNN
-F 2 "Package_TO_SOT_SMD:SOT-23" H 9030 1565 50  0001 L CIN
+F 2 "digitalSystemBoard:SO65P210X100-3N" H 9030 1565 50  0001 L CIN
 F 3 "http://www.infineon.com/dgdl/Infineon-BC847SERIES_BC848SERIES_BC849SERIES_BC850SERIES-DS-v01_01-en.pdf?fileId=db3a304314dca389011541d4630a1657" H 8830 1640 50  0001 L CNN
 	1    8830 1640
@@
 F 0 "Q14" H 2351 3396 50  0000 L CNN
 F 1 "BC847" H 2351 3305 50  0000 L CNN
-F 2 "Package_TO_SOT_SMD:SOT-23" H 2360 3275 50  0001 L CIN
+F 2 "digitalSystemBoard:SO65P210X100-3N" H 2360 3275 50  0001 L CIN
 F 3 "http://www.infineon.com/dgdl/Infineon-BC847SERIES_BC848SERIES_BC849SERIES_BC850SERIES-DS-v01_01-en.pdf?fileId=db3a304314dca389011541d4630a1657" H 2160 3350 50  0001 L CNN
 	1    2160 3350
@@
 F 0 "Q15" H 4501 3376 50  0000 L CNN
 F 1 "BC847" H 4501 3285 50  0000 L CNN
-F 2 "Package_TO_SOT_SMD:SOT-23" H 4510 3255 50  0001 L CIN
+F 2 "digitalSystemBoard:SO65P210X100-3N" H 4510 3255 50  0001 L CIN
 F 3 "http://www.infineon.com/dgdl/Infineon-BC847SERIES_BC848SERIES_BC849SERIES_BC850SERIES-DS-v01_01-en.pdf?fileId=db3a304314dca389011541d4630a1657" H 4310 3330 50  0001 L CNN
 	1    4310 3330
@@
 F 0 "Q16" H 6741 3386 50  0000 L CNN
 F 1 "BC847" H 6741 3295 50  0000 L CNN
-F 2 "Package_TO_SOT_SMD:SOT-23" H 6750 3265 50  0001 L CIN
+F 2 "digitalSystemBoard:SO65P210X100-3N" H 6750 3265 50  0001 L CIN
 F 3 "http://www.infineon.com/dgdl/Infineon-BC847SERIES_BC848SERIES_BC849SERIES_BC850SERIES-DS-v01_01-en.pdf?fileId=db3a304314dca389011541d4630a1657" H 6550 3340 50  0001 L CNN
 	1    6550 3340
@@
 F 0 "Q17" H 9011 3386 50  0000 L CNN
 F 1 "BC847" H 9011 3295 50  0000 L CNN
-F 2 "Package_TO_SOT_SMD:SOT-23" H 9020 3265 50  0001 L CIN
+F 2 "digitalSystemBoard:SO65P210X100-3N" H 9020 3265 50  0001 L CIN
 F 3 "http://www.infineon.com/dgdl/Infineon-BC847SERIES_BC848SERIES_BC849SERIES_BC850SERIES-DS-v01_01-en.pdf?fileId=db3a304314dca389011541d4630a1657" H 8820 3340 50  0001 L CNN
 	1    8820 3340

Commit message: Fix name of all device
Parts:
- C0: renamed from C6; LCSC (none) -> C14663
- C1: renamed from C5; LCSC (none) -> C14663
- C2: renamed from C7; LCSC (none) -> C14663
- C3: renamed from C8; LCSC (none) -> C14663
- C4: renamed from C9; LCSC (none) -> C14663
- renumbered D2 to D0, D3 to D1, D4 to D2, D5 to D3, D6 to D4, D7 to D5, D8 to D6, D9 to D7, Q12 to Q10, Q13 to Q11, Q14 to Q12, Q15 to Q13, Q16 to Q14, Q17 to Q15, Q10 to Q8, Q11 to Q9, R53 to R52, R52 to R53, U6 to SW1, U7 to SW2, U8 to SW3, U9 to SW4, U10 to SW5, U11 to SW6, U12 to SW7, U13 to SW8, U14 to U4, U15 to U5

Commit message: Update voltage bias for LED green and LED yellow
Parts:
- R28, R31, R34, R37, R40, R43, R46, R49: value 10k -> 27k
- R29, R32, R35, R38, R41, R44, R47, R50: value 1k8 -> 4.7k
- R30, R33, R36, R39, R42, R45, R48, R51: value 470 -> 1.8k
Changed lines of the file:
@@
 P 1610 1650
 F 0 "R28" V 1403 1650 50  0000 C CNN
-F 1 "10k" V 1494 1650 50  0000 C CNN
+F 1 "27k" V 1494 1650 50  0000 C CNN
 F 2 "Resistor_SMD:R_0603_1608Metric" V 1540 1650 50  0001 C CNN
 F 3 "~" H 1610 1650 50  0001 C CNN
@@
 P 2250 850
 F 0 "R30" H 2320 896 50  0000 L CNN
-F 1 "470" H 2320 805 50  0000 L CNN
+F 1 "1.8k" H 2320 805 50  0000 L CNN
 F 2 "Resistor_SMD:R_0603_1608Metric" V 2180 850 50  0001 C CNN
 F 3 "~" H 2250 850 50  0001 C CNN
@@
 P 1770 1960
 F 0 "R29" H 1700 1914 50  0000 R CNN
-F 1 "1k8" H 1700 2005 50  0000 R CNN
+F 1 "4.7k" H 1700 2005 50  0000 R CNN
 F 2 "Resistor_SMD:R_0603_1608Metric" V 1700 1960 50  0001 C CNN
 F 3 "~" H 1770 1960 50  0001 C CNN
@@
 P 3760 1630
 F 0 "R31" V 3553 1630 50  0000 C CNN
-F 1 "10k" V 3644 1630 50  0000 C CNN
+F 1 "27k" V 3644 1630 50  0000 C CNN
 F 2 "Resistor_SMD:R_0603_1608Metric" V 3690 1630 50  0001 C CNN
 F 3 "~" H 3760 1630 50  0001 C CNN
@@
 P 4400 830
 F 0 "R33" H 4470 876 50  0000 L CNN
-F 1 "470" H 4470 785 50  0000 L CNN
+F 1 "1.8k" H 4470 785 50  0000 L CNN
 F 2 "Resistor_SMD:R_0603_1608Metric" V 4330 830 50  0001 C CNN
 F 3 "~" H 4400 830 50  0001 C CNN
@@
 P 3920 1940
 F 0 "R32" H 3850 1894 50  0000 R CNN
-F 1 "1k8" H 3850 1985 50  0000 R CNN
+F 1 "4.7k" H 3850 1985 50  0000 R CNN
 F 2 "Resistor_SMD:R_0603_1608Metric" V 3850 1940 50  0001 C CNN
 F 3 "~" H 3920 1940 50  0001 C CNN
@@
 P 6060 1630
 F 0 "R34" V 5853 1630 50  0000 C CNN
-F 1 "10k" V 5944 1630 50  0000 C CNN
+F 1 "27k" V 5944 1630 50  0000 C CNN
 F 2 "Resistor_SMD:R_0603_1608Metric" V 5990 1630 50  0001 C CNN
 F 3 "~" H 6060 1630 50  0001 C CNN
@@
 P 6700 830
 F 0 "R36" H 6770 876 50  0000 L CNN
-F 1 "470" H 6770 785 50  0000 L CNN
+F 1 "1.8k" H 6770 785 50  0000 L CNN
 F 2 "Resistor_SMD:R_0603_1608Metric" V 6630 830 50  0001 C CNN
 F 3 "~" H 6700 830 50  0001 C CNN
@@
 P 6220 1940
 F 0 "R35" H 6150 1894 50  0000 R CNN
-F 1 "1k8" H 6150 1985 50  0000 R CNN
+F 1 "4.7k" H 6150 1985 50  0000 R CNN
 F 2 "Resistor_SMD:R_0603_1608Metric" V 6150 1940 50  0001 C CNN
 F 3 "~" H 6220 1940 50  0001 C CNN
@@
 P 8290 1640
 F 0 "R37" V 8083 1640 50  0000 C CNN
-F 1 "10k" V 8174 1640 50  0000 C CNN
+F 1 "27k" V 8174 1640 50  0000 C CNN
 F 2 "Resistor_SMD:R_0603_1608Metric" V 8220 1640 50  0001 C CNN
 F 3 "~" H 8290 1640 50  0001 C CNN
@@
 P 8930 840
 F 0 "R39" H 9000 886 50  0000 L CNN
-F 1 "470" H 9000 795 50  0000 L CNN
+F 1 "1.8k" H 9000 795 50  0000 L CNN
 F 2 "Resistor_SMD:R_0603_1608Metric" V 8860 840 50  0001 C CNN
 F 3 "~" H 8930 840 50  0001 C CNN
@@
 P 8450 1950
 F 0 "R38" H 8380 1904 50  0000 R CNN
-F 1 "1k8" H 8380 1995 50  0000 R CNN
+F 1 "4.7k" H 8380 1995 50  0000 R CNN
 F 2 "Resistor_SMD:R_0603_1608Metric" V 8380 1950 50  0001 C CNN
 F 3 "~" H 8450 1950 50  0001 C CNN
@@
 P 1620 3350
 F 0 "R40" V 1413 3350 50  0000 C CNN
-F 1 "10k" V 1504 3350 50  0000 C CNN
+F 1 "27k" V 1504 3350 50  0000 C CNN
 F 2 "Resistor_SMD:R_0603_1608Metric" V 1550 3350 50  0001 C CNN
 F 3 "~" H 1620 3350 50  0001 C CNN
@@
 P 2260 2550
 F 0 "R42" H 2330 2596 50  0000 L CNN
-F 1 "470" H 2330 2505 50  0000 L CNN
+F 1 "1.8k" H 2330 2505 50  0000 L CNN
 F 2 "Resistor_SMD:R_0603_1608Metric" V 2190 2550 50  0001 C CNN
 F 3 "~" H 2260 2550 50  0001 C CNN
@@
 P 1780 3660
 F 0 "R41" H 1710 3614 50  0000 R CNN
-F 1 "1k8" H 1710 3705 50  0000 R CNN
+F 1 "4.7k" H 1710 3705 50  0000 R CNN
 F 2 "Resistor_SMD:R_0603_1608Metric" V 1710 3660 50  0001 C CNN
 F 3 "~" H 1780 3660 50  0001 C CNN
@@
 P 3770 3330
 F 0 "R43" V 3563 3330 50  0000 C CNN
-F 1 "10k" V 3654 3330 50  0000 C CNN
+F 1 "27k" V 3654 3330 50  0000 C CNN
 F 2 "Resistor_SMD:R_0603_1608Metric" V 3700 3330 50  0001 C CNN
 F 3 "~" H 3770 3330 50  0001 C CNN
@@
 P 4410 2530
 F 0 "R45" H 4480 2576 50  0000 L CNN
-F 1 "470" H 4480 2485 50  0000 L CNN
+F 1 "1.8k" H 4480 2485 50  0000 L CNN
 F 2 "Resistor_SMD:R_0603_1608Metric" V 4340 2530 50  0001 C CNN
 F 3 "~" H 4410 2530 50  0001 C CNN
@@
 P 3930 3640
 F 0 "R44" H 3860 3594 50  0000 R CNN
-F 1 "1k8" H 3860 3685 50  0000 R CNN
+F 1 "4.7k" H 3860 3685 50  0000 R CNN
 F 2 "Resistor_SMD:R_0603_1608Metric" V 3860 3640 50  0001 C CNN
 F 3 "~" H 3930 3640 50  0001 C CNN
@@
 P 6010 3340
 F 0 "R46" V 5803 3340 50  0000 C CNN
-F 1 "10k" V 5894 3340 50  0000 C CNN
+F 1 "27k" V 5894 3340 50  0000 C CNN
 F 2 "Resistor_SMD:R_0603_1608Metric" V 5940 3340 50  0001 C CNN
 F 3 "~" H 6010 3340 50  0001 C CNN
@@
 P 6650 2540
 F 0 "R48" H 6720 2586 50  0000 L CNN
-F 1 "470" H 6720 2495 50  0000 L CNN
+F 1 "1.8k" H 6720 2495 50  0000 L CNN
 F 2 "Resistor_SMD:R_0603_1608Metric" V 6580 2540 50  0001 C CNN
 F 3 "~" H 6650 2540 50  0001 C CNN
@@
 P 6170 3650
 F 0 "R47" H 6100 3604 50  0000 R CNN
-F 1 "1k8" H 6100 3695 50  0000 R CNN
+F 1 "4.7k" H 6100 3695 50  0000 R CNN
 F 2 "Resistor_SMD:R_0603_1608Metric" V 6100 3650 50  0001 C CNN
 F 3 "~" H 6170 3650 50  0001 C CNN
@@
 P 8280 3340
 F 0 "R49" V 8073 3340 50  0000 C CNN
-F 1 "10k" V 8164 3340 50  0000 C CNN
+F 1 "27k" V 8164 3340 50  0000 C CNN
 F 2 "Resistor_SMD:R_0603_1608Metric" V 8210 3340 50  0001 C CNN
 F 3 "~" H 8280 3340 50  0001 C CNN
@@
 P 8920 2540
 F 0 "R51" H 8990 2586 50  0000 L CNN
-F 1 "470" H 8990 2495 50  0000 L CNN
+F 1 "1.8k" H 8990 2495 50  0000 L CNN
 F 2 "Resistor_SMD:R_0603_1608Metric" V 8850 2540 50  0001 C CNN
 F 3 "~" H 8920 2540 50  0001 C CNN
@@
 P 8440 3650
 F 0 "R50" H 8370 3604 50  0000 R CNN
-F 1 "1k8" H 8370 3695 50  0000 R CNN
+F 1 "4.7k" H 8370 3695 50  0000 R CNN
 F 2 "Resistor_SMD:R_0603_1608Metric" V 8370 3650 50  0001 C CNN
 F 3 "~" H 8440 3650 50  0001 C CNN

Commit message: Add BOM file and CPL file
Parts:
- D0, D1, D2, D3, D4, D5, D6, D7: LCSC (none) -> C72043
- Q10, Q11, Q12, Q13, Q14, Q15, Q8, Q9: LCSC (none) -> C8659
- R28, R31, R34, R37, R40, R43, R46, R49: LCSC (none) -> C25589
- R29, R32, R35, R38, R41, R44, R47, R50: LCSC (none) -> C105428
- R30, R33, R36, R39, R42, R45, R48, R51: LCSC (none) -> C103360
- R52, R53, R54, R55, R56: LCSC (none) -> C98220
- U4: LCSC (none) -> C6796

Commit message: Update LED footprint
Parts:
- R29, R32, R35, R38, R41, R44, R47, R50: LCSC C105428 -> C23162
- U4: value 74LS04 -> 74HC04; LCSC C6796 -> C5590
Changed lines of the file:
@@
 P 3540 5550
 F 0 "U4" H 3540 5867 50  0000 C CNN
-F 1 "74LS04" H 3540 5776 50  0000 C CNN
+F 1 "74HC04" H 3540 5776 50  0000 C CNN
 F 2 "Package_SO:SOIC-14_3.9x8.7mm_P1.27mm" H 3540 5550 50  0001 C CNN
 F 3 "http://www.ti.com/lit/gpn/sn74LS04" H 3540 5550 50  0001 C CNN
-F 4 "C6796" H 3540 5550 50  0001 C CNN "LCSC"
+F 4 "C5590" H 3540 5550 50  0001 C CNN "LCSC"
 	1    3540 5550
 	1    0    0    -1
@@
 P 6830 5070
 F 0 "U4" H 7060 5116 50  0000 L CNN
-F 1 "74LS04" H 7060 5025 50  0000 L CNN
+F 1 "74HC04" H 7060 5025 50  0000 L CNN
 F 2 "Package_SO:SOIC-14_3.9x8.7mm_P1.27mm" H 6830 5070 50  0001 C CNN
 F 3 "http://www.ti.com/lit/gpn/sn74LS04" H 6830 5070 50  0001 C CNN
-F 4 "C6796" H 6830 5070 50  0001 C CNN "LCSC"
+F 4 "C5590" H 6830 5070 50  0001 C CNN "LCSC"
 	7    6830 5070
 	1    0    0    -1
@@
 F 2 "Resistor_SMD:R_0603_1608Metric" V 1700 1960 50  0001 C CNN
 F 3 "~" H 1770 1960 50  0001 C CNN
-F 4 "C105428" H 1770 1960 50  0001 C CNN "LCSC"
+F 4 "C23162" H 1770 1960 50  0001 C CNN "LCSC"
 	1    1770 1960
 	-1   0    0    1
@@
 F 2 "Resistor_SMD:R_0603_1608Metric" V 3850 1940 50  0001 C CNN
 F 3 "~" H 3920 1940 50  0001 C CNN
-F 4 "C105428" H 3920 1940 50  0001 C CNN "LCSC"
+F 4 "C23162" H 3920 1940 50  0001 C CNN "LCSC"
 	1    3920 1940
 	-1   0    0    1
@@
 F 2 "Resistor_SMD:R_0603_1608Metric" V 6150 1940 50  0001 C CNN
 F 3 "~" H 6220 1940 50  0001 C CNN
-F 4 "C105428" H 6220 1940 50  0001 C CNN "LCSC"
+F 4 "C23162" H 6220 1940 50  0001 C CNN "LCSC"
 	1    6220 1940
 	-1   0    0    1
@@
 F 2 "Resistor_SMD:R_0603_1608Metric" V 8380 1950 50  0001 C CNN
 F 3 "~" H 8450 1950 50  0001 C CNN
-F 4 "C105428" H 8450 1950 50  0001 C CNN "LCSC"
+F 4 "C23162" H 8450 1950 50  0001 C CNN "LCSC"
 	1    8450 1950
 	-1   0    0    1
@@
 F 2 "Resistor_SMD:R_0603_1608Metric" V 1710 3660 50  0001 C CNN
 F 3 "~" H 1780 3660 50  0001 C CNN
-F 4 "C105428" H 1780 3660 50  0001 C CNN "LCSC"
+F 4 "C23162" H 1780 3660 50  0001 C CNN "LCSC"
 	1    1780 3660
 	-1   0    0    1
@@
 F 2 "Resistor_SMD:R_0603_1608Metric" V 3860 3640 50  0001 C CNN
 F 3 "~" H 3930 3640 50  0001 C CNN
-F 4 "C105428" H 3930 3640 50  0001 C CNN "LCSC"
+F 4 "C23162" H 3930 3640 50  0001 C CNN "LCSC"
 	1    3930 3640
 	-1   0    0    1
@@
 F 2 "Resistor_SMD:R_0603_1608Metric" V 6100 3650 50  0001 C CNN
 F 3 "~" H 6170 3650 50  0001 C CNN
-F 4 "C105428" H 6170 3650 50  0001 C CNN "LCSC"
+F 4 "C23162" H 6170 3650 50  0001 C CNN "LCSC"
 	1    6170 3650
 	-1   0    0    1
@@
 F 2 "Resistor_SMD:R_0603_1608Metric" V 8370 3650 50  0001 C CNN
 F 3 "~" H 8440 3650 50  0001 C CNN
-F 4 "C105428" H 8440 3650 50  0001 C CNN "LCSC"
+F 4 "C23162" H 8440 3650 50  0001 C CNN "LCSC"
 	1    8440 3650
 	-1   0    0    1
