File: digitalSystemBoard/Header.sch (KiCad schematic (older format))
At the start: 0 parts

Commit message: Update Schematic for review
Parts:
- added J10, J11, J12: Conn_02x03_Odd_Even, symbol Connector_Generic:Conn_02x03_Odd_Even
- added J3, J5: Conn_02x04_Odd_Even, symbol Connector_Generic:Conn_02x04_Odd_Even
- added J4, J6: Conn_02x07_Odd_Even, symbol Connector_Generic:Conn_02x07_Odd_Even
- added J7, J8: Conn_02x08_Odd_Even, symbol Connector_Generic:Conn_02x08_Odd_Even
- added J9: Conn_02x02_Odd_Even, symbol Connector_Generic:Conn_02x02_Odd_Even
Connections:
- new net CLK_OUT: J10.1 (Pin_1), J10.2 (Pin_2), J10.3 (Pin_3), J10.4 (Pin_4), J10.5 (Pin_5), J10.6 (Pin_6)
- new net GND: J12.1 (Pin_1), J12.2 (Pin_2), J12.3 (Pin_3), J12.4 (Pin_4), J12.5 (Pin_5), J12.6 (Pin_6)
- new net GPIO_BCD_A_0: J3.1 (Pin_1), J3.2 (Pin_2)
- new net GPIO_BCD_A_1: J5.1 (Pin_1), J5.2 (Pin_2)
- new net GPIO_BCD_B_0: J3.3 (Pin_3), J3.4 (Pin_4)
- new net GPIO_BCD_B_1: J5.3 (Pin_3), J5.4 (Pin_4)
- new net GPIO_BCD_C_0: J3.5 (Pin_5), J3.6 (Pin_6)
- new net GPIO_BCD_C_1: J5.5 (Pin_5), J5.6 (Pin_6)
- new net GPIO_BCD_D_0: J3.7 (Pin_7), J3.8 (Pin_8)
- new net GPIO_BCD_D_1: J5.7 (Pin_7), J5.8 (Pin_8)
- new net GPIO_LED_1: J7.1 (Pin_1), J7.2 (Pin_2)
- new net GPIO_LED_2: J7.3 (Pin_3), J7.4 (Pin_4)
- new net GPIO_LED_3: J7.5 (Pin_5), J7.6 (Pin_6)
- new net GPIO_LED_4: J7.7 (Pin_7), J7.8 (Pin_8)
- new net GPIO_LED_5: J7.10 (Pin_10), J7.9 (Pin_9)
- new net GPIO_LED_6: J7.11 (Pin_11), J7.12 (Pin_12)
- new net GPIO_LED_7: J7.13 (Pin_13), J7.14 (Pin_14)
- new net GPIO_LED_8: J7.15 (Pin_15), J7.16 (Pin_16)
- new net KEY0: J9.1 (Pin_1), J9.2 (Pin_2)
- new net KEY1: J9.3 (Pin_3), J9.4 (Pin_4)
- new net SEG_A_0: J4.1 (Pin_1), J4.2 (Pin_2)
- new net SEG_A_1: J6.1 (Pin_1), J6.2 (Pin_2)
- new net SEG_B_0: J4.3 (Pin_3), J4.4 (Pin_4)
- new net SEG_B_1: J6.3 (Pin_3), J6.4 (Pin_4)
- new net SEG_C_0: J4.5 (Pin_5), J4.6 (Pin_6)
- new net SEG_C_1: J6.5 (Pin_5), J6.6 (Pin_6)
- new net SEG_D_0: J4.7 (Pin_7), J4.8 (Pin_8)
- new net SEG_D_1: J6.7 (Pin_7), J6.8 (Pin_8)
- new net SEG_E_0: J4.10 (Pin_10), J4.9 (Pin_9)
- new net SEG_E_1: J6.10 (Pin_10), J6.9 (Pin_9)
- new net SEG_F_0: J4.11 (Pin_11), J4.12 (Pin_12)
- new net SEG_F_1: J6.11 (Pin_11), J6.12 (Pin_12)
- new net SEG_G_0: J4.13 (Pin_13), J4.14 (Pin_14)
- new net SEG_G_1: J6.13 (Pin_13), J6.14 (Pin_14)
- new net SW1: J8.1 (Pin_1), J8.2 (Pin_2)
- new net SW2: J8.3 (Pin_3), J8.4 (Pin_4)
- new net SW3: J8.5 (Pin_5), J8.6 (Pin_6)
- new net SW4: J8.7 (Pin_7), J8.8 (Pin_8)
- new net SW5: J8.10 (Pin_10), J8.9 (Pin_9)
- new net SW6: J8.11 (Pin_11), J8.12 (Pin_12)
- new net SW7: J8.13 (Pin_13), J8.14 (Pin_14)
- new net SW8: J8.15 (Pin_15), J8.16 (Pin_16)
- new net VCC5V: J11.1 (Pin_1), J11.2 (Pin_2), J11.3 (Pin_3), J11.4 (Pin_4), J11.5 (Pin_5), J11.6 (Pin_6)

Commit message: Add footprint
Parts:
- J10, J11, J12: footprint (none) -> Connector_PinHeader_2.54mm:PinHeader_2x03_P2.54mm_Vertical_SMD
- J3: footprint (none) -> Connector_IDC:IDC-Header_2x04_P2.54mm_Vertical
- J4: footprint (none) -> Connector_IDC:IDC-Header_2x07_P2.54mm_Vertical
- J5: footprint (none) -> Connector_PinHeader_2.54mm:PinHeader_2x04_P2.54mm_Vertical_SMD
- J6: footprint (none) -> Connector_PinHeader_2.54mm:PinHeader_2x07_P2.54mm_Vertical_SMD
- J7, J8: footprint (none) -> Connector_PinHeader_2.54mm:PinHeader_2x08_P2.54mm_Vertical_SMD
- J9: footprint (none) -> Connector_PinHeader_2.54mm:PinHeader_2x02_P2.54mm_Vertical_SMD
Changed lines of the file:
@@
 F 0 "J3" H 2250 2417 50  0000 C CNN
 F 1 "Conn_02x04_Odd_Even" H 2250 2326 50  0000 C CNN
-F 2 "" H 2200 2100 50  0001 C CNN
+F 2 "Connector_IDC:IDC-Header_2x04_P2.54mm_Vertical" H 2200 2100 50  0001 C CNN
 F 3 "~" H 2200 2100 50  0001 C CNN
 	1    2200 2100
@@
 F 0 "J5" H 4050 2417 50  0000 C CNN
 F 1 "Conn_02x04_Odd_Even" H 4050 2326 50  0000 C CNN
-F 2 "" H 4000 2100 50  0001 C CNN
+F 2 "Connector_PinHeader_2.54mm:PinHeader_2x04_P2.54mm_Vertical_SMD" H 4000 2100 50  0001 C CNN
 F 3 "~" H 4000 2100 50  0001 C CNN
 	1    4000 2100
@@
 F 0 "J8" H 2250 6817 50  0000 C CNN
 F 1 "Conn_02x08_Odd_Even" H 2250 6726 50  0000 C CNN
-F 2 "" H 2200 6300 50  0001 C CNN
+F 2 "Connector_PinHeader_2.54mm:PinHeader_2x08_P2.54mm_Vertical_SMD" H 2200 6300 50  0001 C CNN
 F 3 "~" H 2200 6300 50  0001 C CNN
 	1    2200 6300
@@
 F 0 "J10" H 9760 2417 50  0000 C CNN
 F 1 "Conn_02x03_Odd_Even" H 9760 2326 50  0000 C CNN
-F 2 "" H 9710 2100 50  0001 C CNN
+F 2 "Connector_PinHeader_2.54mm:PinHeader_2x03_P2.54mm_Vertical_SMD" H 9710 2100 50  0001 C CNN
 F 3 "~" H 9710 2100 50  0001 C CNN
 	1    9710 2100
@@
 F 0 "J4" H 2250 4417 50  0000 C CNN
 F 1 "Conn_02x07_Odd_Even" H 2250 4326 50  0000 C CNN
-F 2 "" H 2200 3900 50  0001 C CNN
+F 2 "Connector_IDC:IDC-Header_2x07_P2.54mm_Vertical" H 2200 3900 50  0001 C CNN
 F 3 "~" H 2200 3900 50  0001 C CNN
 	1    2200 3900
@@
 F 0 "J6" H 4050 4417 50  0000 C CNN
 F 1 "Conn_02x07_Odd_Even" H 4050 4326 50  0000 C CNN
-F 2 "" H 4000 3900 50  0001 C CNN
+F 2 "Connector_PinHeader_2.54mm:PinHeader_2x07_P2.54mm_Vertical_SMD" H 4000 3900 50  0001 C CNN
 F 3 "~" H 4000 3900 50  0001 C CNN
 	1    4000 3900
@@
 F 0 "J9" H 3950 6217 50  0000 C CNN
 F 1 "Conn_02x02_Odd_Even" H 3950 6126 50  0000 C CNN
-F 2 "" H 3900 6000 50  0001 C CNN
+F 2 "Connector_PinHeader_2.54mm:PinHeader_2x02_P2.54mm_Vertical_SMD" H 3900 6000 50  0001 C CNN
 F 3 "~" H 3900 6000 50  0001 C CNN
 	1    3900 6000
@@
 F 0 "J7" H 6150 2817 50  0000 C CNN
 F 1 "Conn_02x08_Odd_Even" H 6150 2726 50  0000 C CNN
-F 2 "" H 6100 2300 50  0001 C CNN
+F 2 "Connector_PinHeader_2.54mm:PinHeader_2x08_P2.54mm_Vertical_SMD" H 6100 2300 50  0001 C CNN
 F 3 "~" H 6100 2300 50  0001 C CNN
 	1    6100 2300
@@
 F 0 "J11" H 8250 4417 50  0000 C CNN
 F 1 "Conn_02x03_Odd_Even" H 8250 4326 50  0000 C CNN
-F 2 "" H 8200 4100 50  0001 C CNN
+F 2 "Connector_PinHeader_2.54mm:PinHeader_2x03_P2.54mm_Vertical_SMD" H 8200 4100 50  0001 C CNN
 F 3 "~" H 8200 4100 50  0001 C CNN
 	1    8200 4100
@@
 F 0 "J12" H 8250 5417 50  0000 C CNN
 F 1 "Conn_02x03_Odd_Even" H 8250 5326 50  0000 C CNN
-F 2 "" H 8200 5100 50  0001 C CNN
+F 2 "Connector_PinHeader_2.54mm:PinHeader_2x03_P2.54mm_Vertical_SMD" H 8200 5100 50  0001 C CNN
 F 3 "~" H 8200 5100 50  0001 C CNN
 	1    8200 5100
