File: digitalSystemBoard/Header_and_Mounting.sch (KiCad schematic (older format))
At the start: 10 parts, among them J10 Conn_02x03_Odd_Even, J11 Conn_02x03_Odd_Even, J12 Conn_02x03_Odd_Even, J3 Conn_02x04_Odd_Even, J4 Conn_02x07_Odd_Even, J5 Conn_02x04_Odd_Even, J6 Conn_02x07_Odd_Even, J7 Conn_02x08_Odd_Even, J8 Conn_02x08_Odd_Even, J9 Conn_02x03_Odd_Even

Commit message: Add full footprint. Draw layout board
Parts:
- added H0, H1, H2, H3: MountingHole, digitalSystemBoard:Mountinghole_M3, symbol Mechanical:MountingHole
- renumbered J5 to J4, J7 to J5, J4 to J6, J6 to J7
Other:
- moved on the sheet: J11, J12
Changed lines of the file:
@@
 $EndComp
 $Comp
-L Connector_Generic:Conn_02x04_Odd_Even J5
+L Connector_Generic:Conn_02x04_Odd_Even J4
 U 1 1 5FC88FC0
 P 4000 2100
-F 0 "J5" H 4050 2417 50  0000 C CNN
+F 0 "J4" H 4050 2417 50  0000 C CNN
 F 1 "Conn_02x04_Odd_Even" H 4050 2326 50  0000 C CNN
 F 2 "digitalSystemBoard:DC3_2x04_PIN" H 4000 2100 50  0001 C CNN
@@
 $EndComp
 $Comp
-L Connector_Generic:Conn_02x07_Odd_Even J4
+L Connector_Generic:Conn_02x07_Odd_Even J6
 U 1 1 5FC928BF
 P 2200 3900
-F 0 "J4" H 2250 4417 50  0000 C CNN
+F 0 "J6" H 2250 4417 50  0000 C CNN
 F 1 "Conn_02x07_Odd_Even" H 2250 4326 50  0000 C CNN
 F 2 "digitalSystemBoard:DC3_2x07_PIN" H 2200 3900 50  0001 C CNN
@@
 $EndComp
 $Comp
-L Connector_Generic:Conn_02x07_Odd_Even J6
+L Connector_Generic:Conn_02x07_Odd_Even J7
 U 1 1 5FC93EAD
 P 4000 3900
-F 0 "J6" H 4050 4417 50  0000 C CNN
+F 0 "J7" H 4050 4417 50  0000 C CNN
 F 1 "Conn_02x07_Odd_Even" H 4050 4326 50  0000 C CNN
 F 2 "digitalSystemBoard:DC3_2x07_PIN" H 4000 3900 50  0001 C CNN
@@
 GPIO_LED_1
 $Comp
-L Connector_Generic:Conn_02x08_Odd_Even J7
+L Connector_Generic:Conn_02x08_Odd_Even J5
 U 1 1 5FC8A515
 P 6100 2300
-F 0 "J7" H 6150 2817 50  0000 C CNN
+F 0 "J5" H 6150 2817 50  0000 C CNN
 F 1 "Conn_02x08_Odd_Even" H 6150 2726 50  0000 C CNN
 F 2 "digitalSystemBoard:DC3_2x08_PIN" H 6100 2300 50  0001 C CNN
@@
 L Connector_Generic:Conn_02x03_Odd_Even J11
 U 1 1 5FD1AE53
-P 8200 4100
-F 0 "J11" H 8250 4417 50  0000 C CNN
-F 1 "Conn_02x03_Odd_Even" H 8250 4326 50  0000 C CNN
-F 2 "digitalSystemBoard:DC3_2x03_PIN" H 8200 4100 50  0001 C CNN
-F 3 "~" H 8200 4100 50  0001 C CNN
-	1    8200 4100
+P 6930 4850
+F 0 "J11" H 6980 5167 50  0000 C CNN
+F 1 "Conn_02x03_Odd_Even" H 6980 5076 50  0000 C CNN
+F 2 "digitalSystemBoard:DC3_2x03_PIN" H 6930 4850 50  0001 C CNN
+F 3 "~" H 6930 4850 50  0001 C CNN
+	1    6930 4850
 	1    0    0    -1
 $EndComp
@@
 L Connector_Generic:Conn_02x03_Odd_Even J12
 U 1 1 5FD1B6CA
-P 8200 5100
-F 0 "J12" H 8250 5417 50  0000 C CNN
-F 1 "Conn_02x03_Odd_Even" H 8250 5326 50  0000 C CNN
-F 2 "digitalSystemBoard:DC3_2x03_PIN" H 8200 5100 50  0001 C CNN
-F 3 "~" H 8200 5100 50  0001 C CNN
-	1    8200 5100
-	1    0    0    -1
-$EndComp
-Text HLabel 8000 4000 0    50   Input ~ 0
-VCC5V
-Text HLabel 8000 4100 0    50   Input ~ 0
-VCC5V
-Text HLabel 8000 4200 0    50   Input ~ 0
-VCC5V
-Text HLabel 8500 4200 2    50   Input ~ 0
-VCC5V
-Text HLabel 8500 4100 2    50   Input ~ 0
-VCC5V
-Text HLabel 8500 4000 2    50   Input ~ 0
+P 6930 5850
+F 0 "J12" H 6980 6167 50  0000 C CNN
+F 1 "Conn_02x03_Odd_Even" H 6980 6076 50  0000 C CNN
+F 2 "digitalSystemBoard:DC3_2x03_PIN" H 6930 5850 50  0001 C CNN
+F 3 "~" H 6930 5850 50  0001 C CNN
+	1    6930 5850
+	1    0    0    -1
+$EndComp
+Text HLabel 6730 4750 0    50   Input ~ 0
+VCC5V
+Text HLabel 6730 4850 0    50   Input ~ 0
+VCC5V
+Text HLabel 6730 4950 0    50   Input ~ 0
+VCC5V
+Text HLabel 7230 4950 2    50   Input ~ 0
+VCC5V
+Text HLabel 7230 4850 2    50   Input ~ 0
+VCC5V
+Text HLabel 7230 4750 2    50   Input ~ 0
 VCC5V
 $Comp
 L power:GND #PWR0106
 U 1 1 5FD2ED5A
-P 8000 5000
-F 0 "#PWR0106" H 8000 4750 50  0001 C CNN
-F 1 "GND" V 8005 4872 50  0000 R CNN
-F 2 "" H 8000 5000 50  0001 C CNN
-F 3 "" H 8000 5000 50  0001 C CNN
-	1    8000 5000
+P 6730 5750
+F 0 "#PWR0106" H 6730 5500 50  0001 C CNN
+F 1 "GND" V 6735 5622 50  0000 R CNN
+F 2 "" H 6730 5750 50  0001 C CNN
+F 3 "" H 6730 5750 50  0001 C CNN
+	1    6730 5750
 	0    1    1    0
 $EndComp
@@
 L power:GND #PWR0146
 U 1 1 5FD2F2EC
-P 8000 5100
-F 0 "#PWR0146" H 8000 4850 50  0001 C CNN
-F 1 "GND" V 8005 4972 50  0000 R CNN
-F 2 "" H 8000 5100 50  0001 C CNN
-F 3 "" H 8000 5100 50  0001 C CNN
-	1    8000 5100
+P 6730 5850
+F 0 "#PWR0146" H 6730 5600 50  0001 C CNN
+F 1 "GND" V 6735 5722 50  0000 R CNN
+F 2 "" H 6730 5850 50  0001 C CNN
+F 3 "" H 6730 5850 50  0001 C CNN
+	1    6730 5850
 	0    1    1    0
 $EndComp
@@
 L power:GND #PWR0147
 U 1 1 5FD2F922
-P 8000 5200
-F 0 "#PWR0147" H 8000 4950 50  0001 C CNN
-F 1 "GND" V 8005 5072 50  0000 R CNN
-F 2 "" H 8000 5200 50  0001 C CNN
-F 3 "" H 8000 5200 50  0001 C CNN
-	1    8000 5200
+P 6730 5950
+F 0 "#PWR0147" H 6730 5700 50  0001 C CNN
+F 1 "GND" V 6735 5822 50  0000 R CNN
+F 2 "" H 6730 5950 50  0001 C CNN
+F 3 "" H 6730 5950 50  0001 C CNN
+	1    6730 5950
 	0    1    1    0
 $EndComp
@@
 L power:GND #PWR0148
 U 1 1 5FD31990
-P 8500 5200
-F 0 "#PWR0148" H 8500 4950 50  0001 C CNN
-F 1 "GND" V 8505 5072 50  0000 R CNN
-F 2 "" H 8500 5200 50  0001 C CNN
-F 3 "" H 8500 5200 50  0001 C CNN
-	1    8500 5200
+P 7230 5950
+F 0 "#PWR0148" H 7230 5700 50  0001 C CNN
+F 1 "GND" V 7235 5822 50  0000 R CNN
+F 2 "" H 7230 5950 50  0001 C CNN
+F 3 "" H 7230 5950 50  0001 C CNN
+	1    7230 5950
 	0    -1   -1   0
 $EndComp
@@
 L power:GND #PWR0149
 U 1 1 5FD31996
-P 8500 5100
-F 0 "#PWR0149" H 8500 4850 50  0001 C CNN
-F 1 "GND" V 8505 4972 50  0000 R CNN
-F 2 "" H 8500 5100 50  0001 C CNN
-F 3 "" H 8500 5100 50  0001 C CNN
-	1    8500 5100
+P 7230 5850
+F 0 "#PWR0149" H 7230 5600 50  0001 C CNN
+F 1 "GND" V 7235 5722 50  0000 R CNN
+F 2 "" H 7230 5850 50  0001 C CNN
+F 3 "" H 7230 5850 50  0001 C CNN
+	1    7230 5850
 	0    -1   -1   0
 $EndComp
@@
 L power:GND #PWR0157
 U 1 1 5FD3199C
-P 8500 5000
-F 0 "#PWR0157" H 8500 4750 50  0001 C CNN
-F 1 "GND" V 8505 4872 50  0000 R CNN
-F 2 "" H 8500 5000 50  0001 C CNN
-F 3 "" H 8500 5000 50  0001 C CNN
-	1    8500 5000
+P 7230 5750
+F 0 "#PWR0157" H 7230 5500 50  0001 C CNN
+F 1 "GND" V 7235 5622 50  0000 R CNN
+F 2 "" H 7230 5750 50  0001 C CNN
+F 3 "" H 7230 5750 50  0001 C CNN
+	1    7230 5750
 	0    -1   -1   0
 $EndComp
@@
 	1    0    0    -1
 $EndComp
+$Comp
+L Mechanical:MountingHole H1
+U 1 1 5FCEEBC4
+P 10000 4000
+F 0 "H1" H 10100 4046 50  0000 L CNN
+F 1 "MountingHole" H 10100 3955 50  0000 L CNN
+F 2 "digitalSystemBoard:Mountinghole_M3" H 10000 4000 50  0001 C CNN
+F 3 "~" H 10000 4000 50  0001 C CNN
+	1    10000 4000
+	1    0    0    -1
+$EndComp
+$Comp
+L Mechanical:MountingHole H3
+U 1 1 5FCEF50C
+P 10000 5000
+F 0 "H3" H 10100 5046 50  0000 L CNN
+F 1 "MountingHole" H 10100 4955 50  0000 L CNN
+F 2 "digitalSystemBoard:Mountinghole_M3" H 10000 5000 50  0001 C CNN
+F 3 "~" H 10000 5000 50  0001 C CNN
+	1    10000 5000
+	1    0    0    -1
+$EndComp
+$Comp
+L Mechanical:MountingHole H0
+U 1 1 5FCF2F5D
+P 9000 4000
+F 0 "H0" H 9100 4046 50  0000 L CNN
+F 1 "MountingHole" H 9100 3955 50  0000 L CNN
+F 2 "digitalSystemBoard:Mountinghole_M3" H 9000 4000 50  0001 C CNN
+F 3 "~" H 9000 4000 50  0001 C CNN
+	1    9000 4000
+	1    0    0    -1
+$EndComp
+$Comp
+L Mechanical:MountingHole H2
+U 1 1 5FCF37FA
+P 9000 5000
+F 0 "H2" H 9100 5046 50  0000 L CNN
+F 1 "MountingHole" H 9100 4955 50  0000 L CNN
+F 2 "digitalSystemBoard:Mountinghole_M3" H 9000 5000 50  0001 C CNN
+F 3 "~" H 9000 5000 50  0001 C CNN
+	1    9000 5000
+	1    0    0    -1
+$EndComp

Commit message: Update layout
Parts:
- J10, J11, J12, J9: footprint digitalSystemBoard:DC3_2x03_PIN -> Connector_IDC:IDC-Header_2x03_P2.54mm_Vertical
- J3, J4: footprint digitalSystemBoard:DC3_2x04_PIN -> Connector_IDC:IDC-Header_2x04_P2.54mm_Vertical
- J5, J8: footprint digitalSystemBoard:DC3_2x08_PIN -> Connector_IDC:IDC-Header_2x08_P2.54mm_Vertical
- J6, J7: footprint digitalSystemBoard:DC3_2x07_PIN -> Connector_IDC:IDC-Header_2x07_P2.54mm_Vertical
Connections:
- net GPIO_BCD_A_0: now also J3.7 (Pin_7), J3.8 (Pin_8); no longer J3.1 (Pin_1), J3.2 (Pin_2)
- net GPIO_BCD_A_1: now also J4.7 (Pin_7), J4.8 (Pin_8); no longer J4.1 (Pin_1), J4.2 (Pin_2)
- net GPIO_BCD_B_0: now also J3.5 (Pin_5), J3.6 (Pin_6); no longer J3.3 (Pin_3), J3.4 (Pin_4)
- net GPIO_BCD_B_1: now also J4.5 (Pin_5), J4.6 (Pin_6); no longer J4.3 (Pin_3), J4.4 (Pin_4)
- net GPIO_BCD_C_0: now also J3.3 (Pin_3), J3.4 (Pin_4); no longer J3.5 (Pin_5), J3.6 (Pin_6)
- net GPIO_BCD_C_1: now also J4.3 (Pin_3), J4.4 (Pin_4); no longer J4.5 (Pin_5), J4.6 (Pin_6)
- net GPIO_BCD_D_0: now also J3.1 (Pin_1), J3.2 (Pin_2); no longer J3.7 (Pin_7), J3.8 (Pin_8)
- net GPIO_BCD_D_1: now also J4.1 (Pin_1), J4.2 (Pin_2); no longer J4.7 (Pin_7), J4.8 (Pin_8)
- net KEY0: now also J9.5 (Pin_5), J9.6 (Pin_6); no longer J9.1 (Pin_1), J9.2 (Pin_2)
- net SW1: now also J8.15 (Pin_15), J8.16 (Pin_16); no longer J8.1 (Pin_1), J8.2 (Pin_2)
- net SW2: now also J8.13 (Pin_13), J8.14 (Pin_14); no longer J8.3 (Pin_3), J8.4 (Pin_4)
- net SW3: now also J8.11 (Pin_11), J8.12 (Pin_12); no longer J8.5 (Pin_5), J8.6 (Pin_6)
- net SW4: now also J8.10 (Pin_10), J8.9 (Pin_9); no longer J8.7 (Pin_7), J8.8 (Pin_8)
- net SW5: now also J8.7 (Pin_7), J8.8 (Pin_8); no longer J8.10 (Pin_10), J8.9 (Pin_9)
- net SW6: now also J8.5 (Pin_5), J8.6 (Pin_6); no longer J8.11 (Pin_11), J8.12 (Pin_12)
- net SW7: now also J8.3 (Pin_3), J8.4 (Pin_4); no longer J8.13 (Pin_13), J8.14 (Pin_14)
- net SW8: now also J8.1 (Pin_1), J8.2 (Pin_2); no longer J8.15 (Pin_15), J8.16 (Pin_16)
Changed lines of the file:
@@
 L Connector_Generic:Conn_02x04_Odd_Even J3
 U 1 1 5FC86773
-P 2200 2100
-F 0 "J3" H 2250 2417 50  0000 C CNN
-F 1 "Conn_02x04_Odd_Even" H 2250 2326 50  0000 C CNN
-F 2 "digitalSystemBoard:DC3_2x04_PIN" H 2200 2100 50  0001 C CNN
-F 3 "~" H 2200 2100 50  0001 C CNN
-	1    2200 2100
-	1    0    0    -1
+P 2300 2200
+F 0 "J3" H 2350 2517 50  0000 C CNN
+F 1 "Conn_02x04_Odd_Even" H 2350 2426 50  0000 C CNN
+F 2 "Connector_IDC:IDC-Header_2x04_P2.54mm_Vertical" H 2300 2200 50  0001 C CNN
+F 3 "~" H 2300 2200 50  0001 C CNN
+	1    2300 2200
+	-1   0    0    1
 $EndComp
 $Comp
 L Connector_Generic:Conn_02x04_Odd_Even J4
 U 1 1 5FC88FC0
-P 4000 2100
-F 0 "J4" H 4050 2417 50  0000 C CNN
-F 1 "Conn_02x04_Odd_Even" H 4050 2326 50  0000 C CNN
-F 2 "digitalSystemBoard:DC3_2x04_PIN" H 4000 2100 50  0001 C CNN
-F 3 "~" H 4000 2100 50  0001 C CNN
-	1    4000 2100
-	1    0    0    -1
-$EndComp
-$Comp
-L Connector_Generic:Conn_02x08_Odd_Even J8
-U 1 1 5FC8D8A2
-P 2200 6300
-F 0 "J8" H 2250 6817 50  0000 C CNN
-F 1 "Conn_02x08_Odd_Even" H 2250 6726 50  0000 C CNN
-F 2 "digitalSystemBoard:DC3_2x08_PIN" H 2200 6300 50  0001 C CNN
-F 3 "~" H 2200 6300 50  0001 C CNN
-	1    2200 6300
-	1    0    0    -1
+P 4100 2200
+F 0 "J4" H 4150 2517 50  0000 C CNN
+F 1 "Conn_02x04_Odd_Even" H 4150 2426 50  0000 C CNN
+F 2 "Connector_IDC:IDC-Header_2x04_P2.54mm_Vertical" H 4100 2200 50  0001 C CNN
+F 3 "~" H 4100 2200 50  0001 C CNN
+	1    4100 2200
+	-1   0    0    1
 $EndComp
 $Comp
@@
 F 0 "J10" H 9760 2417 50  0000 C CNN
 F 1 "Conn_02x03_Odd_Even" H 9760 2326 50  0000 C CNN
-F 2 "digitalSystemBoard:DC3_2x03_PIN" H 9710 2100 50  0001 C CNN
+F 2 "Connector_IDC:IDC-Header_2x03_P2.54mm_Vertical" H 9710 2100 50  0001 C CNN
 F 3 "~" H 9710 2100 50  0001 C CNN
 	1    9710 2100
@@
 F 0 "J6" H 2250 4417 50  0000 C CNN
 F 1 "Conn_02x07_Odd_Even" H 2250 4326 50  0000 C CNN
-F 2 "digitalSystemBoard:DC3_2x07_PIN" H 2200 3900 50  0001 C CNN
+F 2 "Connector_IDC:IDC-Header_2x07_P2.54mm_Vertical" H 2200 3900 50  0001 C CNN
 F 3 "~" H 2200 3900 50  0001 C CNN
 	1    2200 3900
@@
 F 0 "J7" H 4050 4417 50  0000 C CNN
 F 1 "Conn_02x07_Odd_Even" H 4050 4326 50  0000 C CNN
-F 2 "digitalSystemBoard:DC3_2x07_PIN" H 4000 3900 50  0001 C CNN
+F 2 "Connector_IDC:IDC-Header_2x07_P2.54mm_Vertical" H 4000 3900 50  0001 C CNN
 F 3 "~" H 4000 3900 50  0001 C CNN
 	1    4000 3900
@@
 F 0 "J5" H 6150 2817 50  0000 C CNN
 F 1 "Conn_02x08_Odd_Even" H 6150 2726 50  0000 C CNN
-F 2 "digitalSystemBoard:DC3_2x08_PIN" H 6100 2300 50  0001 C CNN
+F 2 "Connector_IDC:IDC-Header_2x08_P2.54mm_Vertical" H 6100 2300 50  0001 C CNN
 F 3 "~" H 6100 2300 50  0001 C CNN
 	1    6100 2300
@@
 Text HLabel 3800 4200 0    50   Input ~ 0
 SEG_G_1
-Text HLabel 2000 6000 0    50   Input ~ 0
-SW1
-Text HLabel 2000 6100 0    50   Input ~ 0
-SW2
-Text HLabel 2000 6200 0    50   Input ~ 0
-SW3
-Text HLabel 2000 6300 0    50   Input ~ 0
-SW4
-Text HLabel 2000 6400 0    50   Input ~ 0
-SW5
-Text HLabel 2000 6500 0    50   Input ~ 0
-SW6
-Text HLabel 2000 6600 0    50   Input ~ 0
-SW7
-Text HLabel 2000 6700 0    50   Input ~ 0
-SW8
-Text HLabel 2500 6000 2    50   Input ~ 0
-SW1
-Text HLabel 2500 6100 2    50   Input ~ 0
-SW2
-Text HLabel 2500 6200 2    50   Input ~ 0
-SW3
-Text HLabel 2500 6300 2    50   Input ~ 0
-SW4
-Text HLabel 2500 6400 2    50   Input ~ 0
-SW5
-Text HLabel 2500 6500 2    50   Input ~ 0
-SW6
-Text HLabel 2500 6600 2    50   Input ~ 0
-SW7
-Text HLabel 2500 6700 2    50   Input ~ 0
-SW8
 Text HLabel 3700 6000 0    50   Input ~ 0
 KEY0
@@
 F 0 "J11" H 6980 5167 50  0000 C CNN
 F 1 "Conn_02x03_Odd_Even" H 6980 5076 50  0000 C CNN
-F 2 "digitalSystemBoard:DC3_2x03_PIN" H 6930 4850 50  0001 C CNN
+F 2 "Connector_IDC:IDC-Header_2x03_P2.54mm_Vertical" H 6930 4850 50  0001 C CNN
 F 3 "~" H 6930 4850 50  0001 C CNN
 	1    6930 4850
@@
 F 0 "J12" H 6980 6167 50  0000 C CNN
 F 1 "Conn_02x03_Odd_Even" H 6980 6076 50  0000 C CNN
-F 2 "digitalSystemBoard:DC3_2x03_PIN" H 6930 5850 50  0001 C CNN
+F 2 "Connector_IDC:IDC-Header_2x03_P2.54mm_Vertical" H 6930 5850 50  0001 C CNN
 F 3 "~" H 6930 5850 50  0001 C CNN
 	1    6930 5850
@@
 L Connector_Generic:Conn_02x03_Odd_Even J9
 U 1 1 5FCBF79B
-P 3900 6100
-F 0 "J9" H 3950 6417 50  0000 C CNN
-F 1 "Conn_02x03_Odd_Even" H 3950 6326 50  0000 C CNN
-F 2 "digitalSystemBoard:DC3_2x03_PIN" H 3900 6100 50  0001 C CNN
-F 3 "~" H 3900 6100 50  0001 C CNN
-	1    3900 6100
-	1    0    0    -1
+P 4000 6100
+F 0 "J9" H 4050 6417 50  0000 C CNN
+F 1 "Conn_02x03_Odd_Even" H 4050 6326 50  0000 C CNN
+F 2 "Connector_IDC:IDC-Header_2x03_P2.54mm_Vertical" H 4000 6100 50  0001 C CNN
+F 3 "~" H 4000 6100 50  0001 C CNN
+	1    4000 6100
+	-1   0    0    1
 $EndComp
 $Comp
@@
 	1    0    0    -1
 $EndComp
+$Comp
+L Connector_Generic:Conn_02x08_Odd_Even J8
+U 1 1 5FC8D8A2
+P 2300 6400
+F 0 "J8" H 2350 6917 50  0000 C CNN
+F 1 "Conn_02x08_Odd_Even" H 2350 6826 50  0000 C CNN
+F 2 "Connector_IDC:IDC-Header_2x08_P2.54mm_Vertical" H 2300 6400 50  0001 C CNN
+F 3 "~" H 2300 6400 50  0001 C CNN
+	1    2300 6400
+	-1   0    0    1
+$EndComp
+Text HLabel 2500 6700 2    50   Input ~ 0
+SW8
+Text HLabel 2500 6600 2    50   Input ~ 0
+SW7
+Text HLabel 2500 6500 2    50   Input ~ 0
+SW6
+Text HLabel 2500 6400 2    50   Input ~ 0
+SW5
+Text HLabel 2500 6300 2    50   Input ~ 0
+SW4
+Text HLabel 2500 6200 2    50   Input ~ 0
+SW3
+Text HLabel 2500 6100 2    50   Input ~ 0
+SW2
+Text HLabel 2500 6000 2    50   Input ~ 0
+SW1
+Text HLabel 2000 6700 0    50   Input ~ 0
+SW8
+Text HLabel 2000 6600 0    50   Input ~ 0
+SW7
+Text HLabel 2000 6500 0    50   Input ~ 0
+SW6
+Text HLabel 2000 6400 0    50   Input ~ 0
+SW5
+Text HLabel 2000 6300 0    50   Input ~ 0
+SW4
+Text HLabel 2000 6200 0    50   Input ~ 0
+SW3
+Text HLabel 2000 6100 0    50   Input ~ 0
+SW2
+Text HLabel 2000 6000 0    50   Input ~ 0
+SW1
 $EndSCHEMATC
