File: digitalSystemBoard/Header_and_Mounting.sch (KiCad schematic (older format))
At the start: 30 parts, among them J10 Conn_02x03_Odd_Even, J11 Conn_02x03_Odd_Even, J12 Conn_02x03_Odd_Even, J3 Conn_02x04_Odd_Even, J4 Conn_02x04_Odd_Even, J5 Conn_02x08_Odd_Even, J6 Conn_02x07_Odd_Even, J7 Conn_02x07_Odd_Even, J8 Conn_02x08_Odd_Even, J9 Conn_02x03_Odd_Even

Commit message: Fix name of all device
Parts:
- renumbered J11 to J10, J12 to J11, J3 to J2, J4 to J3, J5 to J4, J6 to J5, J7 to J6, J8 to J7, J9 to J8, J10 to J9, R79 to R74, R80 to R75, R81 to R76, R82 to R77, R83 to R78, R84 to R79, R85 to R80, R86 to R81, R87 to R82, R88 to R83, R89 to R84, R90 to R85, R91 to R86, R92 to R87, R93 to R88, R94 to R89
Changed lines of the file:
@@
 $EndDescr
 $Comp
-L Connector_Generic:Conn_02x04_Odd_Even J3
+L Connector_Generic:Conn_02x04_Odd_Even J2
 U 1 1 5FC86773
 P 2200 2100
-F 0 "J3" H 2250 2417 50  0000 C CNN
+F 0 "J2" H 2250 2417 50  0000 C CNN
 F 1 "Conn_02x04_Odd_Even" H 2250 2326 50  0000 C CNN
 F 2 "Connector_IDC:IDC-Header_2x04_P2.54mm_Vertical" H 2200 2100 50  0001 C CNN
@@
 $EndComp
 $Comp
-L Connector_Generic:Conn_02x08_Odd_Even J8
+L Connector_Generic:Conn_02x08_Odd_Even J7
 U 1 1 5FC8D8A2
 P 2200 6300
-F 0 "J8" H 2250 6817 50  0000 C CNN
+F 0 "J7" H 2250 6817 50  0000 C CNN
 F 1 "Conn_02x08_Odd_Even" H 2250 6726 50  0000 C CNN
 F 2 "Connector_IDC:IDC-Header_2x08_P2.54mm_Vertical" H 2200 6300 50  0001 C CNN
@@
 $EndComp
 $Comp
-L Connector_Generic:Conn_02x03_Odd_Even J10
+L Connector_Generic:Conn_02x03_Odd_Even J9
 U 1 1 5FC907A2
 P 6930 3920
-F 0 "J10" H 6980 4237 50  0000 C CNN
+F 0 "J9" H 6980 4237 50  0000 C CNN
 F 1 "Conn_02x03_Odd_Even" H 6980 4146 50  0000 C CNN
 F 2 "Connector_IDC:IDC-Header_2x03_P2.54mm_Vertical" H 6930 3920 50  0001 C CNN
@@
 $EndComp
 $Comp
-L Connector_Generic:Conn_02x07_Odd_Even J6
+L Connector_Generic:Conn_02x07_Odd_Even J5
 U 1 1 5FC928BF
 P 2200 3900
-F 0 "J6" H 2250 4417 50  0000 C CNN
+F 0 "J5" H 2250 4417 50  0000 C CNN
 F 1 "Conn_02x07_Odd_Even" H 2250 4326 50  0000 C CNN
 F 2 "Connector_IDC:IDC-Header_2x07_P2.54mm_Vertical" H 2200 3900 50  0001 C CNN
@@
 $EndComp
 $Comp
-L Connector_Generic:Conn_02x07_Odd_Even J7
+L Connector_Generic:Conn_02x07_Odd_Even J6
 U 1 1 5FC93EAD
 P 4000 3900
-F 0 "J7" H 4050 4417 50  0000 C CNN
+F 0 "J6" H 4050 4417 50  0000 C CNN
 F 1 "Conn_02x07_Odd_Even" H 4050 4326 50  0000 C CNN
 F 2 "Connector_IDC:IDC-Header_2x07_P2.54mm_Vertical" H 4000 3900 50  0001 C CNN
@@
 GPIO_LED_1
 $Comp
-L Connector_Generic:Conn_02x08_Odd_Even J5
+L Connector_Generic:Conn_02x08_Odd_Even J4
 U 1 1 5FC8A515
 P 6100 2300
-F 0 "J5" H 6150 2817 50  0000 C CNN
+F 0 "J4" H 6150 2817 50  0000 C CNN
 F 1 "Conn_02x08_Odd_Even" H 6150 2726 50  0000 C CNN
 F 2 "Connector_IDC:IDC-Header_2x08_P2.54mm_Vertical" H 6100 2300 50  0001 C CNN
@@
 CLK_OUT
 $Comp
-L Connector_Generic:Conn_02x03_Odd_Even J11
+L Connector_Generic:Conn_02x03_Odd_Even J10
 U 1 1 5FD1AE53
 P 6930 4850
-F 0 "J11" H 6980 5167 50  0000 C CNN
+F 0 "J10" H 6980 5167 50  0000 C CNN
 F 1 "Conn_02x03_Odd_Even" H 6980 5076 50  0000 C CNN
 F 2 "Connector_IDC:IDC-Header_2x03_P2.54mm_Vertical" H 6930 4850 50  0001 C CNN
@@
 $EndComp
 $Comp
-L Connector_Generic:Conn_02x03_Odd_Even J12
+L Connector_Generic:Conn_02x03_Odd_Even J11
 U 1 1 5FD1B6CA
 P 6930 5850
-F 0 "J12" H 6980 6167 50  0000 C CNN
+F 0 "J11" H 6980 6167 50  0000 C CNN
 F 1 "Conn_02x03_Odd_Even" H 6980 6076 50  0000 C CNN
 F 2 "Connector_IDC:IDC-Header_2x03_P2.54mm_Vertical" H 6930 5850 50  0001 C CNN
@@
 $EndComp
 $Comp
-L Connector_Generic:Conn_02x03_Odd_Even J9
+L Connector_Generic:Conn_02x03_Odd_Even J8
 U 1 1 5FCBF79B
 P 3900 6100
-F 0 "J9" H 3950 6417 50  0000 C CNN
+F 0 "J8" H 3950 6417 50  0000 C CNN
 F 1 "Conn_02x03_Odd_Even" H 3950 6326 50  0000 C CNN
 F 2 "Connector_IDC:IDC-Header_2x03_P2.54mm_Vertical" H 3900 6100 50  0001 C CNN
@@
 SEG_A_1
 $Comp
-L Connector_Generic:Conn_02x04_Odd_Even J4
+L Connector_Generic:Conn_02x04_Odd_Even J3
 U 1 1 5FC88FC0
 P 4000 2100
-F 0 "J4" H 4050 2417 50  0000 C CNN
+F 0 "J3" H 4050 2417 50  0000 C CNN
 F 1 "Conn_02x04_Odd_Even" H 4050 2326 50  0000 C CNN
 F 2 "Connector_IDC:IDC-Header_2x04_P2.54mm_Vertical" H 4000 2100 50  0001 C CNN
@@
 P 7880 2000
 AR Path="/5FB71076/606D777B" Ref="R?"  Part="1"
-AR Path="/5FBA3F95/606D777B" Ref="R79"  Part="1"
-F 0 "R79" V 7880 2000 50  0000 C CNN
+AR Path="/5FBA3F95/606D777B" Ref="R74"  Part="1"
+F 0 "R74" V 7880 2000 50  0000 C CNN
 F 1 "10k" V 7790 2010 50  0000 C CNN
 F 2 "Resistor_SMD:R_0603_1608Metric" V 7810 2000 50  0001 C CNN
@@
 P 7880 2170
 AR Path="/5FB71076/606DB14E" Ref="R?"  Part="1"
-AR Path="/5FBA3F95/606DB14E" Ref="R80"  Part="1"
-F 0 "R80" V 7880 2170 50  0000 C CNN
+AR Path="/5FBA3F95/606DB14E" Ref="R75"  Part="1"
+F 0 "R75" V 7880 2170 50  0000 C CNN
 F 1 "10k" V 7790 2180 50  0000 C CNN
 F 2 "Resistor_SMD:R_0603_1608Metric" V 7810 2170 50  0001 C CNN
@@
 P 7880 2340
 AR Path="/5FB71076/606DB388" Ref="R?"  Part="1"
-AR Path="/5FBA3F95/606DB388" Ref="R81"  Part="1"
-F 0 "R81" V 7880 2340 50  0000 C CNN
+AR Path="/5FBA3F95/606DB388" Ref="R76"  Part="1"
+F 0 "R76" V 7880 2340 50  0000 C CNN
 F 1 "10k" V 7790 2350 50  0000 C CNN
 F 2 "Resistor_SMD:R_0603_1608Metric" V 7810 2340 50  0001 C CNN
@@
 P 7880 2510
 AR Path="/5FB71076/606DBE31" Ref="R?"  Part="1"
-AR Path="/5FBA3F95/606DBE31" Ref="R82"  Part="1"
-F 0 "R82" V 7880 2510 50  0000 C CNN
+AR Path="/5FBA3F95/606DBE31" Ref="R77"  Part="1"
+F 0 "R77" V 7880 2510 50  0000 C CNN
 F 1 "10k" V 7790 2520 50  0000 C CNN
 F 2 "Resistor_SMD:R_0603_1608Metric" V 7810 2510 50  0001 C CNN
@@
 P 7880 2680
 AR Path="/5FB71076/606DBE37" Ref="R?"  Part="1"
-AR Path="/5FBA3F95/606DBE37" Ref="R83"  Part="1"
-F 0 "R83" V 7880 2680 50  0000 C CNN
+AR Path="/5FBA3F95/606DBE37" Ref="R78"  Part="1"
+F 0 "R78" V 7880 2680 50  0000 C CNN
 F 1 "10k" V 7790 2690 50  0000 C CNN
 F 2 "Resistor_SMD:R_0603_1608Metric" V 7810 2680 50  0001 C CNN
@@
 P 7880 2850
 AR Path="/5FB71076/606DBE3D" Ref="R?"  Part="1"
-AR Path="/5FBA3F95/606DBE3D" Ref="R84"  Part="1"
-F 0 "R84" V 7880 2850 50  0000 C CNN
+AR Path="/5FBA3F95/606DBE3D" Ref="R79"  Part="1"
+F 0 "R79" V 7880 2850 50  0000 C CNN
 F 1 "10k" V 7790 2860 50  0000 C CNN
 F 2 "Resistor_SMD:R_0603_1608Metric" V 7810 2850 50  0001 C CNN
@@
 P 7880 3030
 AR Path="/5FB71076/606DC7D3" Ref="R?"  Part="1"
-AR Path="/5FBA3F95/606DC7D3" Ref="R85"  Part="1"
-F 0 "R85" V 7880 3030 50  0000 C CNN
+AR Path="/5FBA3F95/606DC7D3" Ref="R80"  Part="1"
+F 0 "R80" V 7880 3030 50  0000 C CNN
 F 1 "10k" V 7790 3040 50  0000 C CNN
 F 2 "Resistor_SMD:R_0603_1608Metric" V 7810 3030 50  0001 C CNN
@@
 P 7880 3200
 AR Path="/5FB71076/606DC7D9" Ref="R?"  Part="1"
-AR Path="/5FBA3F95/606DC7D9" Ref="R86"  Part="1"
-F 0 "R86" V 7880 3200 50  0000 C CNN
+AR Path="/5FBA3F95/606DC7D9" Ref="R81"  Part="1"
+F 0 "R81" V 7880 3200 50  0000 C CNN
 F 1 "10k" V 7790 3210 50  0000 C CNN
 F 2 "Resistor_SMD:R_0603_1608Metric" V 7810 3200 50  0001 C CNN
@@
 P 9800 1990
 AR Path="/5FB71076/606E0AB8" Ref="R?"  Part="1"
-AR Path="/5FBA3F95/606E0AB8" Ref="R87"  Part="1"
-F 0 "R87" V 9800 1990 50  0000 C CNN
+AR Path="/5FBA3F95/606E0AB8" Ref="R82"  Part="1"
+F 0 "R82" V 9800 1990 50  0000 C CNN
 F 1 "10k" V 9710 2000 50  0000 C CNN
 F 2 "Resistor_SMD:R_0603_1608Metric" V 9730 1990 50  0001 C CNN
@@
 P 9800 2160
 AR Path="/5FB71076/606E0ABE" Ref="R?"  Part="1"
-AR Path="/5FBA3F95/606E0ABE" Ref="R88"  Part="1"
-F 0 "R88" V 9800 2160 50  0000 C CNN
+AR Path="/5FBA3F95/606E0ABE" Ref="R83"  Part="1"
+F 0 "R83" V 9800 2160 50  0000 C CNN
 F 1 "10k" V 9710 2170 50  0000 C CNN
 F 2 "Resistor_SMD:R_0603_1608Metric" V 9730 2160 50  0001 C CNN
@@
 P 9800 2330
 AR Path="/5FB71076/606E0AC4" Ref="R?"  Part="1"
-AR Path="/5FBA3F95/606E0AC4" Ref="R89"  Part="1"
-F 0 "R89" V 9800 2330 50  0000 C CNN
+AR Path="/5FBA3F95/606E0AC4" Ref="R84"  Part="1"
+F 0 "R84" V 9800 2330 50  0000 C CNN
 F 1 "10k" V 9710 2340 50  0000 C CNN
 F 2 "Resistor_SMD:R_0603_1608Metric" V 9730 2330 50  0001 C CNN
@@
 P 9800 2500
 AR Path="/5FB71076/606E0ACA" Ref="R?"  Part="1"
-AR Path="/5FBA3F95/606E0ACA" Ref="R90"  Part="1"
-F 0 "R90" V 9800 2500 50  0000 C CNN
+AR Path="/5FBA3F95/606E0ACA" Ref="R85"  Part="1"
+F 0 "R85" V 9800 2500 50  0000 C CNN
 F 1 "10k" V 9710 2510 50  0000 C CNN
 F 2 "Resistor_SMD:R_0603_1608Metric" V 9730 2500 50  0001 C CNN
@@
 P 9800 2670
 AR Path="/5FB71076/606E0AD0" Ref="R?"  Part="1"
-AR Path="/5FBA3F95/606E0AD0" Ref="R91"  Part="1"
-F 0 "R91" V 9800 2670 50  0000 C CNN
+AR Path="/5FBA3F95/606E0AD0" Ref="R86"  Part="1"
+F 0 "R86" V 9800 2670 50  0000 C CNN
 F 1 "10k" V 9710 2680 50  0000 C CNN
 F 2 "Resistor_SMD:R_0603_1608Metric" V 9730 2670 50  0001 C CNN
@@
 P 9800 2840
 AR Path="/5FB71076/606E0AD6" Ref="R?"  Part="1"
-AR Path="/5FBA3F95/606E0AD6" Ref="R92"  Part="1"
-F 0 "R92" V 9800 2840 50  0000 C CNN
+AR Path="/5FBA3F95/606E0AD6" Ref="R87"  Part="1"
+F 0 "R87" V 9800 2840 50  0000 C CNN
 F 1 "10k" V 9710 2850 50  0000 C CNN
 F 2 "Resistor_SMD:R_0603_1608Metric" V 9730 2840 50  0001 C CNN
@@
 P 9800 3020
 AR Path="/5FB71076/606E0ADC" Ref="R?"  Part="1"
-AR Path="/5FBA3F95/606E0ADC" Ref="R93"  Part="1"
-F 0 "R93" V 9800 3020 50  0000 C CNN
+AR Path="/5FBA3F95/606E0ADC" Ref="R88"  Part="1"
+F 0 "R88" V 9800 3020 50  0000 C CNN
 F 1 "10k" V 9710 3030 50  0000 C CNN
 F 2 "Resistor_SMD:R_0603_1608Metric" V 9730 3020 50  0001 C CNN
@@
 P 9800 3190
 AR Path="/5FB71076/606E0AE2" Ref="R?"  Part="1"
-AR Path="/5FBA3F95/606E0AE2" Ref="R94"  Part="1"
-F 0 "R94" V 9800 3190 50  0000 C CNN
+AR Path="/5FBA3F95/606E0AE2" Ref="R89"  Part="1"
+F 0 "R89" V 9800 3190 50  0000 C CNN
 F 1 "10k" V 9710 3200 50  0000 C CNN
 F 2 "Resistor_SMD:R_0603_1608Metric" V 9730 3190 50  0001 C CNN
