File: digitalSystemBoard/Header_and_Mounting.sch (KiCad schematic (older format))
At the start: 30 parts, among them J10 Conn_02x03_Odd_Even, J11 Conn_02x03_Odd_Even, J2 Conn_02x04_Odd_Even, J3 Conn_02x04_Odd_Even, J4 Conn_02x08_Odd_Even, J5 Conn_02x07_Odd_Even, J6 Conn_02x07_Odd_Even, J7 Conn_02x08_Odd_Even, J8 Conn_02x03_Odd_Even, J9 Conn_02x03_Odd_Even

Commit message: Add BOM file and CPL file
Parts:
- R74, R75, R76, R77, R78, R79, R80, R81, R82, R83, R84, R85, R86, R87, R88, R89: LCSC (none) -> C98220
Changed lines of the file:
@@
 F 2 "Resistor_SMD:R_0603_1608Metric" V 7810 2000 50  0001 C CNN
 F 3 "~" H 7880 2000 50  0001 C CNN
+F 4 "C98220" V 7880 2000 50  0001 C CNN "LCSC"
 	1    7880 2000
 	0    1    1    0
@@
 F 2 "Resistor_SMD:R_0603_1608Metric" V 7810 2170 50  0001 C CNN
 F 3 "~" H 7880 2170 50  0001 C CNN
+F 4 "C98220" V 7880 2170 50  0001 C CNN "LCSC"
 	1    7880 2170
 	0    1    1    0
@@
 F 2 "Resistor_SMD:R_0603_1608Metric" V 7810 2340 50  0001 C CNN
 F 3 "~" H 7880 2340 50  0001 C CNN
+F 4 "C98220" V 7880 2340 50  0001 C CNN "LCSC"
 	1    7880 2340
 	0    1    1    0
@@
 F 2 "Resistor_SMD:R_0603_1608Metric" V 7810 2510 50  0001 C CNN
 F 3 "~" H 7880 2510 50  0001 C CNN
+F 4 "C98220" V 7880 2510 50  0001 C CNN "LCSC"
 	1    7880 2510
 	0    1    1    0
@@
 F 2 "Resistor_SMD:R_0603_1608Metric" V 7810 2680 50  0001 C CNN
 F 3 "~" H 7880 2680 50  0001 C CNN
+F 4 "C98220" V 7880 2680 50  0001 C CNN "LCSC"
 	1    7880 2680
 	0    1    1    0
@@
 F 2 "Resistor_SMD:R_0603_1608Metric" V 7810 2850 50  0001 C CNN
 F 3 "~" H 7880 2850 50  0001 C CNN
+F 4 "C98220" V 7880 2850 50  0001 C CNN "LCSC"
 	1    7880 2850
 	0    1    1    0
@@
 F 2 "Resistor_SMD:R_0603_1608Metric" V 7810 3030 50  0001 C CNN
 F 3 "~" H 7880 3030 50  0001 C CNN
+F 4 "C98220" V 7880 3030 50  0001 C CNN "LCSC"
 	1    7880 3030
 	0    1    1    0
@@
 F 2 "Resistor_SMD:R_0603_1608Metric" V 7810 3200 50  0001 C CNN
 F 3 "~" H 7880 3200 50  0001 C CNN
+F 4 "C98220" V 7880 3200 50  0001 C CNN "LCSC"
 	1    7880 3200
 	0    1    1    0
@@
 F 2 "Resistor_SMD:R_0603_1608Metric" V 9730 1990 50  0001 C CNN
 F 3 "~" H 9800 1990 50  0001 C CNN
+F 4 "C98220" V 9800 1990 50  0001 C CNN "LCSC"
 	1    9800 1990
 	0    1    1    0
@@
 F 2 "Resistor_SMD:R_0603_1608Metric" V 9730 2160 50  0001 C CNN
 F 3 "~" H 9800 2160 50  0001 C CNN
+F 4 "C98220" V 9800 2160 50  0001 C CNN "LCSC"
 	1    9800 2160
 	0    1    1    0
@@
 F 2 "Resistor_SMD:R_0603_1608Metric" V 9730 2330 50  0001 C CNN
 F 3 "~" H 9800 2330 50  0001 C CNN
+F 4 "C98220" V 9800 2330 50  0001 C CNN "LCSC"
 	1    9800 2330
 	0    1    1    0
@@
 F 2 "Resistor_SMD:R_0603_1608Metric" V 9730 2500 50  0001 C CNN
 F 3 "~" H 9800 2500 50  0001 C CNN
+F 4 "C98220" V 9800 2500 50  0001 C CNN "LCSC"
 	1    9800 2500
 	0    1    1    0
@@
 F 2 "Resistor_SMD:R_0603_1608Metric" V 9730 2670 50  0001 C CNN
 F 3 "~" H 9800 2670 50  0001 C CNN
+F 4 "C98220" V 9800 2670 50  0001 C CNN "LCSC"
 	1    9800 2670
 	0    1    1    0
@@
 F 2 "Resistor_SMD:R_0603_1608Metric" V 9730 2840 50  0001 C CNN
 F 3 "~" H 9800 2840 50  0001 C CNN
+F 4 "C98220" V 9800 2840 50  0001 C CNN "LCSC"
 	1    9800 2840
 	0    1    1    0
@@
 F 2 "Resistor_SMD:R_0603_1608Metric" V 9730 3020 50  0001 C CNN
 F 3 "~" H 9800 3020 50  0001 C CNN
+F 4 "C98220" V 9800 3020 50  0001 C CNN "LCSC"
 	1    9800 3020
 	0    1    1    0
@@
 F 2 "Resistor_SMD:R_0603_1608Metric" V 9730 3190 50  0001 C CNN
 F 3 "~" H 9800 3190 50  0001 C CNN
+F 4 "C98220" V 9800 3190 50  0001 C CNN "LCSC"
 	1    9800 3190
 	0    1    1    0

Commit message: Change part for R47K and C22pF
Parts:
- R74, R75, R76, R77, R78, R79, R80, R81: value 10k -> 47k
Changed lines of the file:
@@
 AR Path="/5FBA3F95/606D777B" Ref="R74"  Part="1"
 F 0 "R74" V 7880 2000 50  0000 C CNN
-F 1 "10k" V 7790 2010 50  0000 C CNN
+F 1 "47k" V 7790 2010 50  0000 C CNN
 F 2 "Resistor_SMD:R_0603_1608Metric" V 7810 2000 50  0001 C CNN
 F 3 "~" H 7880 2000 50  0001 C CNN
@@
 AR Path="/5FBA3F95/606DB14E" Ref="R75"  Part="1"
 F 0 "R75" V 7880 2170 50  0000 C CNN
-F 1 "10k" V 7790 2180 50  0000 C CNN
+F 1 "47k" V 7790 2180 50  0000 C CNN
 F 2 "Resistor_SMD:R_0603_1608Metric" V 7810 2170 50  0001 C CNN
 F 3 "~" H 7880 2170 50  0001 C CNN
@@
 AR Path="/5FBA3F95/606DB388" Ref="R76"  Part="1"
 F 0 "R76" V 7880 2340 50  0000 C CNN
-F 1 "10k" V 7790 2350 50  0000 C CNN
+F 1 "47k" V 7790 2350 50  0000 C CNN
 F 2 "Resistor_SMD:R_0603_1608Metric" V 7810 2340 50  0001 C CNN
 F 3 "~" H 7880 2340 50  0001 C CNN
@@
 AR Path="/5FBA3F95/606DBE31" Ref="R77"  Part="1"
 F 0 "R77" V 7880 2510 50  0000 C CNN
-F 1 "10k" V 7790 2520 50  0000 C CNN
+F 1 "47k" V 7790 2520 50  0000 C CNN
 F 2 "Resistor_SMD:R_0603_1608Metric" V 7810 2510 50  0001 C CNN
 F 3 "~" H 7880 2510 50  0001 C CNN
@@
 AR Path="/5FBA3F95/606DBE37" Ref="R78"  Part="1"
 F 0 "R78" V 7880 2680 50  0000 C CNN
-F 1 "10k" V 7790 2690 50  0000 C CNN
+F 1 "47k" V 7790 2690 50  0000 C CNN
 F 2 "Resistor_SMD:R_0603_1608Metric" V 7810 2680 50  0001 C CNN
 F 3 "~" H 7880 2680 50  0001 C CNN
@@
 AR Path="/5FBA3F95/606DBE3D" Ref="R79"  Part="1"
 F 0 "R79" V 7880 2850 50  0000 C CNN
-F 1 "10k" V 7790 2860 50  0000 C CNN
+F 1 "47k" V 7790 2860 50  0000 C CNN
 F 2 "Resistor_SMD:R_0603_1608Metric" V 7810 2850 50  0001 C CNN
 F 3 "~" H 7880 2850 50  0001 C CNN
@@
 AR Path="/5FBA3F95/606DC7D3" Ref="R80"  Part="1"
 F 0 "R80" V 7880 3030 50  0000 C CNN
-F 1 "10k" V 7790 3040 50  0000 C CNN
+F 1 "47k" V 7790 3040 50  0000 C CNN
 F 2 "Resistor_SMD:R_0603_1608Metric" V 7810 3030 50  0001 C CNN
 F 3 "~" H 7880 3030 50  0001 C CNN
@@
 AR Path="/5FBA3F95/606DC7D9" Ref="R81"  Part="1"
 F 0 "R81" V 7880 3200 50  0000 C CNN
-F 1 "10k" V 7790 3210 50  0000 C CNN
+F 1 "47k" V 7790 3210 50  0000 C CNN
 F 2 "Resistor_SMD:R_0603_1608Metric" V 7810 3200 50  0001 C CNN
 F 3 "~" H 7880 3200 50  0001 C CNN
