File: digitalSystemBoard/digitalSystemBoard.kicad_pcb (KiCad board)
At the start: 2 copper layers, 188 x 120 mm, 168 parts, among them J1 Barrel_Jack, J10 Conn_02x03_Odd_Even, J11 Conn_02x03_Odd_Even, J12 Conn_02x03_Odd_Even, J2 USB-B, J3 Conn_02x04_Odd_Even, J4 Conn_02x04_Odd_Even, J5 Conn_02x08_Odd_Even, J6 Conn_02x07_Odd_Even, J7 Conn_02x07_Odd_Even, J8 Conn_02x08_Odd_Even, J9 Conn_02x03_Odd_Even, Q1 MJD122T4G, Q10 BC847, Q11 BC847, Q12 BC847, Q13 BC847, Q14 BC847, Q15 BC847, Q16 BC847, Q17 BC847, Q2 BC847, Q3 BC847, Q4 BC847, Q5 BC847, Q6 BC847, Q7 BC847, Q8 BC847, Q9 BC847, SW1 SW_SPDT, SW9 ButtonFirst, U1 LM317, U10 IO_Switch, U11 IO_Switch, U12 IO_Switch, U13 IO_Switch, U14 74LS04, U15 Potentiometer, U16 ATmega32U4-AU, U17 ICSP, U18 74LS165, U19 74HC164, U2 KCSA02-105, U20 74LS165, U21 74HC164, U3 KCSA02-105, U4 74LS47, U5 74LS47, U6 IO_Switch, U7 IO_Switch, U8 IO_Switch, U9 IO_Switch, Y1 16MHz

Commit message: Layout power block
Parts:
- R3: value 220 -> 330
- moved C3 307.4 mm to (63.0, 96.0)
- moved C4 305.9 mm to (69.0, 76.0)
- moved R3 301.5 mm to (69.0, 84.0), turned to 180 degrees
- moved U1 294.0 mm to (58.0, 86.0), turned to 180 degrees
- moved R5 293.1 mm to (145.0, 111.5)
- moved D1 292.9 mm to (69.0, 80.0), turned to 180 degrees
- moved C1 292.8 mm to (56.0, 116.0), turned to 180 degrees
- moved R6 286.6 mm to (144.9, 104.8)
- moved Q1 282.4 mm to (58.0, 77.0), turned to 180 degrees
- moved C2 280.9 mm to (56.0, 94.0)
- moved R1 280.4 mm to (63.0, 92.0)
- moved C6 277.4 mm to (149.0, 140.0), turned to 180 degrees
- moved R52 273.7 mm to (142.0, 140.0)
- moved R53 269.1 mm to (155.0, 140.0)
- moved C5 264.5 mm to (136.0, 140.0), turned to 180 degrees
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Routing:
- net GND: track 133.1 -> 565.0 mm
- net /VCC5V: track 105.0 -> 217.9 mm
- net /CHANGE_CLK_SRC: track 5.00 -> 73.0 mm, vias 0 -> 1
- net /DOWN_CLOCK: track 5.00 -> 60.6 mm, vias 0 -> 1
- net Net-(C1-Pad1): track 0.00 -> 51.5 mm
- net /UP_CLOCK: track 5.00 -> 48.2 mm, vias 0 -> 1
- net Net-(C2-Pad1): track 0.00 -> 37.7 mm
- net Net-(C6-Pad1): track 5.00 -> 32.7 mm, vias 0 -> 1
- net Net-(C4-Pad1): track 0.00 -> 25.8 mm
- net Net-(J1-Pad1): track 0.00 -> 24.9 mm
- net /SW8: track 0.00 -> 23.5 mm, vias 0 -> 1
- net /SW7: track 0.00 -> 23.5 mm, vias 0 -> 1
- net /SW6: track 0.00 -> 23.5 mm, vias 0 -> 1
- net /SW5: track 0.00 -> 23.5 mm, vias 0 -> 1
- net /SW4: track 0.00 -> 23.5 mm, vias 0 -> 1
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
Commit message: Layout element
Parts:
- moved R8 286.6 mm to (149.9, 113.8)
- moved R9 283.0 mm to (149.9, 109.8)
- moved R12 282.0 mm to (155.5, 108.8)
- moved R11 277.7 mm to (155.3, 112.9)
- moved R10 274.0 mm to (155.3, 117.4)
- moved R16 272.3 mm to (165.7, 118.2)
- moved R15 271.7 mm to (160.8, 109.9)
- moved R13 268.5 mm to (160.5, 118.0)
- moved R18 266.8 mm to (165.5, 110.1)
- moved R19 266.5 mm to (171.2, 118.3)
- moved Q6 265.8 mm to (165.8, 123.3)
- moved R17 262.7 mm to (165.7, 114.3)
- moved R24 260.0 mm to (176.5, 110.1)
- moved R20 256.7 mm to (171.3, 114.4)
- moved R23 256.0 mm to (176.5, 114.3)
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Routing:
- net /VCC5V: track 217.9 -> 200.1 mm
- net GND: track 565.0 -> 547.4 mm
- net /GPIO_LED_8: track 0.00 -> 2.54 mm
- net /GPIO_LED_7: track 0.00 -> 2.54 mm
- net /GPIO_LED_6: track 0.00 -> 2.54 mm
- net /GPIO_LED_5: track 0.00 -> 2.54 mm
- net /GPIO_LED_4: track 0.00 -> 2.54 mm
- net /GPIO_LED_3: track 0.00 -> 2.54 mm
- net /GPIO_LED_2: track 0.00 -> 2.54 mm
- net /GPIO_LED_1: track 0.00 -> 2.54 mm
Other:
- board size 188 x 120 mm -> 180 x 120 mm
- net class Default: clearance 0.2 -> 0.4; trace_width 0.25 -> 0.35
- rule trace_clearance: 0.2 -> 0.4

Commit message: Layout 70 percent board
Parts:
- moved D10 216.6 mm to (75.0, 142.0)
- moved FB2 204.3 mm to (109.0, 110.0), turned to 90 degrees
- moved R58 204.2 mm to (70.0, 136.0), turned to 180 degrees
- moved U16 201.4 mm to (117.0, 92.0)
- moved R59 200.5 mm to (70.0, 140.0), turned to 180 degrees
- moved C14 195.6 mm to (103.0, 93.0), turned to 180 degrees
- moved C15 192.1 mm to (103.0, 89.0), turned to 180 degrees
- moved DS1 189.5 mm to (-34.3, 68.6), turned to 0 degrees
- moved C17 184.7 mm to (103.0, 85.0), turned to 180 degrees
- moved R60 181.8 mm to (75.0, 136.0)
- moved FB0 181.7 mm to (70.0, 144.0), turned to 180 degrees
- moved C16 180.8 mm to (109.0, 104.0), turned to 270 degrees
- moved C13 178.9 mm to (103.0, 81.0), turned to 180 degrees
- moved FB3 172.0 mm to (97.0, 85.0)
- moved C10 170.4 mm to (75.0, 148.0), turned to 180 degrees
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Connections:
- J2 pad 2: Net-(D10-Pad4) -> Net-(D10-Pad6)
- J2 pad 3: Net-(D10-Pad6) -> Net-(D10-Pad4)
- J9 pad 3: /KEY1 -> Net-(J9-Pad3)
- J9 pad 4: /KEY1 -> Net-(J9-Pad4)
- J9 pad 5: Net-(J9-Pad5) -> /KEY1
- J9 pad 6: Net-(J9-Pad6) -> /KEY1
- R13 pad 2: /LED5 -> /LED4
- R16 pad 2: /LED4 -> /LED5
- R58 pad 2: Net-(D10-Pad6) -> Net-(D10-Pad4)
- R59 pad 2: Net-(D10-Pad4) -> Net-(D10-Pad6)
Routing:
- net GND: track 547.4 -> 826.8 mm
- net /VCC5V: track 200.1 -> 395.8 mm
- net /SEG_F_0: track 0.00 -> 91.8 mm, vias 0 -> 2
- net /SEG_G_0: track 0.00 -> 91.0 mm, vias 0 -> 2
- net /ADJ_CLOCK: track 0.00 -> 87.1 mm
- net /MCU/IC_CLOCK: track 0.00 -> 85.2 mm
- net /SEG_E_1: track 0.00 -> 78.7 mm, vias 0 -> 1
- net /SEG_C_1: track 0.00 -> 77.9 mm, vias 0 -> 1
- net /SEG_D_1: track 0.00 -> 77.0 mm, vias 0 -> 1
- net /SEG_B_1: track 0.00 -> 76.7 mm, vias 0 -> 1
- net /LED8: track 0.00 -> 72.3 mm, vias 0 -> 2
- net /SEG_A_0: track 0.00 -> 72.1 mm, vias 0 -> 2
- net /SEG_A_1: track 0.00 -> 69.4 mm, vias 0 -> 1
- net /SEG_B_0: track 0.00 -> 67.1 mm, vias 0 -> 2
- net /SEG_E_0: track 0.00 -> 64.5 mm, vias 0 -> 2
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
Commit message: Edit LCD footprint
Parts:
- moved DS1 124.3 mm to (90.0, 69.0)
- moved C5 13.0 mm to (149.0, 140.0)
- moved C6 13.0 mm to (136.0, 140.0)
- moved KEY0 13.0 mm to (152.0, 150.0)
- moved KEY1 13.0 mm to (139.0, 150.0)
- moved R52 13.0 mm to (155.0, 140.0)
- moved R53 13.0 mm to (142.0, 140.0)
- moved U2 2.00 mm to (189.0, 93.0)
- moved U3 2.00 mm to (174.0, 93.0)
Routing:
- net /SEG_A_1: track 69.4 -> 157.7 mm, vias 1 -> 2
- net /SEG_B_1: track 76.7 -> 164.7 mm, vias 1 -> 2
- net /SEG_C_1: track 77.9 -> 164.9 mm, vias 1 -> 2
- net /SEG_D_1: track 77.0 -> 162.9 mm, vias 1 -> 2
- net /SEG_E_1: track 78.7 -> 163.7 mm, vias 1 -> 2
- net /SEG_F_1: track 53.9 -> 133.9 mm, vias 1 -> 2
- net /SEG_G_1: track 57.7 -> 136.9 mm, vias 1 -> 2
- net Net-(C6-Pad1): track 45.8 -> 33.8 mm
- net /KEY0: track 36.4 -> 48.3 mm
- net /SEG_A_0: track 72.1 -> 75.7 mm
- net /SEG_B_0: track 67.1 -> 69.9 mm
- net /SEG_F_0: track 91.8 -> 94.0 mm
- net /SEG_G_0: track 91.0 -> 92.6 mm
- net /SEG_C_0: track 61.2 -> 62.4 mm
- net /SEG_D_0: track 64.1 -> 65.2 mm
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
Commit message: Add net for ICSP and USB
Parts:
- moved U14 58.8 mm to (145.5, 65.0), turned to 180 degrees
Routing:
- net /MCU/RESET: track 11.0 -> 99.5 mm, vias 0 -> 4
- net /MCU/D-: track 1.81 -> 85.5 mm, vias 0 -> 2
- net /MCU/VBUS: track 6.08 -> 87.4 mm, vias 0 -> 2
- net /MCU/D+: track 1.80 -> 81.0 mm, vias 0 -> 2
- net /MCU/MISO: track 1.78 -> 59.5 mm, vias 0 -> 2
- net /MCU/SCK: track 1.81 -> 57.4 mm, vias 0 -> 2
- net /MCU/MOSI: track 1.80 -> 45.7 mm, vias 0 -> 2
- net /MCU/LCD_0: track 1.65 -> 24.5 mm
- net /MCU/LCD_1: track 1.63 -> 22.8 mm
- net /MCU/LCD_2: track 1.64 -> 21.0 mm
- net /MCU/MCU_TO_IC_164: track 1.79 -> 19.8 mm, vias 0 -> 2
- net GND: track 826.8 -> 844.8 mm
- net /MCU/LCD_3: track 1.63 -> 19.4 mm
- net /MCU/LCD_4: track 1.61 -> 19.0 mm
- net Net-(C16-Pad1): track 19.4 -> 33.4 mm
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
Commit message: Resize board
Parts:
- moved J10 10.0 mm to (131.0, 36.0)
- moved J11 10.0 mm to (67.0, 36.0)
- moved J12 10.0 mm to (84.0, 36.0)
- moved J3 10.0 mm to (218.0, 36.0)
- moved J4 10.0 mm to (198.0, 36.0)
- moved J5 10.0 mm to (178.0, 36.0)
- moved J8 10.0 mm to (114.0, 36.0)
- moved J9 10.0 mm to (148.0, 36.0)
Routing:
- net /UP_CLOCK: track 61.9 -> 93.6 mm, vias 1 -> 2
- net /DOWN_CLOCK: track 73.6 -> 105.0 mm, vias 1 -> 2
- net /CHANGE_CLK_SRC: track 85.4 -> 116.3 mm, vias 1 -> 2
- net /GPIO_BCD_A_0: track 28.0 -> 2.54 mm, vias 1 -> 0
- net /GPIO_BCD_D_1: track 27.8 -> 2.54 mm, vias 1 -> 0
- net /GPIO_LED_1: track 25.9 -> 2.54 mm, vias 1 -> 0
- net /GPIO_LED_8: track 25.8 -> 2.54 mm, vias 1 -> 0
- net /GPIO_BCD_B_0: track 25.4 -> 2.54 mm, vias 1 -> 0
- net /GPIO_BCD_C_1: track 25.2 -> 2.54 mm, vias 1 -> 0
- net /GPIO_LED_7: track 23.8 -> 2.54 mm, vias 1 -> 0
- net /GPIO_LED_2: track 23.7 -> 2.54 mm, vias 1 -> 0
- net /GPIO_BCD_C_0: track 22.7 -> 2.54 mm, vias 1 -> 0
- net /GPIO_BCD_B_1: track 22.5 -> 2.54 mm, vias 1 -> 0
- net /GPIO_LED_6: track 22.4 -> 2.54 mm, vias 1 -> 0
- net /GPIO_LED_3: track 22.3 -> 2.54 mm, vias 1 -> 0
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Other:
- board size 180 x 120 mm -> 180 x 130 mm

Commit message: Switch Connected
Routing:
- net /SW8: track 26.0 -> 191.6 mm, vias 1 -> 2
- net /SW7: track 26.0 -> 185.0 mm, vias 1 -> 2
- net /SW6: track 26.0 -> 178.5 mm, vias 1 -> 2
- net /SW5: track 26.0 -> 172.0 mm, vias 1 -> 2
- net /SW4: track 26.0 -> 165.5 mm, vias 1 -> 2
- net /SW3: track 26.0 -> 159.0 mm, vias 1 -> 2
- net /SW2: track 26.0 -> 152.7 mm, vias 1 -> 2
- net /SW1: track 26.0 -> 146.5 mm, vias 1 -> 2
- net /KEY0: track 48.3 -> 145.2 mm
- net Net-(C6-Pad1): track 33.8 -> 102.3 mm, vias 1 -> 2
- net /CHANGE_CLK_SRC: track 116.3 -> 148.3 mm
- net /DOWN_CLOCK: track 105.0 -> 135.9 mm
- net /UP_CLOCK: track 93.6 -> 123.5 mm
- net /MCU/SCK: track 57.4 -> 55.5 mm
- net /MCU/MISO: track 59.5 -> 57.9 mm
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
Commit message: LCD connected
Routing:
- net /ADJ_CLOCK: track 87.1 -> 168.4 mm, vias 0 -> 1
- net /MCU/LCD_ENABLE: track 4.65 -> 53.0 mm, vias 0 -> 3
- net /MCU/LCD_5: track 4.49 -> 49.8 mm, vias 0 -> 1
- net /MCU/LCD_6: track 4.62 -> 41.3 mm, vias 0 -> 1
- net /MCU/LCD_7: track 4.56 -> 40.1 mm, vias 0 -> 1
- net /MCU/LCD_RS: track 4.81 -> 1.84 mm
- net /MCU/LCD_0: track 24.5 -> 21.5 mm, vias 0 -> 1
- net /MCU/LCD_1: track 22.8 -> 20.8 mm, vias 0 -> 1
- net Net-(C16-Pad1): track 33.4 -> 31.8 mm
- net /MCU/LCD_2: track 21.0 -> 20.1 mm, vias 0 -> 1
- net /MCU/LCD_4: track 19.0 -> 18.7 mm, vias 0 -> 1
- net /MCU/LCD_3: track 19.4 -> 19.3 mm, vias 0 -> 1
Other:
- net class Default: clearance 0.4 -> 0.2
- rule trace_clearance: 0.4 -> 0.2
