File: digitalSystemBoard/digitalSystemBoard.kicad_pcb (KiCad board)
At the start: 2 copper layers, 180 x 130 mm, 168 parts, among them J1 Barrel_Jack, J10 Conn_02x03_Odd_Even, J11 Conn_02x03_Odd_Even, J12 Conn_02x03_Odd_Even, J2 USB-B, J3 Conn_02x04_Odd_Even, J4 Conn_02x04_Odd_Even, J5 Conn_02x08_Odd_Even, J6 Conn_02x07_Odd_Even, J7 Conn_02x07_Odd_Even, J8 Conn_02x08_Odd_Even, J9 Conn_02x03_Odd_Even, Q1 MJD122T4G, Q10 BC847, Q11 BC847, Q12 BC847, Q13 BC847, Q14 BC847, Q15 BC847, Q16 BC847, Q17 BC847, Q2 BC847, Q3 BC847, Q4 BC847, Q5 BC847, Q6 BC847, Q7 BC847, Q8 BC847, Q9 BC847, SW1 SW_SPDT, SW9 ButtonFirst, U1 LM317, U10 IO_Switch, U11 IO_Switch, U12 IO_Switch, U13 IO_Switch, U14 74LS04, U15 Potentiometer, U16 ATmega32U4-AU, U17 ICSP, U18 74LS165, U19 74HC164, U2 KCSA02-105, U20 74LS165, U21 74HC164, U3 KCSA02-105, U4 74LS47, U5 74LS47, U6 IO_Switch, U7 IO_Switch, U8 IO_Switch, U9 IO_Switch, Y1 16MHz

Commit message: finish wiring
Parts:
- added REF**: POWER_VIA, digitalSystemBoard:POWER_VIA, F.Cu at (127.7, 110.5)
- added REF**: POWER_VIA, digitalSystemBoard:POWER_VIA, F.Cu at (204.9, 51.1)
- added REF**: POWER_VIA, digitalSystemBoard:POWER_VIA, F.Cu at (181.2, 67.6)
- added REF**: POWER_VIA, digitalSystemBoard:POWER_VIA, F.Cu at (152.2, 73.6)
- added REF**: POWER_VIA, digitalSystemBoard:POWER_VIA, F.Cu at (152.2, 110.5)
- added REF**: POWER_VIA, digitalSystemBoard:POWER_VIA, F.Cu at (180.4, 120.1)
- added REF**: POWER_VIA, digitalSystemBoard:POWER_VIA, F.Cu at (187.5, 121.2)
- added REF**: POWER_VIA, digitalSystemBoard:POWER_VIA, F.Cu at (215.9, 121.2)
- added REF**: POWER_VIA, digitalSystemBoard:POWER_VIA, F.Cu at (127.7, 97.6)
- added REF**: POWER_VIA, digitalSystemBoard:POWER_VIA, F.Cu at (181.2, 54.5)
- added REF**: POWER_VIA, digitalSystemBoard:POWER_VIA, F.Cu at (181.2, 63.2)
- added REF**: POWER_VIA, digitalSystemBoard:POWER_VIA, F.Cu at (190.5, 67.6)
- moved R3 2.00 mm to (69.0, 82.0)
- moved D1 1.00 mm to (69.0, 79.0)
Connections:
- SW1 pad 1: Net-(SW1-Pad1) -> Net-(C1-Pad1)
- SW1 pad 3: Net-(C1-Pad1) -> Net-(SW1-Pad3)
Routing:
- net /VCC5V: track 395.8 -> 1157.4 mm, vias 0 -> 1
- net GND: track 837.0 -> 1458.9 mm, vias 0 -> 8
- net Net-(C1-Pad1): track 51.5 -> 57.6 mm
- net /ADJ_CLOCK: track 168.4 -> 171.0 mm
- net /7SEGLED_TEST_OFF: track 88.5 -> 89.9 mm
- net /MCU/IC_CLOCK: track 218.3 -> 219.3 mm
- net Net-(D1-Pad2): track 4.00 -> 3.00 mm
- net /BCD_D_1: track 32.8 -> 31.8 mm
- net /MCU/IC_165_CTRL: track 129.7 -> 130.3 mm
- net /BCD_A_1: track 25.7 -> 25.2 mm
Other:
- net class Default: clearance 0.4 -> 0.2
- rule trace_clearance: 0.4 -> 0.2

Commit message: pour cu
Routing:
- added copper zone on B.Cu, net GND
- added copper zone on F.Cu, net GND
Changed lines of the file:
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@@
   (segment (start 203.17063 70.32001) (end 173.57065 70.32001) (width 0.35) (layer F.Cu) (net 163))
   (segment (start 205.31564 68.175) (end 203.17063 70.32001) (width 0.35) (layer F.Cu) (net 163))
+  (zone (net 1) (net_name GND) (layer F.Cu) (hatch edge 0.508)
+    (connect_pads (clearance 0.508))
+    (min_thickness 0.254)
+    (fill yes (arc_segments 32) (thermal_gap 0.508) (thermal_bridge_width 0.508))
+    (polygon
+      (pts
+        (xy 230 160) (xy 50 160) (xy 50 30) (xy 230 30)
+      )
+    )
+  )
+  (zone (net 1) (net_name GND) (layer B.Cu) (hatch edge 0.508)
+    (connect_pads (clearance 0.508))
+    (min_thickness 0.254)
+    (fill yes (arc_segments 32) (thermal_gap 0.508) (thermal_bridge_width 0.508) (smoothing fillet))
+    (polygon
+      (pts
+        (xy 230 160) (xy 50 160) (xy 50 30) (xy 230 30)
+      )
+    )
+  )
 )

Commit message: added pin map
Other:
- board outline removed
- board text added: "0"
- board text added: "1"
- board text added: "12VDC"
- board text added: "3A FUSE"
- board text added: "5V"
- board text added: "ADJ"
- board text added: "BCD0_A"
- board text added: "BCD0_B"
- board text added: "BCD0_C"
- board text added: "BCD0_D"
- board text added: "BCD1_A"
- board text added: "BCD1_B"
- board text added: "BCD1_C"
- board text added: "BCD1_D"
- board text added: "CLK"
- board text added: "DO NOT TOUCH"
- board text added: "GND"
- board text added: "ICSP"
- board text added: "KEY_0"
- board text added: "KEY_1"
- board text added: "KEY_A"
- board text added: "KEY_B"
- board text added: "LED_0"
- board text added: "LED_1"
- board text added: "LED_2"
- board text added: "LED_3"
- board text added: "LED_4"
- board text added: "LED_5"
- board text added: "LED_6"
- board text added: "LED_7"
- board text added: "OFF"
- board text added: "ON"
- board text added: "RESET"
- board text added: "SEG0"
- board text added: "SEG0_A"
- board text added: "SEG0_B"
- board text added: "SEG0_C"
- board text added: "SEG0_D"
- board text added: "SEG0_E"
- board text added: "SEG0_F"
- board text added: "SEG0_G"
- board text added: "SEG1"
- board text added: "SEG1_A"
- board text added: "SEG1_B"
- board text added: "SEG1_C"
- board text added: "SEG1_D"
- board text added: "SEG1_E"
- board text added: "SEG1_F"
- board text added: "SEG1_G"
- board text added: "SW0"
- board text added: "SW1"
- board text added: "SW2"
- board text added: "SW3"
- board text added: "SW4"
- board text added: "SW5"
- board text added: "SW6"
- board text added: "SW7"

Commit message: Hot fix: modifiy LCD footprint
Parts:
- DS1: footprint Display:WC1602A -> digitalSystemBoard:WC1602A
Connections:
- U4 pad 10: /SEG_D_0 -> Net-(R66-Pad2)
- U4 pad 11: /SEG_C_0 -> Net-(R65-Pad2)
- U4 pad 12: /SEG_B_0 -> Net-(R64-Pad2)
- U4 pad 13: /SEG_A_0 -> Net-(R63-Pad2)
- U4 pad 14: /SEG_G_0 -> Net-(R69-Pad2)
- U4 pad 15: /SEG_F_0 -> Net-(R68-Pad2)
- U4 pad 9: /SEG_E_0 -> Net-(R67-Pad2)
- U5 pad 10: /SEG_D_1 -> Net-(R73-Pad2)
- U5 pad 11: /SEG_C_1 -> Net-(R72-Pad2)
- U5 pad 12: /SEG_B_1 -> Net-(R71-Pad2)
- U5 pad 13: /SEG_A_1 -> Net-(R70-Pad2)
- U5 pad 14: /SEG_G_1 -> Net-(R76-Pad2)
- U5 pad 15: /SEG_F_1 -> Net-(R75-Pad2)
- U5 pad 9: /SEG_E_1 -> Net-(R74-Pad2)
Routing:
- net /VCC5V: track 1157.4 -> 1158.4 mm
- net GND: track 1458.9 -> 1457.9 mm
- net /MCU/LCD_RS: track 27.4 -> 27.9 mm
- net /MCU/LCD_ENABLE: track 53.9 -> 54.4 mm
- net /MCU/LCD_7: track 40.1 -> 40.6 mm
- net /MCU/LCD_6: track 41.3 -> 41.8 mm
- net /MCU/LCD_5: track 49.9 -> 50.4 mm
- net /MCU/LCD_4: track 18.7 -> 19.2 mm
- net /MCU/LCD_3: track 19.3 -> 19.8 mm
- net /MCU/LCD_2: track 21.1 -> 21.6 mm
- net /MCU/LCD_1: track 22.7 -> 23.2 mm
- net /MCU/LCD_0: track 24.3 -> 24.8 mm
- removed copper zone on B.Cu, net GND
- removed copper zone on F.Cu, net GND
Other:
- board text added: "KEY_C"

Commit message: Hot fix: move fuse
Parts:
- added R63: 330, Resistor_SMD:R_0603_1608Metric, F.Cu at (206.0, 83.5)
- added R64: 330, Resistor_SMD:R_0603_1608Metric, F.Cu at (202.8, 82.5)
- added R65: 330, Resistor_SMD:R_0603_1608Metric, F.Cu at (202.8, 88.5)
- added R66: 330, Resistor_SMD:R_0603_1608Metric, F.Cu at (206.0, 87.5)
- added R67: 330, Resistor_SMD:R_0603_1608Metric, F.Cu at (202.8, 86.5)
- added R68: 330, Resistor_SMD:R_0603_1608Metric, F.Cu at (202.8, 84.5)
- added R69: 330, Resistor_SMD:R_0603_1608Metric, F.Cu at (206.0, 85.5)
- added R70: 330, Resistor_SMD:R_0603_1608Metric, F.Cu at (167.0, 84.5)
- added R71: 330, Resistor_SMD:R_0603_1608Metric, F.Cu at (170.2, 85.5)
- added R72: 330, Resistor_SMD:R_0603_1608Metric, F.Cu at (167.0, 86.5)
- added R73: 330, Resistor_SMD:R_0603_1608Metric, F.Cu at (170.2, 87.5)
- added R74: 330, Resistor_SMD:R_0603_1608Metric, F.Cu at (167.0, 88.5)
- added R75: 330, Resistor_SMD:R_0603_1608Metric, F.Cu at (170.2, 83.5)
- added R76: 330, Resistor_SMD:R_0603_1608Metric, F.Cu at (167.0, 82.5)
- moved F1 2.00 mm to (65.0, 55.0)
Connections:
- D10 pad 3: Net-(D10-Pad3) -> (no net)
- D10 pad 5: Net-(D10-Pad5) -> (no net)
- J9 pad 3: Net-(J9-Pad3) -> (no net)
- J9 pad 4: Net-(J9-Pad4) -> (no net)
- SW1 pad 3: Net-(SW1-Pad3) -> (no net)
- SW9 pad 2: Net-(SW9-Pad2) -> (no net)
- SW9 pad 4: Net-(SW9-Pad4) -> (no net)
- U18 pad 7: Net-(U18-Pad7) -> (no net)
- U2 pad 1: /SEG_E_0 -> Net-(R67-Pad1)
- U2 pad 10: /SEG_G_0 -> Net-(R69-Pad1)
- U2 pad 2: /SEG_D_0 -> Net-(R66-Pad1)
- U2 pad 4: /SEG_C_0 -> Net-(R65-Pad1)
- U2 pad 5: Net-(U2-Pad5) -> (no net)
- U2 pad 6: /SEG_B_0 -> Net-(R64-Pad1)
- U2 pad 7: /SEG_A_0 -> Net-(R63-Pad1)
- U2 pad 9: /SEG_F_0 -> Net-(R68-Pad1)
- U20 pad 7: Net-(U20-Pad7) -> (no net)
- U3 pad 1: /SEG_E_1 -> Net-(R74-Pad1)
- U3 pad 10: /SEG_G_1 -> Net-(R76-Pad1)
- U3 pad 2: /SEG_D_1 -> Net-(R73-Pad1)
- U3 pad 4: /SEG_C_1 -> Net-(R72-Pad1)
- U3 pad 5: Net-(U3-Pad5) -> (no net)
- U3 pad 6: /SEG_B_1 -> Net-(R71-Pad1)
- U3 pad 7: /SEG_A_1 -> Net-(R70-Pad1)
- U3 pad 9: /SEG_F_1 -> Net-(R75-Pad1)
- U4 pad 10: Net-(R66-Pad2) -> /SEG_D_0
- U4 pad 11: Net-(R65-Pad2) -> /SEG_C_0
- U4 pad 12: Net-(R64-Pad2) -> /SEG_B_0
- U4 pad 13: Net-(R63-Pad2) -> /SEG_A_0
- U4 pad 14: Net-(R69-Pad2) -> /SEG_G_0
- U4 pad 15: Net-(R68-Pad2) -> /SEG_F_0
- U4 pad 9: Net-(R67-Pad2) -> /SEG_E_0
- U5 pad 10: Net-(R73-Pad2) -> /SEG_D_1
- U5 pad 11: Net-(R72-Pad2) -> /SEG_C_1
- U5 pad 12: Net-(R71-Pad2) -> /SEG_B_1
- U5 pad 13: Net-(R70-Pad2) -> /SEG_A_1
- U5 pad 14: Net-(R76-Pad2) -> /SEG_G_1
- U5 pad 15: Net-(R75-Pad2) -> /SEG_F_1
- U5 pad 9: Net-(R74-Pad2) -> /SEG_E_1
Routing:
- net /SEG_G_0: track 93.0 -> 70.4 mm
- net Net-(R69-Pad1): track 0.00 -> 21.2 mm
- net /SEG_A_1: track 157.7 -> 138.1 mm
- net /SEG_B_1: track 164.7 -> 145.2 mm
- net /SEG_C_1: track 164.9 -> 145.5 mm
- net /SEG_D_0: track 65.5 -> 46.8 mm
- net /SEG_E_0: track 65.4 -> 46.9 mm
- net Net-(R70-Pad1): track 0.00 -> 18.1 mm
- net Net-(R71-Pad1): track 0.00 -> 17.9 mm
- net Net-(R72-Pad1): track 0.00 -> 17.9 mm
- net Net-(R66-Pad1): track 0.00 -> 17.1 mm
- net Net-(R67-Pad1): track 0.00 -> 16.8 mm
- net /SEG_F_0: track 94.4 -> 78.0 mm
- net Net-(R68-Pad1): track 0.00 -> 14.8 mm
- net /SEG_A_0: track 76.0 -> 62.1 mm
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- added copper zone on B.Cu, net GND
- added copper zone on F.Cu, net GND

Commit message: Hot fix: change symbol and footprint of the barrell jack
Connections:
- D10 pad 3: (no net) -> Net-(D10-Pad3)
- D10 pad 5: (no net) -> Net-(D10-Pad5)
- J1 pad 3: (no net) -> GND
- J9 pad 3: (no net) -> Net-(J9-Pad3)
- J9 pad 4: (no net) -> Net-(J9-Pad4)
- SW1 pad 3: (no net) -> Net-(SW1-Pad3)
- SW9 pad 2: (no net) -> Net-(SW9-Pad2)
- SW9 pad 4: (no net) -> Net-(SW9-Pad4)
- U18 pad 7: (no net) -> Net-(U18-Pad7)
- U2 pad 5: (no net) -> Net-(U2-Pad5)
- U20 pad 7: (no net) -> Net-(U20-Pad7)
- U3 pad 5: (no net) -> Net-(U3-Pad5)
Routing:
- net /7SEGLED_TEST_ON: track 85.3 -> 84.5 mm
- net /MCU/IC_164_CTRL: track 94.1 -> 94.9 mm
- net /7SEGLED_TEST_OFF: track 89.9 -> 89.1 mm
- removed copper zone on B.Cu, net GND
- removed copper zone on F.Cu, net GND

Commit message: re-route power line, reset origin
Routing:
- net GND: track 1457.9 -> 1464.6 mm
- added copper zone on B.Cu, net GND
- added copper zone on F.Cu, net GND
Other:
- board outline added: 180 x 130 mm
