File: digitalSystemBoard/digitalSystemBoard.kicad_pcb (KiCad board)
At the start: 2 copper layers, 180 x 130 mm, 197 parts, among them J1 Barrel_Jack, J10 Conn_02x03_Odd_Even, J11 Conn_02x03_Odd_Even, J12 Conn_02x03_Odd_Even, J2 USB-B, J3 Conn_02x04_Odd_Even, J4 Conn_02x04_Odd_Even, J5 Conn_02x08_Odd_Even, J6 Conn_02x07_Odd_Even, J7 Conn_02x07_Odd_Even, J8 Conn_02x08_Odd_Even, J9 Conn_02x03_Odd_Even, Q1 MJD122T4G, Q10 BC847, Q11 BC847, Q12 BC847, Q13 BC847, Q14 BC847, Q15 BC847, Q16 BC847, Q17 BC847, Q2 BC847, Q3 BC847, Q4 BC847, Q5 BC847, Q6 BC847, Q7 BC847, Q8 BC847, Q9 BC847, SW1 SW_SPDT, SW9 ButtonFirst, U1 LM317, U10 IO_Switch, U11 IO_Switch, U12 IO_Switch, U13 IO_Switch, U14 74LS04, U15 Potentiometer, U16 ATmega32U4-AU, U17 ICSP, U18 74LS165, U19 74HC164, U2 KCSA02-105, U20 74LS165, U21 74HC164, U3 KCSA02-105, U4 74LS47, U5 74LS47, U6 IO_Switch, U7 IO_Switch, U8 IO_Switch, U9 IO_Switch, Y1 16MHz

Commit message: Add keepout areas for Power Block. Modify 7-segment LED schematic
Connections:
- U2 pad 3: GND -> /VCC5V
- U2 pad 8: GND -> /VCC5V
- U3 pad 3: GND -> /VCC5V
- U3 pad 8: GND -> /VCC5V
Routing:
- net GND: track 1491.8 -> 1384.0 mm
- net /VCC5V: track 1149.3 -> 1198.0 mm

Commit message: Fix bug in BCD, add an rheostat on Vo and add an resistor on LED+
Parts:
- added R78: R, Resistor_SMD:R_0603_1608Metric, F.Cu at (127.0, 73.0)
- added RN1: R_Pack08, digitalSystemBoard:Resistor Bar 06030 8P4R, F.Cu at (182.0, 47.0)
- added RN2: R_Pack08, digitalSystemBoard:Resistor Bar 06030 8P4R, F.Cu at (186.0, 47.0)
- added TRIM2: Potentiometer, digitalSystemBoard:TRIM_3296W-1-501, F.Cu at (95.0, 60.0)
- moved REF** 3.32 mm to (204.9, 54.5)
Connections:
- DS1 pad 15: /VCC5V -> Net-(DS1-Pad15)
- DS1 pad 3: /VCC5V -> Net-(DS1-Pad3)
- U4 pad 2: /BCD_D_0 -> /BCD_C_0
Routing:
- net /VCC5V: track 1198.0 -> 1160.5 mm
- net /BCD_D_0: track 27.0 -> 0.00 mm
- net /BCD_C_0: track 20.4 -> 35.0 mm
- net Net-(DS1-Pad3): track 0.00 -> 8.53 mm
- net GND: track 1384.0 -> 1390.4 mm
- net Net-(DS1-Pad15): track 0.00 -> 4.77 mm
- removed copper zone on B.Cu, net GND
- removed copper zone on F.Cu, net GND

Commit message: Reroute VCC5V line
Parts:
- turned RN2 to 270 degrees
Routing:
- net GND: track 1390.4 -> 1417.2 mm
- net /VCC5V: track 1160.5 -> 1175.7 mm

Commit message: Add IC 74HC595 and R for input pin
Parts:
- removed the REF** at (127.7, 110.5)
- removed the REF** at (152.2, 110.5)
- removed the REF** at (180.4, 120.1)
- removed RN1, RN2: R_Pack08, digitalSystemBoard:Resistor Bar 06030 8P4R
- added R79: 10k, Resistor_SMD:R_0603_1608Metric, F.Cu at (182.0, 45.0)
- added R80: 10k, Resistor_SMD:R_0603_1608Metric, F.Cu at (182.0, 47.0)
- added R81: 10k, Resistor_SMD:R_0603_1608Metric, F.Cu at (182.0, 49.0)
- added R82: 10k, Resistor_SMD:R_0603_1608Metric, F.Cu at (182.0, 51.0)
- added R83: 10k, Resistor_SMD:R_0603_1608Metric, F.Cu at (156.0, 51.0)
- added R84: 10k, Resistor_SMD:R_0603_1608Metric, F.Cu at (156.0, 49.0)
- added R85: 10k, Resistor_SMD:R_0603_1608Metric, F.Cu at (156.0, 47.0)
- added R86: 10k, Resistor_SMD:R_0603_1608Metric, F.Cu at (156.0, 45.0)
- added R87: 10k, Resistor_SMD:R_0603_1608Metric, F.Cu at (206.0, 51.0)
- added R88: 10k, Resistor_SMD:R_0603_1608Metric, F.Cu at (206.0, 49.0)
- added R89: 10k, Resistor_SMD:R_0603_1608Metric, F.Cu at (206.0, 47.0)
- added R90: 10k, Resistor_SMD:R_0603_1608Metric, F.Cu at (206.0, 45.0)
- added R91: 10k, Resistor_SMD:R_0603_1608Metric, F.Cu at (202.0, 45.0)
- added R92: 10k, Resistor_SMD:R_0603_1608Metric, F.Cu at (202.0, 47.0)
- added R93: 10k, Resistor_SMD:R_0603_1608Metric, F.Cu at (202.0, 49.0)
- added R94: 10k, Resistor_SMD:R_0603_1608Metric, F.Cu at (202.0, 51.0)
- added REF**: POWER_VIA, digitalSystemBoard:POWER_VIA, F.Cu at (183.0, 121.0)
- U19, U21: value 74HC164 -> 74HC595; footprint Package_SO:SOIC-14_3.9x8.7mm_P1.27mm -> Package_SO:SOIC-16_3.9x9.9mm_P1.27mm
- moved REF** 3.54 mm to (191.0, 121.0)
- moved U19 2.00 mm to (169.0, 119.0), turned to 0 degrees
- moved U21 2.00 mm to (204.0, 119.0), turned to 0 degrees
Connections:
- U16 pad 25: /MCU/IC_164_CTRL -> /MCU/IC_595_CTRL
- U16 pad 8: /MCU/MCU_TO_IC_164 -> /MCU/MCU_TO_IC_595
- U19 pad 1: /MCU/MCU_TO_IC_164 -> /LED2
- U19 pad 10: /LED5 -> /VCC5V
- U19 pad 11: /LED6 -> /MCU/IC_CLOCK
- U19 pad 12: /LED7 -> /MCU/IC_595_CTRL
- U19 pad 13: /LED8 -> GND
- U19 pad 14: /VCC5V -> /MCU/MCU_TO_IC_595
- U19 pad 2: /VCC5V -> /LED3
- U19 pad 3: /LED1 -> /LED4
- U19 pad 4: /LED2 -> /LED5
- U19 pad 5: /LED3 -> /LED6
- U19 pad 6: /LED4 -> /LED7
- U19 pad 7: GND -> /LED8
- U19 pad 8: /MCU/IC_CLOCK -> GND
- U19 pad 9: /MCU/IC_164_CTRL -> Net-(U19-Pad9)
- U21 pad 1: /LED8 -> /BCD_B_0
- U21 pad 10: /BCD_A_1 -> /VCC5V
- U21 pad 11: /BCD_B_1 -> /MCU/IC_CLOCK
- U21 pad 12: /BCD_C_1 -> /MCU/IC_595_CTRL
- U21 pad 13: /BCD_D_1 -> GND
- U21 pad 14: /VCC5V -> Net-(U19-Pad9)
- U21 pad 2: /VCC5V -> /BCD_C_0
- U21 pad 3: /BCD_A_0 -> /BCD_D_0
- U21 pad 4: /BCD_B_0 -> /BCD_A_1
- U21 pad 5: /BCD_C_0 -> /BCD_B_1
- U21 pad 6: /BCD_D_0 -> /BCD_C_1
- U21 pad 7: GND -> /BCD_D_1
- U21 pad 8: /MCU/IC_CLOCK -> GND
- U21 pad 9: /MCU/IC_164_CTRL -> Net-(U21-Pad9)
- U4 pad 6: /BCD_C_0 -> /BCD_D_0
Routing:
- net /MCU/IC_595_CTRL: track 0.00 -> 141.4 mm, vias 0 -> 7
- net /MCU/MCU_TO_IC_164: track 100.2 -> 0.00 mm, vias 4 -> 0
- net /MCU/IC_164_CTRL: track 94.9 -> 0.00 mm
- net /MCU/MCU_TO_IC_595: track 0.00 -> 91.0 mm, vias 0 -> 2
- net Net-(U19-Pad9): track 0.00 -> 46.9 mm, vias 0 -> 2
- net /LED8: track 72.3 -> 27.3 mm
- net /VCC5V: track 1175.7 -> 1217.9 mm
- net /MCU/IC_CLOCK: track 219.3 -> 242.9 mm, vias 6 -> 8
- net /GPIO_LED_5: track 32.2 -> 53.6 mm
- net /GPIO_LED_4: track 30.4 -> 51.6 mm
- net /BCD_C_0: track 35.0 -> 14.1 mm
- net /GPIO_BCD_A_0: track 38.9 -> 59.0 mm
- net /GPIO_BCD_D_1: track 38.8 -> 58.7 mm
- net GND: track 1417.2 -> 1399.7 mm
- net /GPIO_LED_6: track 33.8 -> 51.2 mm
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
Commit message: Edit ground wire
Routing:
- net GND: track 1399.7 -> 1433.8 mm
- net /MCU/IC_595_CTRL: vias 7 -> 6

Commit message: Add Power_module to schematic and pcb
Parts:
- removed C1: 0.1uF, Capacitor_SMD:CP_Elec_5x5.8
- removed C2: 100uF, Capacitor_SMD:CP_Elec_6.3x7.7
- removed C3, C4: 10uF, Capacitor_SMD:C_0603_1608Metric
- removed D1: LED, LED_SMD:LED_0603_1608Metric
- removed Q1: MJD122T4G, digitalSystemBoard:MJD122T4G
- removed R1: 220, Resistor_SMD:R_0603_1608Metric
- removed R2: 0.22_5W, digitalSystemBoard:5W_0.22R
- removed R3: 470, Resistor_SMD:R_0603_1608Metric
- removed R77: 1k, Resistor_SMD:R_0603_1608Metric
- removed the REF** at (71.0, 102.0)
- removed the REF** at (56.1, 70.2)
- removed TRIM1: Potentiometer, digitalSystemBoard:TRIM_3296W-1-501
- removed U1: LM317, digitalSystemBoard:LM317AMDT
- added PW1: Power_Module, digitalSystemBoard:Power_Module, F.Cu at (65.0, 82.4)
- F1: value 2A -> 3A
- moved SW1 8.00 mm to (63.0, 113.0)
- moved F1 1.00 mm to (65.0, 54.0)
- moved H2 1.00 mm to (85.0, 60.0)
Connections:
- F1 pad 1: Net-(C4-Pad1) -> /VCC5V
- F1 pad 2: /VCC5V -> Net-(F1-Pad2)
Routing:
- net Net-(PW1-Pad1): track 160.7 -> 9.62 mm
- net /VCC5V: track 1217.9 -> 1142.0 mm
- net GND: track 1433.8 -> 1365.7 mm
- net Net-(F1-Pad2): track 0.00 -> 52.6 mm
- net Net-(C2-Pad1): track 41.6 -> 0.00 mm
- net Net-(C4-Pad1): track 28.0 -> 0.00 mm
- net Net-(Q1-Pad3): track 15.8 -> 0.00 mm
- net Net-(R1-Pad2): track 14.5 -> 0.00 mm
- net Net-(J1-Pad1): track 24.9 -> 16.0 mm
- net Net-(D1-Pad2): track 3.00 -> 0.00 mm
Other:
- board text removed: "DO NOT TOUCH"

Commit message: Soldermask
Routing:
- added copper zone on B.Cu, net GND
- added copper zone on F.Cu, net GND

Commit message: Fix name of all device
Parts:
- R0: renamed from R78; value R -> 220
- R57: renamed from R60; value 10K -> 10k
- renumbered C6 to C0, C5 to C1, C15 to C10, C16 to C11, C17 to C12, C7 to C2, C8 to C3, C9 to C4, C10 to C5, C11 to C6, C12 to C7, C13 to C8, C14 to C9, D2 to D0, D3 to D1, D4 to D2, D5 to D3, D6 to D4, D7 to D5, D8 to D6, D9 to D7, DS1 to DS0, F1 to F0, J1 to J0, J2 to J1, J11 to J10, J12 to J11, J3 to J2, J4 to J3, J5 to J4, J6 to J5, J7 to J6, J8 to J7, J9 to J8, J10 to J9, LED1 to LED0, LED2 to LED1, LED3 to LED2, LED4 to LED3, LED5 to LED4, LED6 to LED5, LED7 to LED6, LED8 to LED7, PW1 to PM0, Q2 to Q0, Q3 to Q1, Q12 to Q10, Q13 to Q11, Q14 to Q12, Q15 to Q13, Q16 to Q14, Q17 to Q15, Q4 to Q2, Q5 to Q3, Q6 to Q4, Q7 to Q5, Q8 to Q6, Q9 to Q7, Q10 to Q8, Q11 to Q9, R57 to R1, R58 to R2, R59 to R3, R53 to R52, R52 to R53, R61 to R58, R62 to R59, R63 to R60, R64 to R61, R65 to R62, R66 to R63, R67 to R64, R68 to R65, R69 to R66, R70 to R67, R71 to R68, R72 to R69, R73 to R70, R74 to R71, R75 to R72, R76 to R73, R79 to R74, R80 to R75, R81 to R76, R82 to R77, R83 to R78, R84 to R79, R85 to R80, R86 to R81, R87 to R82, R88 to R83, R89 to R84, R90 to R85, R91 to R86, R92 to R87, R93 to R88, R94 to R89, SW1 to SW0, U6 to SW1, U7 to SW2, U8 to SW3, U9 to SW4, U10 to SW5, U11 to SW6, U12 to SW7, U13 to SW8, D10 to TD0, TRIM2 to TRIM0, U2 to U0, U3 to U1, U20 to U10, U21 to U11, U4 to U2, U5 to U3, U14 to U4, U15 to U5, U16 to U6, U17 to U7, U18 to U8, U19 to U9, Y1 to Y0
Routing:
- net GND: track 1365.7 -> 1360.7 mm
