File: digitalSystemBoard/DISPLAY.sch (KiCad schematic (older format))
At the start: 44 parts, among them Q2 BC847, Q3 BC847, Q4 BC847, Q5 BC847, Q6 BC847, Q7 BC847, Q8 BC847, Q9 BC847, U2 KCSA02-105, U3 KCSA02-105, U4 74LS47, U5 74LS47

Commit message: Change grid size to 10mils and wire components in power supply and display sheet
Parts:
- removed Q9: BC847, Package_TO_SOT_SMD:SOT-23, symbol Transistor_BJT:BC847
- removed R25: 10k, symbol Device:R
- removed R26: 1k8, symbol Device:R
- removed R27: 330, symbol Device:R
- added Q2: BC847, Package_TO_SOT_SMD:SOT-23, symbol Transistor_BJT:BC847
- added R4: 10k, symbol Device:R
- added R5: 330, symbol Device:R
- added R6: 1k8, symbol Device:R
- R11, R14, R17, R20, R23, R8: value 1k8 -> 330
- R12, R15, R18, R21, R24, R9: value 330 -> 1k8
- renumbered Q2 to Q1, R4 to R1, R6 to R2, R5 to R3
Connections:
- net GND: now also R12.1, R15.1, R18.1, R21.1, R24.1, R9.1, Q2.2 (E), R6.1; no longer R11.1, R14.1, R17.1, R20.1, R23.1, R8.1
- net LED2: now also R4.2; no longer R7.2
- net LED3: now also R7.2; no longer R10.2
- net LED4: now also R10.2; no longer R13.2
- net LED5: now also R13.2; no longer R16.2
- net LED6: now also R16.2; no longer R19.2
- net LED7: now also R19.2; no longer R22.2
- net LED8: now also R22.2
- net SEG_A_0: now also U2.7 (A)
- net SEG_B_0: now also U2.6 (B)
- net SEG_C_0: now also U2.4 (C)
- net SEG_D_0: now also U2.2 (D)
- net SEG_E_0: now also U2.1 (E)
- net SEG_F_0: now also U2.9 (F)
- net SEG_G_0: now also U2.10 (G)
- net VCC5V: now also R11.1, R14.1, R17.1, R20.1, R23.1, R8.1, R5.1; no longer R12.1, R15.1, R18.1, R21.1, R24.1, R9.1
- net at Q3.1 (B), R7.1: now also R9.2; no longer R8.2
- net at LED2.1 (K): now also Q2.3 (C); no longer Q3.3 (C)
- net at LED2.2 (A): now also R5.2; no longer R9.2
- net at Q4.1 (B), R10.1: now also R12.2; no longer R11.2
- net at LED3.1 (K): now also Q3.3 (C); no longer Q4.3 (C)
- net at LED3.2 (A): now also R8.2; no longer R12.2
- net at Q5.1 (B), R13.1: now also R15.2; no longer R14.2
- net at LED4.1 (K): now also Q4.3 (C); no longer Q5.3 (C)
- net at LED4.2 (A): now also R11.2; no longer R15.2
- net at Q6.1 (B), R16.1: now also R18.2; no longer R17.2
- net at LED5.1 (K): now also Q5.3 (C); no longer Q6.3 (C)
- net at LED5.2 (A): now also R14.2; no longer R18.2
- net at Q7.1 (B), R19.1: now also R21.2; no longer R20.2
- net at LED6.1 (K): now also Q6.3 (C); no longer Q7.3 (C)
- net at LED6.2 (A): now also R17.2; no longer R21.2
- net at Q8.1 (B), R22.1: now also R24.2; no longer R23.2
- net at LED7.1 (K): now also Q7.3 (C); no longer Q8.3 (C)
- net at LED7.2 (A): now also R20.2; no longer R24.2
- net at LED8.1 (K): now also Q8.3 (C)
- net at LED8.2 (A): now also R23.2
- new net: Q2.1 (B), R4.1, R6.2
Other:
- moved on the sheet: R1, U2, U4, U5

Commit message: Update Schematic for review
Parts:
- LED1, LED2, LED3, LED4, LED5, LED6, LED7, LED8: footprint (none) -> LED_SMD:LED_0603_1608Metric
- R10: renamed from R7; footprint (none) -> Resistor_SMD:R_0603_1608Metric
- R11: renamed from R9; footprint (none) -> Resistor_SMD:R_0603_1608Metric
- R12: renamed from R8; footprint (none) -> Resistor_SMD:R_0603_1608Metric
- R13: renamed from R10; footprint (none) -> Resistor_SMD:R_0603_1608Metric
- R14: renamed from R12; footprint (none) -> Resistor_SMD:R_0603_1608Metric
- R15: renamed from R11; footprint (none) -> Resistor_SMD:R_0603_1608Metric
- R16: renamed from R13; footprint (none) -> Resistor_SMD:R_0603_1608Metric
- R17: renamed from R15; footprint (none) -> Resistor_SMD:R_0603_1608Metric
- R18: renamed from R14; footprint (none) -> Resistor_SMD:R_0603_1608Metric
- R19: renamed from R16; footprint (none) -> Resistor_SMD:R_0603_1608Metric
- R20: renamed from R18; footprint (none) -> Resistor_SMD:R_0603_1608Metric
- R21: renamed from R17; footprint (none) -> Resistor_SMD:R_0603_1608Metric
- R22: renamed from R19; footprint (none) -> Resistor_SMD:R_0603_1608Metric
- R23: renamed from R21; footprint (none) -> Resistor_SMD:R_0603_1608Metric
- R24: renamed from R20; footprint (none) -> Resistor_SMD:R_0603_1608Metric
- R25: renamed from R22; footprint (none) -> Resistor_SMD:R_0603_1608Metric
- R26: renamed from R24; footprint (none) -> Resistor_SMD:R_0603_1608Metric
- R27: renamed from R23; footprint (none) -> Resistor_SMD:R_0603_1608Metric
- R4: renamed from R1; footprint (none) -> Resistor_SMD:R_0603_1608Metric
- R5: renamed from R3; footprint (none) -> Resistor_SMD:R_0603_1608Metric
- R6: renamed from R2; footprint (none) -> Resistor_SMD:R_0603_1608Metric
- R7: renamed from R4; footprint (none) -> Resistor_SMD:R_0603_1608Metric
- R8: renamed from R6; footprint (none) -> Resistor_SMD:R_0603_1608Metric
- R9: renamed from R5; footprint (none) -> Resistor_SMD:R_0603_1608Metric
- renumbered Q1 to Q2, Q2 to Q3, Q3 to Q4, Q4 to Q5, Q5 to Q6, Q6 to Q7, Q7 to Q8, Q8 to Q9
Connections:
- net VCC5V: no longer U4.3 (LT), U4.4 (BI), U5.3 (LT), U5.4 (BI)
- new net 7SEGLED_TEST_OFF: U4.4 (BI), U5.4 (BI)
- new net 7SEGLED_TEST_ON: U4.3 (LT), U5.3 (LT)
Other:
- moved on the sheet: U5

Commit message: Add full footprint. Draw layout board
Parts:
- LED1, LED2, LED3, LED4, LED5, LED6, LED7, LED8: footprint LED_SMD:LED_0603_1608Metric -> digitalSystemBoard:LED_3528
- U2, U3: footprint Display_7Segment:KCSC02-105 -> Display_7Segment:7SegmentLED_LTS6760_LTS6780
- U4, U5: footprint (none) -> digitalSystemBoard:DIP_16_PIN_SOCKET
Changed lines of the file:
@@
 F 0 "U5" H 8910 5710 50  0000 C CNN
 F 1 "74LS47" H 8850 5270 50  0000 C CNN
-F 2 "" H 8850 5270 50  0001 C CNN
+F 2 "digitalSystemBoard:DIP_16_PIN_SOCKET" H 8850 5270 50  0001 C CNN
 F 3 "http://www.ti.com/lit/gpn/sn74LS47" H 8850 5270 50  0001 C CNN
 	1    8850 5270
@@
 F 0 "U4" H 6710 5740 50  0000 C CNN
 F 1 "74LS47" H 6630 5280 50  0000 C CNN
-F 2 "" H 6630 5270 50  0001 C CNN
+F 2 "digitalSystemBoard:DIP_16_PIN_SOCKET" H 6630 5270 50  0001 C CNN
 F 3 "http://www.ti.com/lit/gpn/sn74LS47" H 6630 5270 50  0001 C CNN
 	1    6630 5270
@@
 F 0 "LED1" V 3029 1102 50  0000 R CNN
 F 1 "LED" V 2938 1102 50  0000 R CNN
-F 2 "LED_SMD:LED_0603_1608Metric" H 2990 1220 50  0001 C CNN
+F 2 "digitalSystemBoard:LED_3528" H 2990 1220 50  0001 C CNN
 F 3 "~" H 2990 1220 50  0001 C CNN
 	1    2990 1220
@@
 F 0 "U2" H 3170 6007 50  0000 C CNN
 F 1 "KCSA02-105" H 3170 5916 50  0000 C CNN
-F 2 "Display_7Segment:KCSC02-105" H 3170 4740 50  0001 C CNN
+F 2 "Display_7Segment:7SegmentLED_LTS6760_LTS6780" H 3170 4740 50  0001 C CNN
 F 3 "http://www.kingbright.com/attachments/file/psearch/000/00/00/KCSA02-105(Ver.10A).pdf" H 2670 5815 50  0001 L CNN
 	1    3170 5340
@@
 F 0 "U3" H 4820 5987 50  0000 C CNN
 F 1 "KCSA02-105" H 4820 5896 50  0000 C CNN
-F 2 "Display_7Segment:KCSC02-105" H 4820 4720 50  0001 C CNN
+F 2 "Display_7Segment:7SegmentLED_LTS6760_LTS6780" H 4820 4720 50  0001 C CNN
 F 3 "http://www.kingbright.com/attachments/file/psearch/000/00/00/KCSA02-105(Ver.10A).pdf" H 4320 5795 50  0001 L CNN
 	1    4820 5320
@@
 F 0 "LED2" V 4509 1132 50  0000 R CNN
 F 1 "LED" V 4418 1132 50  0000 R CNN
-F 2 "LED_SMD:LED_0603_1608Metric" H 4470 1250 50  0001 C CNN
+F 2 "digitalSystemBoard:LED_3528" H 4470 1250 50  0001 C CNN
 F 3 "~" H 4470 1250 50  0001 C CNN
 	1    4470 1250
@@
 F 0 "LED3" V 6099 1132 50  0000 R CNN
 F 1 "LED" V 6008 1132 50  0000 R CNN
-F 2 "LED_SMD:LED_0603_1608Metric" H 6060 1250 50  0001 C CNN
+F 2 "digitalSystemBoard:LED_3528" H 6060 1250 50  0001 C CNN
 F 3 "~" H 6060 1250 50  0001 C CNN
 	1    6060 1250
@@
 F 0 "LED4" V 7519 1132 50  0000 R CNN
 F 1 "LED" V 7428 1132 50  0000 R CNN
-F 2 "LED_SMD:LED_0603_1608Metric" H 7480 1250 50  0001 C CNN
+F 2 "digitalSystemBoard:LED_3528" H 7480 1250 50  0001 C CNN
 F 3 "~" H 7480 1250 50  0001 C CNN
 	1    7480 1250
@@
 F 0 "LED5" V 3019 2842 50  0000 R CNN
 F 1 "LED" V 2928 2842 50  0000 R CNN
-F 2 "LED_SMD:LED_0603_1608Metric" H 2980 2960 50  0001 C CNN
+F 2 "digitalSystemBoard:LED_3528" H 2980 2960 50  0001 C CNN
 F 3 "~" H 2980 2960 50  0001 C CNN
 	1    2980 2960
@@
 F 0 "LED6" V 4509 2872 50  0000 R CNN
 F 1 "LED" V 4418 2872 50  0000 R CNN
-F 2 "LED_SMD:LED_0603_1608Metric" H 4470 2990 50  0001 C CNN
+F 2 "digitalSystemBoard:LED_3528" H 4470 2990 50  0001 C CNN
 F 3 "~" H 4470 2990 50  0001 C CNN
 	1    4470 2990
@@
 F 0 "LED7" V 6049 2862 50  0000 R CNN
 F 1 "LED" V 5958 2862 50  0000 R CNN
-F 2 "LED_SMD:LED_0603_1608Metric" H 6010 2980 50  0001 C CNN
+F 2 "digitalSystemBoard:LED_3528" H 6010 2980 50  0001 C CNN
 F 3 "~" H 6010 2980 50  0001 C CNN
 	1    6010 2980
@@
 F 0 "LED8" V 7499 2832 50  0000 R CNN
 F 1 "LED" V 7408 2832 50  0000 R CNN
-F 2 "LED_SMD:LED_0603_1608Metric" H 7460 2950 50  0001 C CNN
+F 2 "digitalSystemBoard:LED_3528" H 7460 2950 50  0001 C CNN
 F 3 "~" H 7460 2950 50  0001 C CNN
 	1    7460 2950

Commit message: Hot fix: added resistors for ic 7447
Parts:
- added R63, R64, R65, R66, R67, R68, R69, R70, R71, R72, R73, R74, R75, R76: 330, Resistor_SMD:R_0603_1608Metric, symbol Device:R
Connections:
- net SEG_A_0: now also R63.1; no longer U4.13 (a)
- net SEG_A_1: now also R70.1; no longer U5.13 (a)
- net SEG_B_0: now also R64.1; no longer U4.12 (b)
- net SEG_B_1: now also R71.1; no longer U5.12 (b)
- net SEG_C_0: now also R65.1; no longer U4.11 (c)
- net SEG_C_1: now also R72.1; no longer U5.11 (c)
- net SEG_D_0: now also R66.1; no longer U4.10 (d)
- net SEG_D_1: now also R73.1; no longer U5.10 (d)
- net SEG_E_0: now also R67.1; no longer U4.9 (e)
- net SEG_E_1: now also R74.1; no longer U5.9 (e)
- net SEG_F_0: now also R68.1; no longer U4.15 (f)
- net SEG_F_1: now also R75.1; no longer U5.15 (f)
- net SEG_G_0: now also R69.1; no longer U4.14 (g)
- net SEG_G_1: now also R76.1; no longer U5.14 (g)
- new net: R73.2, U5.10 (d)
- new net: R72.2, U5.11 (c)
- new net: R71.2, U5.12 (b)
- new net: R70.2, U5.13 (a)
- new net: R76.2, U5.14 (g)
- new net: R75.2, U5.15 (f)
- new net: R74.2, U5.9 (e)
- new net: R66.2, U4.10 (d)
- new net: R65.2, U4.11 (c)
- new net: R64.2, U4.12 (b)
- new net: R63.2, U4.13 (a)
- new net: R69.2, U4.14 (g)
- new net: R68.2, U4.15 (f)
- new net: R67.2, U4.9 (e)
Other:
- moved on the sheet: U2, U3, U4
