File: digitalSystemBoard/DISPLAY.sch (KiCad schematic (older format))
At the start: 58 parts, among them Q2 BC847, Q3 BC847, Q4 BC847, Q5 BC847, Q6 BC847, Q7 BC847, Q8 BC847, Q9 BC847, U2 KCSA02-105, U3 KCSA02-105, U4 74LS47, U5 74LS47

Commit message: Hot fix: Change footprint. Fix power schematic.
Parts:
- Q2, Q3, Q4, Q5, Q6, Q7, Q8, Q9: footprint Package_TO_SOT_SMD:SOT-23 -> digitalSystemBoard:SO65P210X100-3N
Changed lines of the file:
@@
 F 0 "Q2" H 3081 1616 50  0000 L CNN
 F 1 "BC847" H 3081 1525 50  0000 L CNN
-F 2 "Package_TO_SOT_SMD:SOT-23" H 3090 1495 50  0001 L CIN
+F 2 "digitalSystemBoard:SO65P210X100-3N" H 3090 1495 50  0001 L CIN
 F 3 "http://www.infineon.com/dgdl/Infineon-BC847SERIES_BC848SERIES_BC849SERIES_BC850SERIES-DS-v01_01-en.pdf?fileId=db3a304314dca389011541d4630a1657" H 2890 1570 50  0001 L CNN
 	1    2890 1570
@@
 F 0 "Q3" H 4561 1646 50  0000 L CNN
 F 1 "BC847" H 4561 1555 50  0000 L CNN
-F 2 "Package_TO_SOT_SMD:SOT-23" H 4570 1525 50  0001 L CIN
+F 2 "digitalSystemBoard:SO65P210X100-3N" H 4570 1525 50  0001 L CIN
 F 3 "http://www.infineon.com/dgdl/Infineon-BC847SERIES_BC848SERIES_BC849SERIES_BC850SERIES-DS-v01_01-en.pdf?fileId=db3a304314dca389011541d4630a1657" H 4370 1600 50  0001 L CNN
 	1    4370 1600
@@
 F 0 "Q4" H 6151 1646 50  0000 L CNN
 F 1 "BC847" H 6151 1555 50  0000 L CNN
-F 2 "Package_TO_SOT_SMD:SOT-23" H 6160 1525 50  0001 L CIN
+F 2 "digitalSystemBoard:SO65P210X100-3N" H 6160 1525 50  0001 L CIN
 F 3 "http://www.infineon.com/dgdl/Infineon-BC847SERIES_BC848SERIES_BC849SERIES_BC850SERIES-DS-v01_01-en.pdf?fileId=db3a304314dca389011541d4630a1657" H 5960 1600 50  0001 L CNN
 	1    5960 1600
@@
 F 0 "Q5" H 7571 1646 50  0000 L CNN
 F 1 "BC847" H 7571 1555 50  0000 L CNN
-F 2 "Package_TO_SOT_SMD:SOT-23" H 7580 1525 50  0001 L CIN
+F 2 "digitalSystemBoard:SO65P210X100-3N" H 7580 1525 50  0001 L CIN
 F 3 "http://www.infineon.com/dgdl/Infineon-BC847SERIES_BC848SERIES_BC849SERIES_BC850SERIES-DS-v01_01-en.pdf?fileId=db3a304314dca389011541d4630a1657" H 7380 1600 50  0001 L CNN
 	1    7380 1600
@@
 F 0 "Q6" H 3071 3356 50  0000 L CNN
 F 1 "BC847" H 3071 3265 50  0000 L CNN
-F 2 "Package_TO_SOT_SMD:SOT-23" H 3080 3235 50  0001 L CIN
+F 2 "digitalSystemBoard:SO65P210X100-3N" H 3080 3235 50  0001 L CIN
 F 3 "http://www.infineon.com/dgdl/Infineon-BC847SERIES_BC848SERIES_BC849SERIES_BC850SERIES-DS-v01_01-en.pdf?fileId=db3a304314dca389011541d4630a1657" H 2880 3310 50  0001 L CNN
 	1    2880 3310
@@
 F 0 "Q7" H 4561 3386 50  0000 L CNN
 F 1 "BC847" H 4561 3295 50  0000 L CNN
-F 2 "Package_TO_SOT_SMD:SOT-23" H 4570 3265 50  0001 L CIN
+F 2 "digitalSystemBoard:SO65P210X100-3N" H 4570 3265 50  0001 L CIN
 F 3 "http://www.infineon.com/dgdl/Infineon-BC847SERIES_BC848SERIES_BC849SERIES_BC850SERIES-DS-v01_01-en.pdf?fileId=db3a304314dca389011541d4630a1657" H 4370 3340 50  0001 L CNN
 	1    4370 3340
@@
 F 0 "Q8" H 6101 3376 50  0000 L CNN
 F 1 "BC847" H 6101 3285 50  0000 L CNN
-F 2 "Package_TO_SOT_SMD:SOT-23" H 6110 3255 50  0001 L CIN
+F 2 "digitalSystemBoard:SO65P210X100-3N" H 6110 3255 50  0001 L CIN
 F 3 "http://www.infineon.com/dgdl/Infineon-BC847SERIES_BC848SERIES_BC849SERIES_BC850SERIES-DS-v01_01-en.pdf?fileId=db3a304314dca389011541d4630a1657" H 5910 3330 50  0001 L CNN
 	1    5910 3330
@@
 F 0 "Q9" H 7551 3346 50  0000 L CNN
 F 1 "BC847" H 7551 3255 50  0000 L CNN
-F 2 "Package_TO_SOT_SMD:SOT-23" H 7560 3225 50  0001 L CIN
+F 2 "digitalSystemBoard:SO65P210X100-3N" H 7560 3225 50  0001 L CIN
 F 3 "http://www.infineon.com/dgdl/Infineon-BC847SERIES_BC848SERIES_BC849SERIES_BC850SERIES-DS-v01_01-en.pdf?fileId=db3a304314dca389011541d4630a1657" H 7360 3300 50  0001 L CNN
 	1    7360 3300

Commit message: Add keepout areas for Power Block. Modify 7-segment LED schematic
Connections:
- net GND: no longer U2.3 (CA), U2.8 (CA), U3.3 (CA), U3.8 (CA)
- net VCC5V: now also U2.3 (CA), U2.8 (CA), U3.3 (CA), U3.8 (CA)
Changed lines of the file:
@@
 SEG_G_0
 NoConn ~ 1800 5790
-$Comp
-L power:GND #PWR0101
-U 1 1 5FCA686C
-P 2460 5790
-F 0 "#PWR0101" H 2460 5540 50  0001 C CNN
-F 1 "GND" H 2465 5617 50  0000 C CNN
-F 2 "" H 2460 5790 50  0001 C CNN
-F 3 "" H 2460 5790 50  0001 C CNN
-	1    2460 5790
-	1    0    0    -1
-$EndComp
 Wire Wire Line
 	2400 5790 2460 5790
@@
 Wire Wire Line
 	2460 5690 2460 5790
-Connection ~ 2460 5790
 $Comp
 L Display_Character:KCSA02-105 U3
@@
 SEG_G_1
 NoConn ~ 3450 5770
-$Comp
-L power:GND #PWR0102
-U 1 1 5FCBD203
-P 4110 5770
-F 0 "#PWR0102" H 4110 5520 50  0001 C CNN
-F 1 "GND" H 4115 5597 50  0000 C CNN
-F 2 "" H 4110 5770 50  0001 C CNN
-F 3 "" H 4110 5770 50  0001 C CNN
-	1    4110 5770
-	1    0    0    -1
-$EndComp
 Wire Wire Line
 	4050 5770 4110 5770
@@
 Wire Wire Line
 	4110 5670 4110 5770
-Connection ~ 4110 5770
 $Comp
 L Transistor_BJT:BC847 Q2
@@
 	0    1    1    0
 $EndComp
+Text HLabel 4110 5670 2    50   Input ~ 0
+VCC5V
+Text HLabel 2460 5690 2    50   Input ~ 0
+VCC5V
 $EndSCHEMATC

Commit message: Fix name of all device
Parts:
- renumbered LED1 to LED0, LED2 to LED1, LED3 to LED2, LED4 to LED3, LED5 to LED4, LED6 to LED5, LED7 to LED6, LED8 to LED7, Q2 to Q0, Q3 to Q1, Q4 to Q2, Q5 to Q3, Q6 to Q4, Q7 to Q5, Q8 to Q6, Q9 to Q7, R63 to R60, R64 to R61, R65 to R62, R66 to R63, R67 to R64, R68 to R65, R69 to R66, R70 to R67, R71 to R68, R72 to R69, R73 to R70, R74 to R71, R75 to R72, R76 to R73, U2 to U0, U3 to U1, U4 to U2, U5 to U3
Other:
- moved on the sheet: R60, R61, R62, R63, R64, R65, R66, U0

Commit message: Update voltage bias for LED green and LED yellow
Parts:
- R10, R13, R16, R19, R22, R25, R4, R7: value 10k -> 15k
- R11, R14, R17, R20, R23, R26, R5, R8: value 1k8 -> 2.49k
- R12, R15, R18, R21, R24, R27, R6, R9: value 330 -> 2.49k
Changed lines of the file:
@@
 P 2990 920
 F 0 "R6" H 3060 966 50  0000 L CNN
-F 1 "330" H 3060 875 50  0000 L CNN
+F 1 "2.49k" H 3060 875 50  0000 L CNN
 F 2 "Resistor_SMD:R_0603_1608Metric" V 2920 920 50  0001 C CNN
 F 3 "~" H 2990 920 50  0001 C CNN
@@
 P 2670 1770
 F 0 "R5" H 2600 1724 50  0000 R CNN
-F 1 "1k8" H 2600 1815 50  0000 R CNN
+F 1 "2.49k" H 2600 1815 50  0000 R CNN
 F 2 "Resistor_SMD:R_0603_1608Metric" V 2600 1770 50  0001 C CNN
 F 3 "~" H 2670 1770 50  0001 C CNN
@@
 P 2450 1570
 F 0 "R4" V 2243 1570 50  0000 C CNN
-F 1 "10k" V 2334 1570 50  0000 C CNN
+F 1 "15k" V 2334 1570 50  0000 C CNN
 F 2 "Resistor_SMD:R_0603_1608Metric" V 2380 1570 50  0001 C CNN
 F 3 "~" H 2450 1570 50  0001 C CNN
@@
 P 4470 950
 F 0 "R9" H 4540 996 50  0000 L CNN
-F 1 "330" H 4540 905 50  0000 L CNN
+F 1 "2.49k" H 4540 905 50  0000 L CNN
 F 2 "Resistor_SMD:R_0603_1608Metric" V 4400 950 50  0001 C CNN
 F 3 "~" H 4470 950 50  0001 C CNN
@@
 P 4150 1800
 F 0 "R8" H 4080 1754 50  0000 R CNN
-F 1 "1k8" H 4080 1845 50  0000 R CNN
+F 1 "2.49k" H 4080 1845 50  0000 R CNN
 F 2 "Resistor_SMD:R_0603_1608Metric" V 4080 1800 50  0001 C CNN
 F 3 "~" H 4150 1800 50  0001 C CNN
@@
 P 3930 1600
 F 0 "R7" V 3723 1600 50  0000 C CNN
-F 1 "10k" V 3814 1600 50  0000 C CNN
+F 1 "15k" V 3814 1600 50  0000 C CNN
 F 2 "Resistor_SMD:R_0603_1608Metric" V 3860 1600 50  0001 C CNN
 F 3 "~" H 3930 1600 50  0001 C CNN
@@
 P 6060 950
 F 0 "R12" H 6130 996 50  0000 L CNN
-F 1 "330" H 6130 905 50  0000 L CNN
+F 1 "2.49k" H 6130 905 50  0000 L CNN
 F 2 "Resistor_SMD:R_0603_1608Metric" V 5990 950 50  0001 C CNN
 F 3 "~" H 6060 950 50  0001 C CNN
@@
 P 5740 1800
 F 0 "R11" H 5670 1754 50  0000 R CNN
-F 1 "1k8" H 5670 1845 50  0000 R CNN
+F 1 "2.49k" H 5670 1845 50  0000 R CNN
 F 2 "Resistor_SMD:R_0603_1608Metric" V 5670 1800 50  0001 C CNN
 F 3 "~" H 5740 1800 50  0001 C CNN
@@
 P 5520 1600
 F 0 "R10" V 5313 1600 50  0000 C CNN
-F 1 "10k" V 5404 1600 50  0000 C CNN
+F 1 "15k" V 5404 1600 50  0000 C CNN
 F 2 "Resistor_SMD:R_0603_1608Metric" V 5450 1600 50  0001 C CNN
 F 3 "~" H 5520 1600 50  0001 C CNN
@@
 P 7480 950
 F 0 "R15" H 7550 996 50  0000 L CNN
-F 1 "330" H 7550 905 50  0000 L CNN
+F 1 "2.49k" H 7550 905 50  0000 L CNN
 F 2 "Resistor_SMD:R_0603_1608Metric" V 7410 950 50  0001 C CNN
 F 3 "~" H 7480 950 50  0001 C CNN
@@
 P 7160 1800
 F 0 "R14" H 7090 1754 50  0000 R CNN
-F 1 "1k8" H 7090 1845 50  0000 R CNN
+F 1 "2.49k" H 7090 1845 50  0000 R CNN
 F 2 "Resistor_SMD:R_0603_1608Metric" V 7090 1800 50  0001 C CNN
 F 3 "~" H 7160 1800 50  0001 C CNN
@@
 P 6940 1600
 F 0 "R13" V 6733 1600 50  0000 C CNN
-F 1 "10k" V 6824 1600 50  0000 C CNN
+F 1 "15k" V 6824 1600 50  0000 C CNN
 F 2 "Resistor_SMD:R_0603_1608Metric" V 6870 1600 50  0001 C CNN
 F 3 "~" H 6940 1600 50  0001 C CNN
@@
 P 2980 2660
 F 0 "R18" H 3050 2706 50  0000 L CNN
-F 1 "330" H 3050 2615 50  0000 L CNN
+F 1 "2.49k" H 3050 2615 50  0000 L CNN
 F 2 "Resistor_SMD:R_0603_1608Metric" V 2910 2660 50  0001 C CNN
 F 3 "~" H 2980 2660 50  0001 C CNN
@@
 P 2660 3510
 F 0 "R17" H 2590 3464 50  0000 R CNN
-F 1 "1k8" H 2590 3555 50  0000 R CNN
+F 1 "2.49k" H 2590 3555 50  0000 R CNN
 F 2 "Resistor_SMD:R_0603_1608Metric" V 2590 3510 50  0001 C CNN
 F 3 "~" H 2660 3510 50  0001 C CNN
@@
 P 2440 3310
 F 0 "R16" V 2233 3310 50  0000 C CNN
-F 1 "10k" V 2324 3310 50  0000 C CNN
+F 1 "15k" V 2324 3310 50  0000 C CNN
 F 2 "Resistor_SMD:R_0603_1608Metric" V 2370 3310 50  0001 C CNN
 F 3 "~" H 2440 3310 50  0001 C CNN
@@
 P 4470 2690
 F 0 "R21" H 4540 2736 50  0000 L CNN
-F 1 "330" H 4540 2645 50  0000 L CNN
+F 1 "2.49k" H 4540 2645 50  0000 L CNN
 F 2 "Resistor_SMD:R_0603_1608Metric" V 4400 2690 50  0001 C CNN
 F 3 "~" H 4470 2690 50  0001 C CNN
@@
 P 4150 3540
 F 0 "R20" H 4080 3494 50  0000 R CNN
-F 1 "1k8" H 4080 3585 50  0000 R CNN
+F 1 "2.49k" H 4080 3585 50  0000 R CNN
 F 2 "Resistor_SMD:R_0603_1608Metric" V 4080 3540 50  0001 C CNN
 F 3 "~" H 4150 3540 50  0001 C CNN
@@
 P 3930 3340
 F 0 "R19" V 3723 3340 50  0000 C CNN
-F 1 "10k" V 3814 3340 50  0000 C CNN
+F 1 "15k" V 3814 3340 50  0000 C CNN
 F 2 "Resistor_SMD:R_0603_1608Metric" V 3860 3340 50  0001 C CNN
 F 3 "~" H 3930 3340 50  0001 C CNN
@@
 P 6010 2680
 F 0 "R24" H 6080 2726 50  0000 L CNN
-F 1 "330" H 6080 2635 50  0000 L CNN
+F 1 "2.49k" H 6080 2635 50  0000 L CNN
 F 2 "Resistor_SMD:R_0603_1608Metric" V 5940 2680 50  0001 C CNN
 F 3 "~" H 6010 2680 50  0001 C CNN
@@
 P 5690 3530
 F 0 "R23" H 5620 3484 50  0000 R CNN
-F 1 "1k8" H 5620 3575 50  0000 R CNN
+F 1 "2.49k" H 5620 3575 50  0000 R CNN
 F 2 "Resistor_SMD:R_0603_1608Metric" V 5620 3530 50  0001 C CNN
 F 3 "~" H 5690 3530 50  0001 C CNN
@@
 P 5470 3330
 F 0 "R22" V 5263 3330 50  0000 C CNN
-F 1 "10k" V 5354 3330 50  0000 C CNN
+F 1 "15k" V 5354 3330 50  0000 C CNN
 F 2 "Resistor_SMD:R_0603_1608Metric" V 5400 3330 50  0001 C CNN
 F 3 "~" H 5470 3330 50  0001 C CNN
@@
 P 7460 2650
 F 0 "R27" H 7530 2696 50  0000 L CNN
-F 1 "330" H 7530 2605 50  0000 L CNN
+F 1 "2.49k" H 7530 2605 50  0000 L CNN
 F 2 "Resistor_SMD:R_0603_1608Metric" V 7390 2650 50  0001 C CNN
 F 3 "~" H 7460 2650 50  0001 C CNN
@@
 P 7140 3500
 F 0 "R26" H 7070 3454 50  0000 R CNN
-F 1 "1k8" H 7070 3545 50  0000 R CNN
+F 1 "2.49k" H 7070 3545 50  0000 R CNN
 F 2 "Resistor_SMD:R_0603_1608Metric" V 7070 3500 50  0001 C CNN
 F 3 "~" H 7140 3500 50  0001 C CNN
@@
 P 6920 3300
 F 0 "R25" V 6713 3300 50  0000 C CNN
-F 1 "10k" V 6804 3300 50  0000 C CNN
+F 1 "15k" V 6804 3300 50  0000 C CNN
 F 2 "Resistor_SMD:R_0603_1608Metric" V 6850 3300 50  0001 C CNN
 F 3 "~" H 6920 3300 50  0001 C CNN

Commit message: Add BOM file and CPL file
Parts:
- E1: renamed from R5; LCSC (none) -> C22908
- LED0, LED1, LED2, LED3, LED4, LED5, LED6, LED7: LCSC (none) -> C73545
- Q0, Q1, Q2, Q3, Q4, Q5, Q6, Q7: LCSC (none) -> C8659
- R10, R13, R16, R19, R22, R25, R4, R7: LCSC (none) -> C100780
- R11, R12, R14, R15, R17, R18, R20, R21, R23, R24, R26, R27, R6, R8, R9: LCSC (none) -> C22908
- R60, R61, R62, R63, R64, R65, R66, R67, R68, R69, R70, R71, R72, R73: LCSC (none) -> C23138
