File: digitalSystemBoard/DISPLAY.sch (KiCad schematic (older format))
At the start: 58 parts, among them Q0 BC847, Q1 BC847, Q2 BC847, Q3 BC847, Q4 BC847, Q5 BC847, Q6 BC847, Q7 BC847, U0 KCSA02-105, U1 KCSA02-105, U2 74LS47, U3 74LS47

Commit message: Synchronize the name of all the device
Parts:
- renumbered E1 to R5
Changed lines of the file:
@@
 $EndComp
 $Comp
-L Device:R E1
+L Device:R R5
 U 1 1 5FBB8D71
 P 2670 1770
-F 0 "E1" H 2600 1724 50  0000 R CNN
+F 0 "R5" H 2600 1724 50  0000 R CNN
 F 1 "2.49k" H 2600 1815 50  0000 R CNN
 F 2 "Resistor_SMD:R_0603_1608Metric" V 2600 1770 50  0001 C CNN
