File: digitalSystemBoard/MCU.sch (KiCad schematic (older format))
At the start: 31 parts, among them J4 USB-B, SW9 ButtonFirst, U16 ATmega32U4-AU, U17 ICSP, U18 74LS165, U19 74HC164, U20 74LS165, U21 74HC164, Y1 16MHz

Commit message: Change grid size of all schematic
Other:
- moved on the sheet: C10, D10, DS1, FB0, J4, R57, R58, R59, R60, SW9

Commit message: Update Schematic for review
Parts:
- C10, C11, C12, C13, C14, C15, C16, C17: footprint (none) -> Capacitor_SMD:C_0603_1608Metric
- D10: footprint SC70-6 -> digitalSystemBoard:SC70-6
- FB0, FB1, FB2, FB3, FB4, FB5: footprint (none) -> footprints:FerriteBead
- J2: renamed from J4; footprint SAMTEC_USB-B-S-X-X-TH-TR -> digitalSystemBoard:SAMTEC_USB-B-S-X-X-TH-TR
- R57, R58, R59, R60, R61, R62: footprint (none) -> Resistor_SMD:R_0603_1608Metric
- SW9: footprint TE_4-1437565-9 -> digitalSystemBoard:Button_CLOCK
- U17: footprint (none) -> Connector_PinHeader_2.54mm:PinHeader_2x03_P2.54mm_Vertical_SMD
- Y1: footprint (none) -> Crystal:Crystal_SMD_Abracon_ABM3B-4Pin_5.0x3.2mm
Connections:
- net 7SEGLED_TEST_ON: now reaches U16.30 (PB6)
- net 7SEGLED_TEST_OFF: now reaches U16.32 (PC7)
- no-connect marks 8 -> 6
Other:
- moved on the sheet: FB0
Changed lines of the file:
@@
 F 0 "R62" H 2040 4386 50  0000 L CNN
 F 1 "1M" H 2020 4320 50  0000 L CNN
-F 2 "" V 1900 4340 50  0001 C CNN
+F 2 "Resistor_SMD:R_0603_1608Metric" V 1900 4340 50  0001 C CNN
 F 3 "~" H 1970 4340 50  0001 C CNN
 	1    1970 4340
@@
 F 0 "Y1" V 1674 4450 50  0000 L CNN
 F 1 "16MHz" V 1710 4210 50  0000 L CNN
-F 2 "" H 1695 4340 50  0001 C CNN
+F 2 "Crystal:Crystal_SMD_Abracon_ABM3B-4Pin_5.0x3.2mm" H 1695 4340 50  0001 C CNN
 F 3 "" H 1695 4340 50  0001 C CNN
 	1    1720 4340
@@
 F 0 "C12" V 1480 4490 50  0000 C CNN
 F 1 "22pF" V 1400 4360 50  0000 C CNN
-F 2 "" H 1398 4340 50  0001 C CNN
+F 2 "Capacitor_SMD:C_0603_1608Metric" H 1398 4340 50  0001 C CNN
 F 3 "~" H 1360 4490 50  0001 C CNN
 	1    1360 4490
@@
 F 0 "C11" V 1230 4190 50  0000 C CNN
 F 1 "22pF" V 1320 4060 50  0000 C CNN
-F 2 "" H 1398 4040 50  0001 C CNN
+F 2 "Capacitor_SMD:C_0603_1608Metric" H 1398 4040 50  0001 C CNN
 F 3 "~" H 1360 4190 50  0001 C CNN
 	1    1360 4190
 	0    1    1    0
-$EndComp
-$Comp
-L MCU_Microchip_ATmega:ATmega32U4-AU U16
-U 1 1 5FBA4BA5
-P 2870 5540
-F 0 "U16" H 2870 5540 50  0000 C CNN
-F 1 "ATmega32U4-AU" H 2770 5460 50  0000 C CNN
-F 2 "Package_QFP:TQFP-44_10x10mm_P0.8mm" H 2870 5540 50  0001 C CIN
-F 3 "http://ww1.microchip.com/downloads/en/DeviceDoc/Atmel-7766-8-bit-AVR-ATmega16U4-32U4_Datasheet.pdf" H 2870 5540 50  0001 C CNN
-	1    2870 5540
-	1    0    0    -1
 $EndComp
 Wire Wire Line
@@
 F 0 "FB4" V 930 5110 50  0000 C CNN
 F 1 "80Ohm" V 860 5110 50  0000 C CNN
-F 2 "" V 1020 5110 50  0001 C CNN
+F 2 "footprints:FerriteBead" V 1020 5110 50  0001 C CNN
 F 3 "~" H 1090 5110 50  0001 C CNN
 	1    1090 5110
@@
 F 0 "C13" V 838 4900 50  0000 C CNN
 F 1 "0.1uF" V 929 4900 50  0000 C CNN
-F 2 "" H 1128 4750 50  0001 C CNN
+F 2 "Capacitor_SMD:C_0603_1608Metric" H 1128 4750 50  0001 C CNN
 F 3 "~" H 1090 4900 50  0001 C CNN
 	1    1090 4900
@@
 F 0 "FB5" V 930 5870 50  0000 C CNN
 F 1 "80Ohm" V 860 5870 50  0000 C CNN
-F 2 "" V 1020 5870 50  0001 C CNN
+F 2 "footprints:FerriteBead" V 1020 5870 50  0001 C CNN
 F 3 "~" H 1090 5870 50  0001 C CNN
 	1    1090 5870
@@
 F 0 "C14" V 900 5660 50  0000 C CNN
 F 1 "0.1uF" V 960 5660 50  0000 C CNN
-F 2 "" H 1128 5510 50  0001 C CNN
+F 2 "Capacitor_SMD:C_0603_1608Metric" H 1128 5510 50  0001 C CNN
 F 3 "~" H 1090 5660 50  0001 C CNN
 	1    1090 5660
@@
 F 0 "FB1" V 1790 3350 50  0000 C CNN
 F 1 "80Ohm" V 1720 3350 50  0000 C CNN
-F 2 "" V 1880 3350 50  0001 C CNN
+F 2 "footprints:FerriteBead" V 1880 3350 50  0001 C CNN
 F 3 "~" H 1950 3350 50  0001 C CNN
 	1    1950 3350
@@
 F 0 "C15" V 1908 3350 50  0000 C CNN
 F 1 "0.1uF" V 1999 3350 50  0000 C CNN
-F 2 "" H 2198 3200 50  0001 C CNN
+F 2 "Capacitor_SMD:C_0603_1608Metric" H 2198 3200 50  0001 C CNN
 F 3 "~" H 2160 3350 50  0001 C CNN
 	1    2160 3350
@@
 F 0 "FB2" V 2600 3350 50  0000 C CNN
 F 1 "80Ohm" V 2530 3350 50  0000 C CNN
-F 2 "" V 2690 3350 50  0001 C CNN
+F 2 "footprints:FerriteBead" V 2690 3350 50  0001 C CNN
 F 3 "~" H 2760 3350 50  0001 C CNN
 	1    2760 3350
@@
 F 0 "C16" V 2718 3350 50  0000 C CNN
 F 1 "0.1uF" V 2809 3350 50  0000 C CNN
-F 2 "" H 3008 3200 50  0001 C CNN
+F 2 "Capacitor_SMD:C_0603_1608Metric" H 3008 3200 50  0001 C CNN
 F 3 "~" H 2970 3350 50  0001 C CNN
 	1    2970 3350
@@
 F 0 "FB3" V 3390 3360 50  0000 C CNN
 F 1 "80Ohm" V 3320 3360 50  0000 C CNN
-F 2 "" V 3480 3360 50  0001 C CNN
+F 2 "footprints:FerriteBead" V 3480 3360 50  0001 C CNN
 F 3 "~" H 3550 3360 50  0001 C CNN
 	1    3550 3360
@@
 F 0 "C17" V 3508 3360 50  0000 C CNN
 F 1 "0.1uF" V 3599 3360 50  0000 C CNN
-F 2 "" H 3798 3210 50  0001 C CNN
+F 2 "Capacitor_SMD:C_0603_1608Metric" H 3798 3210 50  0001 C CNN
 F 3 "~" H 3760 3360 50  0001 C CNN
 	1    3760 3360
@@
 F 0 "R61" V 3800 6140 50  0000 C CNN
 F 1 "10k" V 3870 6140 50  0000 C CNN
-F 2 "" V 3800 6140 50  0001 C CNN
+F 2 "Resistor_SMD:R_0603_1608Metric" V 3800 6140 50  0001 C CNN
 F 3 "~" H 3870 6140 50  0001 C CNN
 	1    3870 6140
@@
 F 0 "U17" H 5968 6938 50  0000 L CNN
 F 1 "ICSP" H 5968 6847 50  0000 L CNN
-F 2 "" H 5690 7050 50  0001 C CNN
+F 2 "Connector_PinHeader_2.54mm:PinHeader_2x03_P2.54mm_Vertical_SMD" H 5690 7050 50  0001 C CNN
 F 3 "" H 5690 7050 50  0001 C CNN
 	1    5440 6950
@@
 F 0 "R60" H 9380 1196 50  0000 L CNN
 F 1 "10K" V 9310 1070 50  0000 L CNN
-F 2 "" V 9240 1150 50  0001 C CNN
+F 2 "Resistor_SMD:R_0603_1608Metric" V 9240 1150 50  0001 C CNN
 F 3 "~" H 9310 1150 50  0001 C CNN
 	1    9310 1150
@@
 F 0 "SW9" H 9850 1835 50  0000 C CNN
 F 1 "ButtonFirst" H 9850 1744 50  0000 C CNN
-F 2 "TE_4-1437565-9" H 9850 1520 50  0001 L BNN
+F 2 "digitalSystemBoard:Button_CLOCK" H 9850 1520 50  0001 L BNN
 F 3 "4-1437565-9" H 9850 1520 50  0001 L BNN
 F 4 "50 mA" H 9850 1520 50  0001 L BNN "Field4"
@@
 F 0 "R59" V 3230 1590 50  0000 C CNN
 F 1 "22" V 3150 1590 50  0000 C CNN
-F 2 "" V 3080 1590 50  0001 C CNN
+F 2 "Resistor_SMD:R_0603_1608Metric" V 3080 1590 50  0001 C CNN
 F 3 "~" H 3150 1590 50  0001 C CNN
 	1    3150 1590
@@
 F 0 "R57" V 1620 1200 50  0000 C CNN
 F 1 "22" V 1700 1190 50  0000 C CNN
-F 2 "" V 1630 1190 50  0001 C CNN
+F 2 "Resistor_SMD:R_0603_1608Metric" V 1630 1190 50  0001 C CNN
 F 3 "~" H 1700 1190 50  0001 C CNN
 	1    1700 1190
@@
 	0    -1   -1   0
 $EndComp
-Text Label 1550 1990 2    50   ~ 0
+Text Label 1550 2020 2    50   ~ 0
 VBUS
 $Comp
 L Device:Ferrite_Bead FB0
 U 1 1 5FBE302A
-P 1550 1840
-F 0 "FB0" V 1340 1840 50  0000 C CNN
-F 1 "80Ohm" V 1420 1840 50  0000 C CNN
-F 2 "" V 1480 1840 50  0001 C CNN
-F 3 "~" H 1550 1840 50  0001 C CNN
-	1    1550 1840
-	-1   0    0    1
-$EndComp
-$Comp
-L digitalSystemBoard:USB-B-S-X-X-TH-TR J4
+P 1550 1870
+F 0 "FB0" V 1340 1870 50  0000 C CNN
+F 1 "80Ohm" V 1420 1870 50  0000 C CNN
+F 2 "footprints:FerriteBead" V 1480 1870 50  0001 C CNN
+F 3 "~" H 1550 1870 50  0001 C CNN
+	1    1550 1870
+	-1   0    0    1
+$EndComp
+$Comp
+L digitalSystemBoard:USB-B-S-X-X-TH-TR J2
 U 1 1 5FBE04C8
 P 1150 1490
-F 0 "J4" H 1043 923 50  0000 C CNN
+F 0 "J2" H 1043 923 50  0000 C CNN
 F 1 "USB-B" H 1043 1014 50  0000 C CNN
-F 2 "SAMTEC_USB-B-S-X-X-TH-TR" H 1150 1490 50  0001 L BNN
+F 2 "digitalSystemBoard:SAMTEC_USB-B-S-X-X-TH-TR" H 1150 1490 50  0001 L BNN
 F 3 "Samtec" H 1150 1490 50  0001 L BNN
 F 4 "Manufacturer Recommendations" H 1150 1490 50  0001 L BNN "Field4"
@@
 Text Label 3470 4940 0    50   ~ 0
 LCD_ENABLE
-NoConn ~ 3470 4640
-NoConn ~ 3470 5040
 Text Label 2150 1700 2    50   ~ 0
 VBUS
@@
 F 0 "D10" H 2500 1650 50  0000 R CNN
 F 1 "SMF05C.TCT" H 3040 1650 50  0000 R CNN
-F 2 "SC70-6" H 2450 1800 50  0001 L BNN
+F 2 "digitalSystemBoard:SC70-6" H 2450 1800 50  0001 L BNN
 F 3 "" H 2450 1800 59  0001 C CNN
 	1    2450 1800
@@
 F 0 "R58" V 3070 1490 50  0000 C CNN
 F 1 "22" V 3150 1490 50  0000 C CNN
-F 2 "" V 3080 1490 50  0001 C CNN
+F 2 "Resistor_SMD:R_0603_1608Metric" V 3080 1490 50  0001 C CNN
 F 3 "~" H 3150 1490 50  0001 C CNN
 	1    3150 1490
@@
 F 0 "C10" H 9075 1650 50  0000 L CNN
 F 1 "0.1uF" H 9050 1550 50  0000 L CNN
-F 2 "" H 9348 1480 50  0001 C CNN
+F 2 "Capacitor_SMD:C_0603_1608Metric" H 9348 1480 50  0001 C CNN
 F 3 "~" H 9310 1630 50  0001 C CNN
 	1    9310 1630
@@
 	1    0    0    -1
 $EndComp
+$Comp
+L MCU_Microchip_ATmega:ATmega32U4-AU U16
+U 1 1 5FBA4BA5
+P 2870 5540
+F 0 "U16" H 2870 5540 50  0000 C CNN
+F 1 "ATmega32U4-AU" H 2770 5460 50  0000 C CNN
+F 2 "Package_QFP:TQFP-44_10x10mm_P0.8mm" H 2870 5540 50  0001 C CIN
+F 3 "http://ww1.microchip.com/downloads/en/DeviceDoc/Atmel-7766-8-bit-AVR-ATmega16U4-32U4_Datasheet.pdf" H 2870 5540 50  0001 C CNN
+	1    2870 5540
+	1    0    0    -1
+$EndComp
+Text HLabel 3470 4640 2    50   Input ~ 0
+7SEGLED_TEST_ON
+Text HLabel 3470 5040 2    50   Input ~ 0
+7SEGLED_TEST_OFF
+Wire Wire Line
+	1550 1690 1550 1720
 $EndSCHEMATC

Commit message: Add full footprint. Draw layout board
Parts:
- FB0, FB1, FB2, FB3, FB4, FB5: footprint footprints:FerriteBead -> digitalSystemBoard:FerriteBead
- U18, U20: footprint (none) -> Package_SO:SOIC-16_3.9x9.9mm_P1.27mm
- U19, U21: footprint (none) -> Package_SO:SOIC-14_3.9x8.7mm_P1.27mm
Connections:
- net GND: now also U17.6 (GND); no longer U17.2 (VCC)
- net MISO: now also U17.1 (MISO); no longer U17.4 (MOSI)
- net MOSI: now also U17.4 (MOSI); no longer U17.3 (SCK)
- net SCK: now also U17.3 (SCK); no longer U17.6 (GND)
- net VCC5V: now also U17.2 (VCC); no longer U17.1 (MISO)
Changed lines of the file:
@@
 F 0 "FB4" V 930 5110 50  0000 C CNN
 F 1 "80Ohm" V 860 5110 50  0000 C CNN
-F 2 "footprints:FerriteBead" V 1020 5110 50  0001 C CNN
+F 2 "digitalSystemBoard:FerriteBead" V 1020 5110 50  0001 C CNN
 F 3 "~" H 1090 5110 50  0001 C CNN
 	1    1090 5110
@@
 F 0 "FB5" V 930 5870 50  0000 C CNN
 F 1 "80Ohm" V 860 5870 50  0000 C CNN
-F 2 "footprints:FerriteBead" V 1020 5870 50  0001 C CNN
+F 2 "digitalSystemBoard:FerriteBead" V 1020 5870 50  0001 C CNN
 F 3 "~" H 1090 5870 50  0001 C CNN
 	1    1090 5870
@@
 F 0 "FB1" V 1790 3350 50  0000 C CNN
 F 1 "80Ohm" V 1720 3350 50  0000 C CNN
-F 2 "footprints:FerriteBead" V 1880 3350 50  0001 C CNN
+F 2 "digitalSystemBoard:FerriteBead" V 1880 3350 50  0001 C CNN
 F 3 "~" H 1950 3350 50  0001 C CNN
 	1    1950 3350
@@
 F 0 "FB2" V 2600 3350 50  0000 C CNN
 F 1 "80Ohm" V 2530 3350 50  0000 C CNN
-F 2 "footprints:FerriteBead" V 2690 3350 50  0001 C CNN
+F 2 "digitalSystemBoard:FerriteBead" V 2690 3350 50  0001 C CNN
 F 3 "~" H 2760 3350 50  0001 C CNN
 	1    2760 3350
@@
 F 0 "FB3" V 3390 3360 50  0000 C CNN
 F 1 "80Ohm" V 3320 3360 50  0000 C CNN
-F 2 "footprints:FerriteBead" V 3480 3360 50  0001 C CNN
+F 2 "digitalSystemBoard:FerriteBead" V 3480 3360 50  0001 C CNN
 F 3 "~" H 3550 3360 50  0001 C CNN
 	1    3550 3360
@@
 Wire Notes Line
 	6970 6540 4330 6540
-Text HLabel 5040 7200 3    50   Input ~ 0
+Text HLabel 5190 7200 3    50   Input ~ 0
 VCC5V
 $Comp
 L power:GND #PWR0115
 U 1 1 5FC0153F
-P 5190 7200
-F 0 "#PWR0115" H 5190 6950 50  0001 C CNN
-F 1 "GND" H 5195 7027 50  0000 C CNN
-F 2 "" H 5190 7200 50  0001 C CNN
-F 3 "" H 5190 7200 50  0001 C CNN
-	1    5190 7200
-	1    0    0    -1
-$EndComp
+P 5790 7200
+F 0 "#PWR0115" H 5790 6950 50  0001 C CNN
+F 1 "GND" H 5795 7027 50  0000 C CNN
+F 2 "" H 5790 7200 50  0001 C CNN
+F 3 "" H 5790 7200 50  0001 C CNN
+	1    5790 7200
+	1    0    0    -1
+$EndComp
+Text Label 5490 7200 3    50   ~ 0
+MOSI
+Text Label 5040 7200 3    50   ~ 0
+MISO
 Text Label 5340 7200 3    50   ~ 0
-MOSI
-Text Label 5490 7200 3    50   ~ 0
-MISO
-Text Label 5790 7200 3    50   ~ 0
 SCK
 Text Label 3470 4140 0    50   ~ 0
@@
 F 0 "U20" H 9405 2730 50  0000 C CNN
 F 1 "74LS165" H 9525 2650 50  0000 C CNN
-F 2 "" H 9290 3590 50  0001 C CNN
+F 2 "Package_SO:SOIC-16_3.9x9.9mm_P1.27mm" H 9290 3590 50  0001 C CNN
 F 3 "http://www.ti.com/lit/gpn/sn74LS165" H 9290 3590 50  0001 C CNN
 	1    9290 3590
@@
 F 0 "U21" H 9180 5955 50  0000 C CNN
 F 1 "74HC164" H 9055 6025 50  0000 C CNN
-F 2 "" H 10190 5200 50  0001 C CNN
+F 2 "Package_SO:SOIC-14_3.9x8.7mm_P1.27mm" H 10190 5200 50  0001 C CNN
 F 3 "https://assets.nexperia.com/documents/data-sheet/74HC_HCT164.pdf" H 10190 5200 50  0001 C CNN
 	1    9290 5500
@@
 F 0 "U19" H 6165 5950 50  0000 C CNN
 F 1 "74HC164" H 6055 6030 50  0000 C CNN
-F 2 "" H 7190 5200 50  0001 C CNN
+F 2 "Package_SO:SOIC-14_3.9x8.7mm_P1.27mm" H 7190 5200 50  0001 C CNN
 F 3 "https://assets.nexperia.com/documents/data-sheet/74HC_HCT164.pdf" H 7190 5200 50  0001 C CNN
 	1    6290 5500
@@
 F 0 "FB0" V 1340 1870 50  0000 C CNN
 F 1 "80Ohm" V 1420 1870 50  0000 C CNN
-F 2 "footprints:FerriteBead" V 1480 1870 50  0001 C CNN
+F 2 "digitalSystemBoard:FerriteBead" V 1480 1870 50  0001 C CNN
 F 3 "~" H 1550 1870 50  0001 C CNN
 	1    1550 1870
@@
 F 0 "U18" H 6380 2720 50  0000 C CNN
 F 1 "74LS165" H 6500 2645 50  0000 C CNN
-F 2 "" H 6290 3590 50  0001 C CNN
+F 2 "Package_SO:SOIC-16_3.9x9.9mm_P1.27mm" H 6290 3590 50  0001 C CNN
 F 3 "http://www.ti.com/lit/gpn/sn74LS165" H 6290 3590 50  0001 C CNN
 	1    6290 3590

Commit message: Layout 70 percent board
Connections:
- net at J2.2 (D-), R59.2: now also D10.6 (IO5); no longer D10.4 (IO3)
- net at J2.3 (D+), R58.2: now also D10.4 (IO3); no longer D10.6 (IO5)
Changed lines of the file:
@@
 NoConn ~ 2350 1700
 NoConn ~ 2750 1700
-Wire Wire Line
-	1550 1490 2950 1490
 $Comp
 L Device:R R58
@@
 	0    1    1    0
 $EndComp
-Wire Wire Line
-	3000 1590 2550 1590
-Wire Wire Line
-	2550 1700 2550 1590
-Connection ~ 2550 1590
-Wire Wire Line
-	2550 1590 1550 1590
-Wire Wire Line
-	2950 1700 2950 1490
-Connection ~ 2950 1490
-Wire Wire Line
-	2950 1490 3000 1490
 Wire Notes Line
 	4330 470  4330 7790
@@
 	1    0    0    -1
 $EndComp
+Wire Wire Line
+	1550 1590 2950 1590
+Wire Wire Line
+	1550 1490 2550 1490
+Wire Wire Line
+	2550 1700 2550 1490
+Connection ~ 2550 1490
+Wire Wire Line
+	2550 1490 3000 1490
+Wire Wire Line
+	2950 1700 2950 1590
+Connection ~ 2950 1590
+Wire Wire Line
+	2950 1590 3000 1590
 $EndSCHEMATC

Commit message: Hot fix: modifiy LCD footprint
Parts:
- DS1: footprint Display:WC1602A -> digitalSystemBoard:WC1602A
Changed lines of the file:
@@
 F 0 "DS1" V 6410 620 50  0000 L CNN
 F 1 "WC1602A" V 6480 620 50  0000 L CNN
-F 2 "Display:WC1602A" H 6060 420 50  0001 C CIN
+F 2 "digitalSystemBoard:WC1602A" H 6060 420 50  0001 C CIN
 F 3 "http://www.wincomlcd.com/pdf/WC1602A-SFYLYHTC06.pdf" H 6760 1320 50  0001 C CNN
 	1    6060 1320
