File: digitalSystemBoard/MCU.sch (KiCad schematic (older format))
At the start: 31 parts, among them J2 USB-B, SW9 ButtonFirst, U16 ATmega32U4-AU, U17 ICSP, U18 74LS165, U19 74HC164, U20 74LS165, U21 74HC164, Y1 16MHz

Commit message: Hot fix: Modify Reset button footprint
Connections:
- net GND: now also SW9.3; no longer SW9.2 (e~)
Changed lines of the file:
@@
 L power:GND #PWR0125
 U 1 1 5FBC2C2D
-P 10190 1420
-F 0 "#PWR0125" H 10190 1170 50  0001 C CNN
-F 1 "GND" V 10195 1292 50  0000 R CNN
-F 2 "" H 10190 1420 50  0001 C CNN
-F 3 "" H 10190 1420 50  0001 C CNN
-	1    10190 1420
+P 10100 1620
+F 0 "#PWR0125" H 10100 1370 50  0001 C CNN
+F 1 "GND" V 10105 1492 50  0000 R CNN
+F 2 "" H 10100 1620 50  0001 C CNN
+F 3 "" H 10100 1620 50  0001 C CNN
+	1    10100 1620
 	0    -1   -1   0
 $EndComp
@@
 Wire Wire Line
 	9600 1420 9310 1420
-Wire Wire Line
-	10190 1420 10100 1420
-NoConn ~ 10100 1620
-NoConn ~ 9600 1620
 $Comp
 L 74xx:74LS165 U18
@@
 	-1   0    0    1
 $EndComp
+NoConn ~ 9600 1620
+NoConn ~ 10100 1420
 $EndSCHEMATC

Commit message: Pull Up/Down Led
Parts:
- added R78: R, symbol Device:R
Connections:
- net VCC5V: now also R78.2; no longer DS1.15 (LED(+))
- new net: DS1.15 (LED(+)), R78.1
Changed lines of the file:
@@
 Text HLabel 6660 1720 3    50   Input ~ 0
 VCC5V
-Text HLabel 6360 1720 3    50   Input ~ 0
+Text HLabel 6360 2020 3    50   Input ~ 0
 VCC5V
 $Comp
@@
 NoConn ~ 9600 1620
 NoConn ~ 10100 1420
+$Comp
+L Device:R R78
+U 1 1 6048C364
+P 6360 1870
+F 0 "R78" H 6430 1916 50  0000 L CNN
+F 1 "R" H 6430 1825 50  0000 L CNN
+F 2 "" V 6290 1870 50  0001 C CNN
+F 3 "~" H 6360 1870 50  0001 C CNN
+	1    6360 1870
+	1    0    0    -1
+$EndComp
 $EndSCHEMATC

Commit message: Fix bug in BCD, add an rheostat on Vo and add an resistor on LED+
Parts:
- added TRIM2: Potentiometer, digitalSystemBoard:TRIM_3296W-1-501, symbol digitalSystemBoard:Potentiometer
- R78: footprint (none) -> Resistor_SMD:R_0603_1608Metric
Connections:
- net GND: now also TRIM2.3
- net VCC5V: now also TRIM2.1; no longer DS1.3 (VO)
- new net: DS1.3 (VO), TRIM2.2
Changed lines of the file:
@@
 $Descr A4 11693 8268
 encoding utf-8
-Sheet 2 5
+Sheet 5 5
 Title ""
 Date ""
@@
 	470  2360 11220 2360
 $Comp
-L Display_Character:WC1602A DS1
-U 1 1 5FC0BB5E
-P 6060 1320
-F 0 "DS1" V 6410 620 50  0000 L CNN
-F 1 "WC1602A" V 6480 620 50  0000 L CNN
-F 2 "digitalSystemBoard:WC1602A" H 6060 420 50  0001 C CIN
-F 3 "http://www.wincomlcd.com/pdf/WC1602A-SFYLYHTC06.pdf" H 6760 1320 50  0001 C CNN
-	1    6060 1320
-	0    1    1    0
-$EndComp
-$Comp
 L power:GND #PWR0116
 U 1 1 5FC0D995
@@
 $EndComp
 Text HLabel 6860 1320 2    50   Input ~ 0
-VCC5V
-Text HLabel 6660 1720 3    50   Input ~ 0
 VCC5V
 Text HLabel 6360 2020 3    50   Input ~ 0
@@
 F 0 "R78" H 6430 1916 50  0000 L CNN
 F 1 "R" H 6430 1825 50  0000 L CNN
-F 2 "" V 6290 1870 50  0001 C CNN
+F 2 "Resistor_SMD:R_0603_1608Metric" V 6290 1870 50  0001 C CNN
 F 3 "~" H 6360 1870 50  0001 C CNN
 	1    6360 1870
 	1    0    0    -1
 $EndComp
+$Comp
+L digitalSystemBoard:Potentiometer TRIM?
+U 1 1 6040D0E5
+P 7240 1910
+AR Path="/6040D0E5" Ref="TRIM?"  Part="1"
+AR Path="/5FBA4597/6040D0E5" Ref="TRIM2"  Part="1"
+F 0 "TRIM2" V 7261 2037 50  0000 L CNN
+F 1 "Potentiometer" V 7170 2037 50  0000 L CNN
+F 2 "digitalSystemBoard:TRIM_3296W-1-501" H 7240 1910 50  0001 C CNN
+F 3 "" H 7240 1910 50  0001 C CNN
+	1    7240 1910
+	0    1    1    0
+$EndComp
+$Comp
+L Display_Character:WC1602A DS1
+U 1 1 5FC0BB5E
+P 6060 1320
+F 0 "DS1" V 6410 620 50  0000 L CNN
+F 1 "WC1602A" V 6480 620 50  0000 L CNN
+F 2 "digitalSystemBoard:WC1602A" H 6060 420 50  0001 C CIN
+F 3 "http://www.wincomlcd.com/pdf/WC1602A-SFYLYHTC06.pdf" H 6760 1320 50  0001 C CNN
+	1    6060 1320
+	0    1    1    0
+$EndComp
+Text HLabel 7240 1610 1    50   Input ~ 0
+VCC5V
+$Comp
+L power:GND #PWR0167
+U 1 1 604177C1
+P 7240 2160
+F 0 "#PWR0167" H 7240 1910 50  0001 C CNN
+F 1 "GND" H 7245 1987 50  0000 C CNN
+F 2 "" H 7240 2160 50  0001 C CNN
+F 3 "" H 7240 2160 50  0001 C CNN
+	1    7240 2160
+	1    0    0    -1
+$EndComp
+Wire Wire Line
+	6660 1720 6660 1860
+Wire Wire Line
+	6660 1860 6890 1860
 $EndSCHEMATC

Commit message: Add IC 74HC595 and R for input pin
Parts:
- removed U19, U21: 74HC164, Package_SO:SOIC-14_3.9x8.7mm_P1.27mm, symbol digitalSystemBoard:74HC164
- added U19, U21: 74HC595, Package_SO:SOIC-16_3.9x9.9mm_P1.27mm, symbol 74xx:74HC595
Connections:
- net BCD_A_0: now also U21.15 (QA)
- net BCD_A_1: now also U21.4 (QE)
- net BCD_B_0: now also U21.1 (QB)
- net BCD_B_1: now also U21.5 (QF)
- net BCD_C_0: now also U21.2 (QC)
- net BCD_C_1: now also U21.6 (QG)
- net BCD_D_0: now also U21.3 (QD)
- net BCD_D_1: now also U21.7 (QH)
- net GND: now also U19.13 (~OE), U19.8 (GND), U21.13 (~OE), U21.8 (GND)
- net IC_CLOCK: now also U19.11 (SRCLK), U21.11 (SRCLK)
- net LED1: now also U19.15 (QA)
- net LED2: now also U19.1 (QB)
- net LED3: now also U19.2 (QC)
- net LED4: now also U19.3 (QD)
- net LED5: now also U19.4 (QE)
- net LED6: now also U19.5 (QF)
- net LED7: now also U19.6 (QG)
- net LED8: now also U19.7 (QH)
- net VCC5V: now also U19.10 (~SRCLR), U19.16 (VCC), U21.10 (~SRCLR), U21.16 (VCC)
- net IC_164_CTRL renamed IC_595_CTRL
- net IC_595_CTRL: now also U19.12 (RCLK), U21.12 (RCLK)
- net MCU_TO_IC_164 renamed MCU_TO_IC_595
- net MCU_TO_IC_595: now also U19.14 (SER)
- new net: U19.9 (QH'), U21.14 (SER)
- no-connect marks 6 -> 7
Changed lines of the file:
@@
 Text Label 6660 920  0    50   ~ 0
 LCD_ENABLE
-$Comp
-L 74xx:74LS165 U20
-U 1 1 5FB97CE1
-P 9290 3590
-F 0 "U20" H 9405 2730 50  0000 C CNN
-F 1 "74LS165" H 9525 2650 50  0000 C CNN
-F 2 "Package_SO:SOIC-16_3.9x9.9mm_P1.27mm" H 9290 3590 50  0001 C CNN
-F 3 "http://www.ti.com/lit/gpn/sn74LS165" H 9290 3590 50  0001 C CNN
-	1    9290 3590
-	1    0    0    -1
-$EndComp
-$Comp
-L digitalSystemBoard:74HC164 U19
-U 1 1 5FB99424
-P 6290 5500
-F 0 "U19" H 6165 5950 50  0000 C CNN
-F 1 "74HC164" H 6055 6030 50  0000 C CNN
-F 2 "Package_SO:SOIC-14_3.9x8.7mm_P1.27mm" H 7190 5200 50  0001 C CNN
-F 3 "https://assets.nexperia.com/documents/data-sheet/74HC_HCT164.pdf" H 7190 5200 50  0001 C CNN
-	1    6290 5500
-	-1   0    0    1
-$EndComp
 Text Label 6060 920  1    50   ~ 0
 LCD_1
@@
 Text Label 6160 920  1    50   ~ 0
 LCD_0
-Text HLabel 6690 5400 2    50   Input ~ 0
-VCC5V
-Text HLabel 9690 5400 2    50   Input ~ 0
-VCC5V
-Text HLabel 6290 6000 3    50   Input ~ 0
-VCC5V
-Text HLabel 9290 6000 3    50   Input ~ 0
-VCC5V
 Text HLabel 6290 2690 1    50   Input ~ 0
 VCC5V
 Text HLabel 9290 2690 1    50   Input ~ 0
 VCC5V
-Text Label 6690 5200 0    50   ~ 0
-IC_CLOCK
-Text Label 9690 5200 0    50   ~ 0
-IC_CLOCK
 Text Label 8790 4190 2    50   ~ 0
 IC_CLOCK
@@
 	1    0    0    -1
 $EndComp
-Wire Wire Line
-	6290 4900 6290 4740
-Wire Wire Line
-	6290 4740 6290 4590
-Connection ~ 6290 4740
 $Comp
 L power:GND #PWR0121
 U 1 1 5FC75B8B
-P 6290 4740
-F 0 "#PWR0121" H 6290 4490 50  0001 C CNN
-F 1 "GND" V 6295 4612 50  0000 R CNN
-F 2 "" H 6290 4740 50  0001 C CNN
-F 3 "" H 6290 4740 50  0001 C CNN
-	1    6290 4740
-	0    1    1    0
-$EndComp
-Wire Wire Line
-	9290 4725 9290 4590
-$Comp
-L power:GND #PWR0122
-U 1 1 5FC7F38D
-P 9290 4725
-F 0 "#PWR0122" H 9290 4475 50  0001 C CNN
-F 1 "GND" V 9295 4597 50  0000 R CNN
-F 2 "" H 9290 4725 50  0001 C CNN
-F 3 "" H 9290 4725 50  0001 C CNN
-	1    9290 4725
-	0    1    1    0
-$EndComp
-Connection ~ 9290 4725
-Wire Wire Line
-	9290 4900 9290 4725
+P 6290 4590
+F 0 "#PWR0121" H 6290 4340 50  0001 C CNN
+F 1 "GND" H 6210 4520 50  0000 R CNN
+F 2 "" H 6290 4590 50  0001 C CNN
+F 3 "" H 6290 4590 50  0001 C CNN
+	1    6290 4590
+	1    0    0    -1
+$EndComp
 $Comp
 L power:GND #PWR0123
@@
 Text Label 9790 2990 0    50   ~ 0
 IC_165_TO_MCU
-Text Label 6690 5500 0    50   ~ 0
-MCU_TO_IC_164
-Text Label 6690 5700 0    50   ~ 0
-IC_164_CTRL
-Text Label 9690 5700 0    50   ~ 0
-IC_164_CTRL
 Text HLabel 5790 3590 0    50   Input ~ 0
 GPIO_LED_6
@@
 Text HLabel 8790 3490 0    50   Input ~ 0
 GPIO_BCD_A_1
-Text HLabel 5890 5800 0    50   Input ~ 0
-LED1
-Text HLabel 5890 5700 0    50   Input ~ 0
-LED2
-Text HLabel 5890 5600 0    50   Input ~ 0
-LED3
-Text HLabel 5890 5500 0    50   Input ~ 0
-LED4
-Text HLabel 5890 5400 0    50   Input ~ 0
-LED5
-Text HLabel 5890 5300 0    50   Input ~ 0
-LED6
-Text HLabel 5890 5200 0    50   Input ~ 0
-LED7
-Text HLabel 5890 5100 0    50   Input ~ 0
-LED8
-Text HLabel 9690 5500 2    50   Input ~ 0
-LED8
-Text HLabel 8890 5800 0    50   Input ~ 0
+Text HLabel 9710 5120 2    50   Input ~ 0
 BCD_A_0
-Text HLabel 8890 5700 0    50   Input ~ 0
+Text HLabel 9710 5220 2    50   Input ~ 0
 BCD_B_0
-Text HLabel 8890 5600 0    50   Input ~ 0
+Text HLabel 9710 5320 2    50   Input ~ 0
 BCD_C_0
-Text HLabel 8890 5500 0    50   Input ~ 0
+Text HLabel 9710 5420 2    50   Input ~ 0
 BCD_D_0
-Text HLabel 8890 5400 0    50   Input ~ 0
+Text HLabel 9710 5520 2    50   Input ~ 0
 BCD_A_1
-Text HLabel 8890 5300 0    50   Input ~ 0
+Text HLabel 9710 5620 2    50   Input ~ 0
 BCD_B_1
-Text HLabel 8890 5200 0    50   Input ~ 0
+Text HLabel 9710 5720 2    50   Input ~ 0
 BCD_C_1
-Text HLabel 8890 5100 0    50   Input ~ 0
+Text HLabel 9710 5820 2    50   Input ~ 0
 BCD_D_1
 $Comp
@@
 IC_CLOCK
 Text Label 3470 4040 0    50   ~ 0
-MCU_TO_IC_164
+MCU_TO_IC_595
 Text Label 3470 5540 0    50   ~ 0
 IC_165_TO_MCU
 Text Label 3470 5640 0    50   ~ 0
-IC_164_CTRL
+IC_595_CTRL
 Text Label 3470 5940 0    50   ~ 0
 IC_165_CTRL
@@
 Wire Wire Line
 	2950 1590 3000 1590
-$Comp
-L digitalSystemBoard:74HC164 U21
-U 1 1 5FB9891A
-P 9290 5500
-F 0 "U21" H 9180 5955 50  0000 C CNN
-F 1 "74HC164" H 9055 6025 50  0000 C CNN
-F 2 "Package_SO:SOIC-14_3.9x8.7mm_P1.27mm" H 10190 5200 50  0001 C CNN
-F 3 "https://assets.nexperia.com/documents/data-sheet/74HC_HCT164.pdf" H 10190 5200 50  0001 C CNN
-	1    9290 5500
-	-1   0    0    1
-$EndComp
 NoConn ~ 9600 1620
 NoConn ~ 10100 1420
@@
 Wire Wire Line
 	6660 1860 6890 1860
+$Comp
+L 74xx:74LS165 U20
+U 1 1 5FB97CE1
+P 9290 3590
+F 0 "U20" H 9405 2730 50  0000 C CNN
+F 1 "74LS165" H 9525 2650 50  0000 C CNN
+F 2 "Package_SO:SOIC-16_3.9x9.9mm_P1.27mm" H 9290 3590 50  0001 C CNN
+F 3 "http://www.ti.com/lit/gpn/sn74LS165" H 9290 3590 50  0001 C CNN
+	1    9290 3590
+	1    0    0    -1
+$EndComp
+$Comp
+L power:GND #PWR0122
+U 1 1 60666149
+P 9290 4590
+F 0 "#PWR0122" H 9290 4340 50  0001 C CNN
+F 1 "GND" H 9210 4520 50  0000 R CNN
+F 2 "" H 9290 4590 50  0001 C CNN
+F 3 "" H 9290 4590 50  0001 C CNN
+	1    9290 4590
+	1    0    0    -1
+$EndComp
+$Comp
+L 74xx:74HC595 U21
+U 1 1 60679472
+P 9310 5520
+F 0 "U21" H 9560 4850 50  0000 C CNN
+F 1 "74HC595" H 9660 4760 50  0000 C CNN
+F 2 "Package_SO:SOIC-16_3.9x9.9mm_P1.27mm" H 9310 5520 50  0001 C CNN
+F 3 "http://www.ti.com/lit/ds/symlink/sn74hc595.pdf" H 9310 5520 50  0001 C CNN
+	1    9310 5520
+	1    0    0    -1
+$EndComp
+$Comp
+L power:GND #PWR0168
+U 1 1 6067E3F0
+P 6290 6230
+F 0 "#PWR0168" H 6290 5980 50  0001 C CNN
+F 1 "GND" H 6295 6057 50  0000 C CNN
+F 2 "" H 6290 6230 50  0001 C CNN
+F 3 "" H 6290 6230 50  0001 C CNN
+	1    6290 6230
+	1    0    0    -1
+$EndComp
+$Comp
+L power:GND #PWR0169
+U 1 1 6067EDB8
+P 9310 6220
+F 0 "#PWR0169" H 9310 5970 50  0001 C CNN
+F 1 "GND" H 9315 6047 50  0000 C CNN
+F 2 "" H 9310 6220 50  0001 C CNN
+F 3 "" H 9310 6220 50  0001 C CNN
+	1    9310 6220
+	1    0    0    -1
+$EndComp
+Text Label 5890 5130 2    50   ~ 0
+MCU_TO_IC_595
+$Comp
+L power:GND #PWR0170
+U 1 1 606883B2
+P 8810 5720
+F 0 "#PWR0170" H 8810 5470 50  0001 C CNN
+F 1 "GND" H 8660 5680 50  0000 C CNN
+F 2 "" H 8810 5720 50  0001 C CNN
+F 3 "" H 8810 5720 50  0001 C CNN
+	1    8810 5720
+	1    0    0    -1
+$EndComp
+Wire Wire Line
+	8910 5720 8810 5720
+Wire Wire Line
+	5890 5730 5790 5730
+$Comp
+L power:GND #PWR0171
+U 1 1 60683491
+P 5790 5730
+F 0 "#PWR0171" H 5790 5480 50  0001 C CNN
+F 1 "GND" H 5640 5690 50  0000 C CNN
+F 2 "" H 5790 5730 50  0001 C CNN
+F 3 "" H 5790 5730 50  0001 C CNN
+	1    5790 5730
+	1    0    0    -1
+$EndComp
+$Comp
+L 74xx:74HC595 U19
+U 1 1 60667CC7
+P 6290 5530
+F 0 "U19" H 6460 4860 50  0000 C CNN
+F 1 "74HC595" H 6550 4780 50  0000 C CNN
+F 2 "Package_SO:SOIC-16_3.9x9.9mm_P1.27mm" H 6290 5530 50  0001 C CNN
+F 3 "http://www.ti.com/lit/ds/symlink/sn74hc595.pdf" H 6290 5530 50  0001 C CNN
+	1    6290 5530
+	1    0    0    -1
+$EndComp
+Text HLabel 6690 5130 2    50   Input ~ 0
+LED1
+Text HLabel 6690 5230 2    50   Input ~ 0
+LED2
+Text HLabel 6690 5330 2    50   Input ~ 0
+LED3
+Text HLabel 6690 5430 2    50   Input ~ 0
+LED4
+Text HLabel 6690 5530 2    50   Input ~ 0
+LED5
+Text HLabel 6690 5630 2    50   Input ~ 0
+LED6
+Text HLabel 6690 5730 2    50   Input ~ 0
+LED7
+Text HLabel 6690 5830 2    50   Input ~ 0
+LED8
+Text HLabel 6290 4930 2    50   Input ~ 0
+VCC5V
+Text HLabel 9310 4920 2    50   Input ~ 0
+VCC5V
+Text HLabel 5890 5430 0    50   Input ~ 0
+VCC5V
+Text HLabel 8910 5420 0    50   Input ~ 0
+VCC5V
+Text Label 5890 5630 2    50   ~ 0
+IC_595_CTRL
+Text Label 8910 5620 2    50   ~ 0
+IC_595_CTRL
+Text Label 5890 5330 2    50   ~ 0
+IC_CLOCK
+Text Label 8910 5320 2    50   ~ 0
+IC_CLOCK
+Wire Wire Line
+	8910 5120 7760 5120
+Wire Wire Line
+	7760 5120 7760 6030
+Wire Wire Line
+	7760 6030 6690 6030
+NoConn ~ 9710 6020
 $EndSCHEMATC

Commit message: Fix name of all device
Parts:
- C10: renamed from C15; LCSC (none) -> C14663
- C11: renamed from C16; LCSC (none) -> C14663
- C12: renamed from C17; LCSC (none) -> C14663
- C5: renamed from C10; LCSC (none) -> C14663
- C6: renamed from C11; LCSC (none) -> C527592
- C7: renamed from C12; LCSC (none) -> C527592
- C8: renamed from C13; LCSC (none) -> C14663
- C9: renamed from C14; LCSC (none) -> C14663
- R0: renamed from R78; value R -> 220
- R57: renamed from R60; value 10K -> 10k
- renumbered DS1 to DS0, J2 to J1, R57 to R1, R58 to R2, R59 to R3, R61 to R58, R62 to R59, D10 to TD0, TRIM2 to TRIM0, U20 to U10, U21 to U11, U17 to U7, U18 to U8, U19 to U9, Y1 to Y0
Changed lines of the file:
@@
 VBUS
 $Comp
-L Device:R R62
+L Device:R R59
 U 1 1 5FBAC76A
 P 1970 4340
-F 0 "R62" H 2040 4386 50  0000 L CNN
+F 0 "R59" H 2040 4386 50  0000 L CNN
 F 1 "1M" H 2020 4320 50  0000 L CNN
 F 2 "Resistor_SMD:R_0603_1608Metric" V 1900 4340 50  0001 C CNN
@@
 $EndComp
 $Comp
-L digitalSystemBoard:Resonator Y1
+L digitalSystemBoard:Resonator Y0
 U 1 1 5FBACC99
 P 1720 4340
-F 0 "Y1" V 1674 4450 50  0000 L CNN
+F 0 "Y0" V 1674 4450 50  0000 L CNN
 F 1 "16MHz" V 1710 4210 50  0000 L CNN
 F 2 "Crystal:Crystal_SMD_Abracon_ABM3B-4Pin_5.0x3.2mm" H 1695 4340 50  0001 C CNN
@@
 $EndComp
 $Comp
-L Device:C C12
+L Device:C C7
 U 1 1 5FBAD313
 P 1360 4490
-F 0 "C12" V 1480 4490 50  0000 C CNN
+F 0 "C7" V 1480 4490 50  0000 C CNN
 F 1 "22pF" V 1400 4360 50  0000 C CNN
 F 2 "Capacitor_SMD:C_0603_1608Metric" H 1398 4340 50  0001 C CNN
 F 3 "~" H 1360 4490 50  0001 C CNN
+F 4 "C527592" H 1360 4490 50  0001 C CNN "LCSC"
 	1    1360 4490
 	0    1    1    0
 $EndComp
 $Comp
-L Device:C C11
+L Device:C C6
 U 1 1 5FBAD67B
 P 1360 4190
-F 0 "C11" V 1230 4190 50  0000 C CNN
+F 0 "C6" V 1230 4190 50  0000 C CNN
 F 1 "22pF" V 1320 4060 50  0000 C CNN
 F 2 "Capacitor_SMD:C_0603_1608Metric" H 1398 4040 50  0001 C CNN
 F 3 "~" H 1360 4190 50  0001 C CNN
+F 4 "C527592" H 1360 4190 50  0001 C CNN "LCSC"
 	1    1360 4190
 	0    1    1    0
@@
 $EndComp
 $Comp
-L Device:C C13
+L Device:C C8
 U 1 1 5FBBEEB7
 P 1090 4900
-F 0 "C13" V 838 4900 50  0000 C CNN
+F 0 "C8" V 838 4900 50  0000 C CNN
 F 1 "0.1uF" V 929 4900 50  0000 C CNN
 F 2 "Capacitor_SMD:C_0603_1608Metric" H 1128 4750 50  0001 C CNN
 F 3 "~" H 1090 4900 50  0001 C CNN
+F 4 "C14663" H 1090 4900 50  0001 C CNN "LCSC"
 	1    1090 4900
 	0    1    1    0
@@
 $EndComp
 $Comp
-L Device:C C14
+L Device:C C9
 U 1 1 5FBC4ABE
 P 1090 5660
-F 0 "C14" V 900 5660 50  0000 C CNN
+F 0 "C9" V 900 5660 50  0000 C CNN
 F 1 "0.1uF" V 960 5660 50  0000 C CNN
 F 2 "Capacitor_SMD:C_0603_1608Metric" H 1128 5510 50  0001 C CNN
 F 3 "~" H 1090 5660 50  0001 C CNN
+F 4 "C14663" H 1090 5660 50  0001 C CNN "LCSC"
 	1    1090 5660
 	0    1    1    0
@@
 $EndComp
 $Comp
-L Device:C C15
+L Device:C C10
 U 1 1 5FBC83FA
 P 2160 3350
-F 0 "C15" V 1908 3350 50  0000 C CNN
+F 0 "C10" V 1908 3350 50  0000 C CNN
 F 1 "0.1uF" V 1999 3350 50  0000 C CNN
 F 2 "Capacitor_SMD:C_0603_1608Metric" H 2198 3200 50  0001 C CNN
 F 3 "~" H 2160 3350 50  0001 C CNN
+F 4 "C14663" H 2160 3350 50  0001 C CNN "LCSC"
 	1    2160 3350
 	-1   0    0    1
@@
 $EndComp
 $Comp
-L Device:C C16
+L Device:C C11
 U 1 1 5FBC8F9A
 P 2970 3350
-F 0 "C16" V 2718 3350 50  0000 C CNN
+F 0 "C11" V 2718 3350 50  0000 C CNN
 F 1 "0.1uF" V 2809 3350 50  0000 C CNN
 F 2 "Capacitor_SMD:C_0603_1608Metric" H 3008 3200 50  0001 C CNN
 F 3 "~" H 2970 3350 50  0001 C CNN
+F 4 "C14663" H 2970 3350 50  0001 C CNN "LCSC"
 	1    2970 3350
 	-1   0    0    1
@@
 $EndComp
 $Comp
-L Device:C C17
+L Device:C C12
 U 1 1 5FBC9C66
 P 3760 3360
-F 0 "C17" V 3508 3360 50  0000 C CNN
+F 0 "C12" V 3508 3360 50  0000 C CNN
 F 1 "0.1uF" V 3599 3360 50  0000 C CNN
 F 2 "Capacitor_SMD:C_0603_1608Metric" H 3798 3210 50  0001 C CNN
 F 3 "~" H 3760 3360 50  0001 C CNN
+F 4 "C14663" H 3760 3360 50  0001 C CNN "LCSC"
 	1    3760 3360
 	-1   0    0    1
@@
 	2160 3740 2770 3740
 $Comp
-L Device:R R61
+L Device:R R58
 U 1 1 5FBDAE81
 P 3870 6140
-F 0 "R61" V 3800 6140 50  0000 C CNN
+F 0 "R58" V 3800 6140 50  0000 C CNN
 F 1 "10k" V 3870 6140 50  0000 C CNN
 F 2 "Resistor_SMD:R_0603_1608Metric" V 3800 6140 50  0001 C CNN
@@
 $EndComp
 $Comp
-L Device:R R60
+L Device:R R57
 U 1 1 5FBBEA10
 P 9310 1150
-F 0 "R60" H 9380 1196 50  0000 L CNN
-F 1 "10K" V 9310 1070 50  0000 L CNN
+F 0 "R57" H 9380 1196 50  0000 L CNN
+F 1 "10k" V 9310 1070 50  0000 L CNN
 F 2 "Resistor_SMD:R_0603_1608Metric" V 9240 1150 50  0001 C CNN
 F 3 "~" H 9310 1150 50  0001 C CNN
@@
 $EndComp
 $Comp
-L Device:R R59
+L Device:R R3
 U 1 1 5FBF198E
 P 3150 1590
-F 0 "R59" V 3230 1590 50  0000 C CNN
+F 0 "R3" V 3230 1590 50  0000 C CNN
 F 1 "22" V 3150 1590 50  0000 C CNN
 F 2 "Resistor_SMD:R_0603_1608Metric" V 3080 1590 50  0001 C CNN
@@
 $EndComp
 $Comp
-L Device:R R57
+L Device:R R1
 U 1 1 5FBE7ED3
 P 1700 1190
-F 0 "R57" V 1620 1200 50  0000 C CNN
+F 0 "R1" V 1620 1200 50  0000 C CNN
 F 1 "22" V 1700 1190 50  0000 C CNN
 F 2 "Resistor_SMD:R_0603_1608Metric" V 1630 1190 50  0001 C CNN
@@
 $EndComp
 $Comp
-L digitalSystemBoard:USB-B-S-X-X-TH-TR J2
+L digitalSystemBoard:USB-B-S-X-X-TH-TR J1
 U 1 1 5FBE04C8
 P 1150 1490
-F 0 "J2" H 1043 923 50  0000 C CNN
+F 0 "J1" H 1043 923 50  0000 C CNN
 F 1 "USB-B" H 1043 1014 50  0000 C CNN
 F 2 "digitalSystemBoard:SAMTEC_USB-B-S-X-X-TH-TR" H 1150 1490 50  0001 L BNN
@@
 VBUS
 $Comp
-L digitalSystemBoard:SMF05C.TCT D10
+L digitalSystemBoard:SMF05C.TCT TD0
 U 1 1 5FBEABB6
 P 2450 1800
-F 0 "D10" H 2500 1650 50  0000 R CNN
+F 0 "TD0" H 2500 1650 50  0000 R CNN
 F 1 "SMF05C.TCT" H 3040 1650 50  0000 R CNN
 F 2 "digitalSystemBoard:SC70-6" H 2450 1800 50  0001 L BNN
@@
 NoConn ~ 2750 1700
 $Comp
-L Device:R R58
+L Device:R R2
 U 1 1 5FBF11A6
 P 3150 1490
-F 0 "R58" V 3070 1490 50  0000 C CNN
+F 0 "R2" V 3070 1490 50  0000 C CNN
 F 1 "22" V 3150 1490 50  0000 C CNN
 F 2 "Resistor_SMD:R_0603_1608Metric" V 3080 1490 50  0001 C CNN
@@
 LCD_7
 $Comp
-L Device:C C10
+L Device:C C5
 U 1 1 5FCA9D34
 P 9310 1630
-F 0 "C10" H 9075 1650 50  0000 L CNN
+F 0 "C5" H 9075 1650 50  0000 L CNN
 F 1 "0.1uF" H 9050 1550 50  0000 L CNN
 F 2 "Capacitor_SMD:C_0603_1608Metric" H 9348 1480 50  0001 C CNN
 F 3 "~" H 9310 1630 50  0001 C CNN
+F 4 "C14663" H 9310 1630 50  0001 C CNN "LCSC"
 	1    9310 1630
 	1    0    0    -1
@@
 	9600 1420 9310 1420
 $Comp
-L 74xx:74LS165 U18
+L 74xx:74LS165 U8
 U 1 1 5FB96DF9
 P 6290 3590
-F 0 "U18" H 6380 2720 50  0000 C CNN
+F 0 "U8" H 6380 2720 50  0000 C CNN
 F 1 "74LS165" H 6500 2645 50  0000 C CNN
 F 2 "Package_SO:SOIC-16_3.9x9.9mm_P1.27mm" H 6290 3590 50  0001 C CNN
@@
 P 2870 5540
 AR Path="/5FBA4BA5" Ref="U16"  Part="1"
-AR Path="/5FBA4597/5FBA4BA5" Ref="U16"  Part="1"
-F 0 "U16" H 2870 5540 50  0000 C CNN
+AR Path="/5FBA4597/5FBA4BA5" Ref="U6"  Part="1"
+F 0 "U6" H 2870 5540 50  0000 C CNN
 F 1 "ATmega32U4-AU" H 2770 5460 50  0000 C CNN
 F 2 "Package_QFP:TQFP-44_10x10mm_P0.8mm" H 2870 5540 50  0001 C CIN
@@
 	1550 1690 1550 1720
 $Comp
-L digitalSystemBoard:ICSP U17
+L digitalSystemBoard:ICSP U7
 U 1 1 5FCA6AE9
 P 5440 6950
-F 0 "U17" H 5968 6938 50  0000 L CNN
+F 0 "U7" H 5968 6938 50  0000 L CNN
 F 1 "ICSP" H 5968 6847 50  0000 L CNN
 F 2 "Connector_PinHeader_2.54mm:PinHeader_2x03_P2.54mm_Vertical_SMD" H 5690 7050 50  0001 C CNN
@@
 NoConn ~ 10100 1420
 $Comp
-L Device:R R78
+L Device:R R0
 U 1 1 6048C364
 P 6360 1870
-F 0 "R78" H 6430 1916 50  0000 L CNN
-F 1 "R" H 6430 1825 50  0000 L CNN
+F 0 "R0" H 6430 1916 50  0000 L CNN
+F 1 "220" H 6430 1825 50  0000 L CNN
 F 2 "Resistor_SMD:R_0603_1608Metric" V 6290 1870 50  0001 C CNN
 F 3 "~" H 6360 1870 50  0001 C CNN
@@
 P 7240 1910
 AR Path="/6040D0E5" Ref="TRIM?"  Part="1"
-AR Path="/5FBA4597/6040D0E5" Ref="TRIM2"  Part="1"
-F 0 "TRIM2" V 7261 2037 50  0000 L CNN
+AR Path="/5FBA4597/6040D0E5" Ref="TRIM0"  Part="1"
+F 0 "TRIM0" V 7261 2037 50  0000 L CNN
 F 1 "Potentiometer" V 7170 2037 50  0000 L CNN
 F 2 "digitalSystemBoard:TRIM_3296W-1-501" H 7240 1910 50  0001 C CNN
@@
 $EndComp
 $Comp
-L Display_Character:WC1602A DS1
+L Display_Character:WC1602A DS0
 U 1 1 5FC0BB5E
 P 6060 1320
-F 0 "DS1" V 6410 620 50  0000 L CNN
+F 0 "DS0" V 6410 620 50  0000 L CNN
 F 1 "WC1602A" V 6480 620 50  0000 L CNN
 F 2 "digitalSystemBoard:WC1602A" H 6060 420 50  0001 C CIN
@@
 	6660 1860 6890 1860
 $Comp
-L 74xx:74LS165 U20
+L 74xx:74LS165 U10
 U 1 1 5FB97CE1
 P 9290 3590
-F 0 "U20" H 9405 2730 50  0000 C CNN
+F 0 "U10" H 9405 2730 50  0000 C CNN
 F 1 "74LS165" H 9525 2650 50  0000 C CNN
 F 2 "Package_SO:SOIC-16_3.9x9.9mm_P1.27mm" H 9290 3590 50  0001 C CNN
@@
 $EndComp
 $Comp
-L 74xx:74HC595 U21
+L 74xx:74HC595 U11
 U 1 1 60679472
 P 9310 5520
-F 0 "U21" H 9560 4850 50  0000 C CNN
+F 0 "U11" H 9560 4850 50  0000 C CNN
 F 1 "74HC595" H 9660 4760 50  0000 C CNN
 F 2 "Package_SO:SOIC-16_3.9x9.9mm_P1.27mm" H 9310 5520 50  0001 C CNN
@@
 $EndComp
 $Comp
-L 74xx:74HC595 U19
+L 74xx:74HC595 U9
 U 1 1 60667CC7
 P 6290 5530
-F 0 "U19" H 6460 4860 50  0000 C CNN
+F 0 "U9" H 6460 4860 50  0000 C CNN
 F 1 "74HC595" H 6550 4780 50  0000 C CNN
 F 2 "Package_SO:SOIC-16_3.9x9.9mm_P1.27mm" H 6290 5530 50  0001 C CNN
