File: digitalSystemBoard/_autosave-digitalSystemBoard.kicad_pcb (KiCad board)
At the start: 2 copper layers, 180 x 130 mm, 200 parts, among them J0 Barrel_Jack, J1 USB-B, J10 Conn_02x03_Odd_Even, J11 Conn_02x03_Odd_Even, J2 Conn_02x04_Odd_Even, J3 Conn_02x04_Odd_Even, J4 Conn_02x08_Odd_Even, J5 Conn_02x07_Odd_Even, J6 Conn_02x07_Odd_Even, J7 Conn_02x08_Odd_Even, J8 Conn_02x03_Odd_Even, J9 Conn_02x03_Odd_Even, Q0 BC847, Q1 BC847, Q10 BC847, Q11 BC847, Q12 BC847, Q13 BC847, Q14 BC847, Q15 BC847, Q2 BC847, Q3 BC847, Q4 BC847, Q5 BC847, Q6 BC847, Q7 BC847, Q8 BC847, Q9 BC847, SW0 SW_SPDT, SW1 IO_Switch, SW2 IO_Switch, SW3 IO_Switch, SW4 IO_Switch, SW5 IO_Switch, SW6 IO_Switch, SW7 IO_Switch, SW8 IO_Switch, SW9 ButtonFirst, U0 KCSA02-105, U1 KCSA02-105, U10 74HC165, U11 74HC595, U2 74LS47, U3 74LS47, U4 74LS04, U5 Potentiometer, U6 ATmega32U4-AU, U7 ICSP, U8 74HC165, U9 74HC595, Y0 16MHz

Commit message: Add new footprint for led and button reset again
Parts:
- moved LED1 0.13 mm to (202.4, 135.0)
- moved LED3 0.13 mm to (182.5, 135.0)
- moved LED4 0.13 mm to (172.4, 135.0)
- moved LED5 0.13 mm to (162.4, 135.0)
- moved LED0 0.13 mm to (212.4, 135.0)
- turned SW9 to 0 degrees
